File: hardware/LCD.sch (KiCad schematic (older format))
At the start: 3 parts, among them IC11 LCD-016N002L

Commit message: Working on layout
Parts:
- RV1: Mfr. (none) -> Vishay; Mfr. No. (none) -> T73YP103KT20; Mouser (none) -> 72-T73YP103KT20
Changed lines of the file:
@@
 F 1 "10k" H 6580 3245 50  0000 R CNN
 F 2 "Potentiometer_THT:Potentiometer_Vishay_T73YP_Vertical" H 6650 3200 50  0001 C CNN
-F 3 "~" H 6650 3200 50  0001 C CNN
+F 3 "http://www.vishay.com/docs/51016/t73.pdf" H 6650 3200 50  0001 C CNN
+F 4 "Vishay" H 6650 3200 50  0001 C CNN "Mfr."
+F 5 "T73YP103KT20 " H 6650 3200 50  0001 C CNN "Mfr. No."
+F 6 "72-T73YP103KT20 " H 6650 3200 50  0001 C CNN "Mouser"
 	1    6650 3200
 	-1   0    0    1
