File: hardware/Processor.sch (KiCad schematic (older format))
At the start: 23 parts, among them IC1 74HC00, IC2 W65C02, IC3 74HC138, IC4 28C256, IC5 AS6C62256A, IC6 W65C22, IC7 W65C51

Commit message: Working on layout
Parts:
- removed R2: 10k, Resistor_THT:R_Axial_DIN0207_L6.3mm_D2.5mm_P7.62mm_Horizontal, symbol Device:R
- C1, C2, C3, C4, C5, C6, C7, C8: footprint Capacitor_THT:C_Rect_L4.6mm_W2.0mm_P2.50mm_MKS02_FKP02 -> Capacitor_THT:C_Rect_L4.0mm_W2.5mm_P2.50mm; Mfr. AVX -> TDK; Mfr. No. SR295E104MAATR2 -> FA18X8R1H104KRU06; Mouser 581-SR295E104MAATR2 -> 810-FA18X8R1H104KRU6
- D8, D9: value D_Schottky -> SD103A
- IC3: symbol Sweet-6502-Computer-rescue:74HC138-74xx -> 74xx:74HC138
- IC4: value 28C256 -> SYSTEM ROM; footprint Socket:DIP_Socket-28_W11.9_W12.7_W15.24_W17.78_W18.5_3M_228-1277-00-0602J -> Package_DIP:DIP-28_W15.24mm_LongPads; Mfr. No. 28-3554-10 -> 28-6553-10*; Mouser 535-28-3554-10 -> 535-28-6553-10
- R1: Mfr. Welwyn -> Vishay / BC Components; Mfr. No. MFR3-1M0FC -> SFR25H0001002JR500; Mouser 756-MFR3-1M0FC -> 594-SFR25H0001002JR5
- XTAL1: value ECS-100X -> 1MHz
Other:
- moved on the sheet: C4

Commit message: Working on Schematic
Parts:
- added C18: 100nF, Capacitor_THT:C_Rect_L4.0mm_W2.5mm_P2.50mm, symbol Device:C
- added D?: SD103A, Diode_THT:D_DO-35_SOD27_P7.62mm_Horizontal, symbol Device:D_Schottky
- added IC10: W65C22, Package_DIP:DIP-40_W15.24mm_LongPads, symbol Western_Design_Center:W65C22
- IC3: symbol 74xx:74HC138 -> Retro-PC-rescue:74HC138-74xx-Retro-PC-rescue
Connections:
- net labels added: LCD[0..7], ~CS_VIA_2, ~IRQ_VIA_2
- wire segments 244 -> 271
- no-connect marks 14 -> 13
Other:
- moved on the sheet: D9

Commit message: Working on layout
Parts:
- gave numbers to parts that had none: 1
Connections:
- net labels added: A[15..0], D[7..0]
- net labels removed: Address, Data
- wire segments 271 -> 272
Other:
- moved on the sheet: D14, D8, D9, R1
Changed lines of the file:
@@
 $Descr A3 16535 11693
 encoding utf-8
-Sheet 2 6
+Sheet 6 6
 Title "Retro PC"
 Date "2019-10-08"
@@
 NoConn ~ 4350 4500
 NoConn ~ 4350 5200
-Wire Wire Line
-	4350 4300 4400 4300
 $Comp
 L Device:R R?
@@
 NoConn ~ 4350 4900
 Wire Wire Line
-	4350 5400 4600 5400
-Wire Wire Line
 	4350 5300 4400 5300
 Wire Wire Line
@@
 Wire Wire Line
 	2850 6300 3250 6300
-Text Label 5050 7100 0    50   ~ 0
-Address
 Wire Wire Line
 	2850 5300 3250 5300
@@
 	4850 5000 4950 5000
 Connection ~ 4850 5000
-Text Label 5050 7000 0    50   ~ 0
-Data
 Wire Wire Line
 	4350 4700 4400 4700
@@
 Entry Wire Line
 	7650 3000 7550 3100
-Text Label 1700 5700 2    50   ~ 0
+Text Label 1700 5350 2    50   ~ 0
 ~IRQ_ACIA
 Wire Wire Line
-	1700 5400 1850 5400
-Wire Wire Line
-	2400 5700 1700 5700
-Text Label 1700 4400 2    50   ~ 0
+	1700 5050 1850 5050
+Wire Wire Line
+	2400 5350 1700 5350
+Text Label 1700 4350 2    50   ~ 0
 ~IRQ_VIA_1
 Wire Wire Line
-	1700 4400 1850 4400
-Wire Wire Line
-	2150 4400 2400 4400
-Wire Wire Line
-	2400 5400 2400 5700
-Wire Wire Line
-	2400 4400 2400 4700
-Connection ~ 2400 5400
-Connection ~ 2400 4400
-Wire Wire Line
-	2400 4150 2400 4400
-Wire Wire Line
-	2150 5400 2400 5400
-Wire Wire Line
-	2400 3750 2400 3850
+	1700 4350 1850 4350
+Wire Wire Line
+	2150 4350 2400 4350
+Wire Wire Line
+	2400 5050 2400 5350
+Connection ~ 2400 5050
+Connection ~ 2400 4350
+Wire Wire Line
+	2400 4100 2400 4350
+Wire Wire Line
+	2150 5050 2400 5050
+Wire Wire Line
+	2400 3700 2400 3800
 $Comp
 L power:+5V #PWR?
 U 1 1 5E0EA16C
-P 2400 3750
+P 2400 3700
 AR Path="/5E0EA16C" Ref="#PWR?"  Part="1"
 AR Path="/5EB09E21/5E0EA16C" Ref="#PWR03"  Part="1"
-F 0 "#PWR03" H 2400 3600 50  0001 C CNN
-F 1 "+5V" H 2415 3923 50  0000 C CNN
-F 2 "" H 2400 3750 50  0001 C CNN
-F 3 "" H 2400 3750 50  0001 C CNN
-	1    2400 3750
+F 0 "#PWR03" H 2400 3550 50  0001 C CNN
+F 1 "+5V" H 2415 3873 50  0000 C CNN
+F 2 "" H 2400 3700 50  0001 C CNN
+F 3 "" H 2400 3700 50  0001 C CNN
+	1    2400 3700
 	1    0    0    -1
 $EndComp
@@
 L Device:R R?
 U 1 1 5E0EA165
-P 2400 4000
+P 2400 3950
 AR Path="/5E0EA165" Ref="R?"  Part="1"
 AR Path="/5EB09E21/5E0EA165" Ref="R1"  Part="1"
-F 0 "R1" H 2470 4046 50  0000 L CNN
-F 1 "10k" H 2470 3955 50  0000 L CNN
-F 2 "Resistor_THT:R_Axial_DIN0207_L6.3mm_D2.5mm_P7.62mm_Horizontal" V 2330 4000 50  0001 C CNN
-F 3 "https://www.mouser.de/datasheet/2/427/sfr16s25-239894.pdf" H 2400 4000 50  0001 C CNN
-F 4 "Vishay / BC Components" H 2400 4000 50  0001 C CNN "Mfr."
-F 5 "SFR25H0001002JR500" H 2400 4000 50  0001 C CNN "Mfr. No."
-F 6 "594-SFR25H0001002JR5" H 2400 4000 50  0001 C CNN "Mouser"
-	1    2400 4000
+F 0 "R1" H 2470 3996 50  0000 L CNN
+F 1 "10k" H 2470 3905 50  0000 L CNN
+F 2 "Resistor_THT:R_Axial_DIN0207_L6.3mm_D2.5mm_P7.62mm_Horizontal" V 2330 3950 50  0001 C CNN
+F 3 "https://www.mouser.de/datasheet/2/427/sfr16s25-239894.pdf" H 2400 3950 50  0001 C CNN
+F 4 "Vishay / BC Components" H 2400 3950 50  0001 C CNN "Mfr."
+F 5 "SFR25H0001002JR500" H 2400 3950 50  0001 C CNN "Mfr. No."
+F 6 "594-SFR25H0001002JR5" H 2400 3950 50  0001 C CNN "Mouser"
+	1    2400 3950
 	-1   0    0    1
 $EndComp
-Text HLabel 1700 5400 0    50   Input ~ 0
+Text HLabel 1700 5050 0    50   Input ~ 0
 ~IRQ
 $Comp
 L Device:D_Schottky D9
 U 1 1 5E0A358A
-P 2000 5400
-F 0 "D9" H 2000 5616 50  0000 C CNN
-F 1 "SD103A" H 2000 5525 50  0000 C CNN
-F 2 "Diode_THT:D_DO-35_SOD27_P7.62mm_Horizontal" H 2000 5400 50  0001 C CNN
-F 3 "https://www.vishay.com/docs/85754/sd103a.pdf" H 2000 5400 50  0001 C CNN
-F 4 "Vishay Semiconductors" H 2000 5400 50  0001 C CNN "Mfr."
-F 5 "SD103A-TR" H 2000 5400 50  0001 C CNN "Mfr. No."
-F 6 "625-SD103A" H 2000 5400 50  0001 C CNN "Mouser"
-	1    2000 5400
+P 2000 5050
+F 0 "D9" H 2000 5266 50  0000 C CNN
+F 1 "SD103A" H 2000 5175 50  0000 C CNN
+F 2 "Diode_THT:D_DO-35_SOD27_P7.62mm_Horizontal" H 2000 5050 50  0001 C CNN
+F 3 "https://www.vishay.com/docs/85754/sd103a.pdf" H 2000 5050 50  0001 C CNN
+F 4 "Vishay Semiconductors" H 2000 5050 50  0001 C CNN "Mfr."
+F 5 "SD103A-TR" H 2000 5050 50  0001 C CNN "Mfr. No."
+F 6 "625-SD103A" H 2000 5050 50  0001 C CNN "Mouser"
+	1    2000 5050
 	1    0    0    -1
 $EndComp
@@
 L Device:D_Schottky D8
 U 1 1 5E087BEB
-P 2000 4400
-F 0 "D8" H 2000 4616 50  0000 C CNN
-F 1 "SD103A" H 2000 4525 50  0000 C CNN
-F 2 "Diode_THT:D_DO-35_SOD27_P7.62mm_Horizontal" H 2000 4400 50  0001 C CNN
-F 3 "https://www.vishay.com/docs/85754/sd103a.pdf" H 2000 4400 50  0001 C CNN
-F 4 "Vishay Semiconductors" H 2000 4400 50  0001 C CNN "Mfr."
-F 5 "SD103A-TR" H 2000 4400 50  0001 C CNN "Mfr. No."
-F 6 "625-SD103A" H 2000 4400 50  0001 C CNN "Mouser"
-	1    2000 4400
+P 2000 4350
+F 0 "D8" H 2000 4566 50  0000 C CNN
+F 1 "SD103A" H 2000 4475 50  0000 C CNN
+F 2 "Diode_THT:D_DO-35_SOD27_P7.62mm_Horizontal" H 2000 4350 50  0001 C CNN
+F 3 "https://www.vishay.com/docs/85754/sd103a.pdf" H 2000 4350 50  0001 C CNN
+F 4 "Vishay Semiconductors" H 2000 4350 50  0001 C CNN "Mfr."
+F 5 "SD103A-TR" H 2000 4350 50  0001 C CNN "Mfr. No."
+F 6 "625-SD103A" H 2000 4350 50  0001 C CNN "Mouser"
+	1    2000 4350
 	1    0    0    -1
 $EndComp
@@
 Text HLabel 10050 1400 2    50   Input ~ 0
 LCD[0..7]
-Text Label 1650 4900 2    50   ~ 0
+Text Label 1700 4700 2    50   ~ 0
 ~IRQ_VIA_1
 Wire Wire Line
-	1650 4900 1800 4900
-$Comp
-L Device:D_Schottky D?
+	1700 4700 1850 4700
+$Comp
+L Device:D_Schottky D14
 U 1 1 5DEA544B
-P 1950 4900
-F 0 "D?" H 1950 5116 50  0000 C CNN
-F 1 "SD103A" H 1950 5025 50  0000 C CNN
-F 2 "Diode_THT:D_DO-35_SOD27_P7.62mm_Horizontal" H 1950 4900 50  0001 C CNN
-F 3 "https://www.vishay.com/docs/85754/sd103a.pdf" H 1950 4900 50  0001 C CNN
-F 4 "Vishay Semiconductors" H 1950 4900 50  0001 C CNN "Mfr."
-F 5 "SD103A-TR" H 1950 4900 50  0001 C CNN "Mfr. No."
-F 6 "625-SD103A" H 1950 4900 50  0001 C CNN "Mouser"
-	1    1950 4900
-	1    0    0    -1
-$EndComp
-Wire Wire Line
-	3250 4700 2400 4700
+P 2000 4700
+F 0 "D14" H 2000 4916 50  0000 C CNN
+F 1 "SD103A" H 2000 4825 50  0000 C CNN
+F 2 "Diode_THT:D_DO-35_SOD27_P7.62mm_Horizontal" H 2000 4700 50  0001 C CNN
+F 3 "https://www.vishay.com/docs/85754/sd103a.pdf" H 2000 4700 50  0001 C CNN
+F 4 "Vishay Semiconductors" H 2000 4700 50  0001 C CNN "Mfr."
+F 5 "SD103A-TR" H 2000 4700 50  0001 C CNN "Mfr. No."
+F 6 "625-SD103A" H 2000 4700 50  0001 C CNN "Mouser"
+	1    2000 4700
+	1    0    0    -1
+$EndComp
+Wire Wire Line
+	2150 4700 2400 4700
 Connection ~ 2400 4700
 Wire Wire Line
-	2400 4700 2400 5400
+	2400 4700 2400 5050
+Wire Wire Line
+	2400 4350 2400 4700
+Wire Wire Line
+	2400 4700 3250 4700
+Wire Bus Line
+	10000 4550 10550 4550
+Connection ~ 10000 4550
+Wire Bus Line
+	10150 4700 10550 4700
+Connection ~ 10150 4700
+Text HLabel 10550 4700 2    50   Output ~ 0
+A[15..0]
+Text HLabel 10550 4550 2    50   BiDi ~ 0
+D[7..0]
+Text HLabel 4800 5400 2    50   Output ~ 0
+R~W
+Wire Wire Line
+	4350 5400 4800 5400
+Text HLabel 4800 4300 2    50   Output ~ 0
+1MHz
+Wire Wire Line
+	4350 4300 4800 4300
+Wire Bus Line
+	10150 4700 10150 7100
 Wire Bus Line
 	7450 2600 7450 7100
 Wire Bus Line
-	10150 3050 10150 7100
+	10150 3050 10150 4700
 Wire Bus Line
 	12950 3100 12950 3800
@@
 	4800 5800 4800 7000
 Wire Bus Line
+	10000 3550 10000 4550
+Wire Bus Line
 	2750 5000 2750 7100
 Wire Bus Line
+	10000 4550 10000 7000
+Wire Bus Line
 	7900 3850 7900 7000
 Wire Bus Line
 	5750 4700 5750 7100
-Wire Bus Line
-	10000 3550 10000 7000
 $EndSCHEMATC

Commit message: Working on layout
Connections:
- wire segments 272 -> 270
Other:
- moved on the sheet: IC1B
Changed lines of the file:
@@
 Connection ~ 2750 7100
 Wire Wire Line
-	6750 7550 6800 7550
+	6750 7450 6800 7450
 $Comp
 L ECS:ECS-100X X?
@@
 Text HLabel 13900 7550 2    50   Output ~ 0
 ACIAReady
-Text Label 6750 7550 2    50   ~ 0
+Text Label 6750 7450 2    50   ~ 0
 1MHz
 Text Label 11200 7350 0    50   ~ 0
@@
 Text Label 11200 3150 0    50   ~ 0
 A2
-Wire Wire Line
-	6800 7750 6150 7750
 Text Label 3000 10200 0    50   ~ 0
 A15
 Entry Wire Line
 	2750 10100 2850 10200
-Wire Wire Line
-	6150 7750 6150 7650
-Wire Wire Line
-	6150 7650 4350 7650
 Wire Wire Line
 	9900 5700 9550 5700
@@
 	9550 6400 9650 6400
 Wire Wire Line
-	9650 6400 9650 7650
+	9650 6400 9650 7550
 Wire Wire Line
 	9650 6300 9550 6300
@@
 	5750 4700 5850 4600
 Wire Wire Line
-	9650 7650 7400 7650
+	9650 7550 7400 7550
 Entry Wire Line
 	2750 9800 2850 9900
@@
 L 74xx:74HC00 IC1
 U 2 1 5DE275DC
-P 7100 7650
-F 0 "IC1" H 7100 7975 50  0000 C CNN
-F 1 "74HC00" H 7100 7884 50  0000 C CNN
-F 2 "Package_DIP:DIP-14_W7.62mm_LongPads" H 7100 7650 50  0001 C CNN
-F 3 "http://www.ti.com/lit/gpn/sn74hc00" H 7100 7650 50  0001 C CNN
-F 4 "Texas Instruments" H 7100 7650 50  0001 C CNN "Mfr."
-F 5 "SN74HC00AN" H 7100 7650 50  0001 C CNN "Mfr. No."
-F 6 "595-SN74HC00AN" H 7100 7650 50  0001 C CNN "Mouser"
-	2    7100 7650
+P 7100 7550
+F 0 "IC1" H 7100 7875 50  0000 C CNN
+F 1 "74HC00" H 7100 7784 50  0000 C CNN
+F 2 "Package_DIP:DIP-14_W7.62mm_LongPads" H 7100 7550 50  0001 C CNN
+F 3 "http://www.ti.com/lit/gpn/sn74hc00" H 7100 7550 50  0001 C CNN
+F 4 "Texas Instruments" H 7100 7550 50  0001 C CNN "Mfr."
+F 5 "SN74HC00AN" H 7100 7550 50  0001 C CNN "Mfr. No."
+F 6 "595-SN74HC00AN" H 7100 7550 50  0001 C CNN "Mouser"
+	2    7100 7550
 	1    0    0    -1
 $EndComp
@@
 Wire Wire Line
 	4350 4300 4800 4300
+Wire Wire Line
+	4350 7650 6800 7650
 Wire Bus Line
 	10150 4700 10150 7100

Commit message: Working on layout
Parts:
- IC3: symbol Retro-PC-rescue:74HC138-74xx-Retro-PC-rescue -> 74xx:74HC138
Changed lines of the file:
@@
 ~CS_VIA_1
 $Comp
-L Retro-PC-rescue:74HC138-74xx-Retro-PC-rescue IC3
+L 74xx:74HC138 IC3
 U 1 1 5DA01AB5
 P 3750 10000
@@
 LCD[0..7]
 Text Label 1700 4700 2    50   ~ 0
-~IRQ_VIA_1
+~IRQ_VIA_2
 Wire Wire Line
 	1700 4700 1850 4700

Commit message: Working on layout
Parts:
- IC3: symbol 74xx:74HC138 -> Retro-PC-rescue:74HC138-74xx
Connections:
- net RxD: now also IC7.12 (RxD)
- net TxD: now also IC7.10 (TxD)
- net LCD0: now reaches IC10.10 (PB0)
- net LCD1: now reaches IC10.11 (PB1)
- net LCD2: now reaches IC10.12 (PB2)
- net PS20: now reaches IC10.16 (PB6)
- net PS21: now reaches IC10.17 (PB7)
- net LCD3: now reaches IC10.2 (PA0)
- net LCD4: now reaches IC10.3 (PA1)
- net LCD5: now reaches IC10.4 (PA2)
- net LCD6: now reaches IC10.5 (PA3)
- net LCD7: now reaches IC10.6 (PA4)
- net LCD8: now reaches IC10.7 (PA5)
- net LCD9: now reaches IC10.8 (PA6)
- net LCD10: now reaches IC10.9 (PA7)
- net ~ReceiverReady: now reaches IC7.11 (DTRB)
- net ~Carrier: now reaches IC7.16 (DCDB)
- net 1MHz renamed Clock
- net ModemReady renamed ~ModemReady
- no-connect marks 13 -> 20
Changed lines of the file:
@@
 $Descr A3 16535 11693
 encoding utf-8
-Sheet 6 6
+Sheet 5 6
 Title "Retro PC"
 Date "2019-10-08"
@@
 Text Label 4600 5400 0    50   ~ 0
 R~W
-Text HLabel 13900 6800 2    50   Output ~ 0
+Text HLabel 13900 7150 2    50   Output ~ 0
 TxD
-Text HLabel 13900 6900 2    50   Input ~ 0
+Text HLabel 13900 7250 2    50   Input ~ 0
 RxD
 Text HLabel 13900 7350 2    50   Output ~ 0
@@
 CTS
 Text HLabel 13900 7750 2    50   Input ~ 0
-ModemReady
-$Comp
-L power:GND #PWR?
-U 1 1 5F24C1CA
-P 12650 8300
-AR Path="/5F24C1CA" Ref="#PWR?"  Part="1"
-AR Path="/5EB09E21/5F24C1CA" Ref="#PWR032"  Part="1"
-F 0 "#PWR032" H 12650 8050 50  0001 C CNN
-F 1 "GND" H 12655 8127 50  0000 C CNN
-F 2 "" H 12650 8300 50  0001 C CNN
-F 3 "" H 12650 8300 50  0001 C CNN
-	1    12650 8300
-	1    0    0    -1
-$EndComp
-Wire Wire Line
-	12650 7850 12650 8300
-Text HLabel 13900 7550 2    50   Output ~ 0
-ACIAReady
+~ModemReady
 Text Label 6750 7450 2    50   ~ 0
 1MHz
@@
 Wire Wire Line
 	12550 6100 12650 6100
-NoConn ~ 12550 7250
+NoConn ~ 12550 7050
 Wire Wire Line
 	11300 6200 11450 6200
@@
 	12550 7750 13900 7750
 Wire Wire Line
-	12550 7850 12650 7850
-Wire Wire Line
 	12000 5250 12000 5900
 Wire Wire Line
 	10250 7000 11450 7000
 Wire Wire Line
-	13900 6900 12550 6900
-Wire Wire Line
-	12550 7550 13900 7550
-Wire Wire Line
-	12550 6800 13900 6800
+	13900 7250 12550 7250
+Wire Wire Line
+	12550 7150 13900 7150
 Wire Wire Line
 	12000 8300 12000 8150
@@
 ~CS_VIA_1
 $Comp
-L 74xx:74HC138 IC3
+L Retro-PC-rescue:74HC138-74xx IC3
 U 1 1 5DA01AB5
 P 3750 10000
@@
 Text Label 7900 2700 0    50   ~ 0
 A2
+Connection ~ 7900 7000
+Wire Bus Line
+	7900 7000 10000 7000
+Wire Bus Line
+	5750 7100 7450 7100
+Connection ~ 7450 7100
+Wire Bus Line
+	7450 7100 10150 7100
+Text HLabel 10050 1400 2    50   BiDi ~ 0
+LCD[0..10]
+Text Label 1700 4700 2    50   ~ 0
+~IRQ_VIA_2
+Wire Wire Line
+	1700 4700 1850 4700
+$Comp
+L Device:D_Schottky D14
+U 1 1 5DEA544B
+P 2000 4700
+F 0 "D14" H 2000 4916 50  0000 C CNN
+F 1 "SD103A" H 2000 4825 50  0000 C CNN
+F 2 "Diode_THT:D_DO-35_SOD27_P7.62mm_Horizontal" H 2000 4700 50  0001 C CNN
+F 3 "https://www.vishay.com/docs/85754/sd103a.pdf" H 2000 4700 50  0001 C CNN
+F 4 "Vishay Semiconductors" H 2000 4700 50  0001 C CNN "Mfr."
+F 5 "SD103A-TR" H 2000 4700 50  0001 C CNN "Mfr. No."
+F 6 "625-SD103A" H 2000 4700 50  0001 C CNN "Mouser"
+	1    2000 4700
+	1    0    0    -1
+$EndComp
+Wire Wire Line
+	2150 4700 2400 4700
+Connection ~ 2400 4700
+Wire Wire Line
+	2400 4700 2400 5050
+Wire Wire Line
+	2400 4350 2400 4700
+Wire Wire Line
+	2400 4700 3250 4700
+Wire Bus Line
+	10000 4550 10550 4550
+Connection ~ 10000 4550
+Wire Bus Line
+	10150 4700 10550 4700
+Connection ~ 10150 4700
+Text HLabel 10550 4700 2    50   Output ~ 0
+A[15..0]
+Text HLabel 10550 4550 2    50   BiDi ~ 0
+D[7..0]
+Text HLabel 4800 5400 2    50   Output ~ 0
+R~W
+Wire Wire Line
+	4350 5400 4800 5400
+Text HLabel 4800 4300 2    50   Output ~ 0
+Clock
+Wire Wire Line
+	4350 4300 4800 4300
+Wire Wire Line
+	4350 7650 6800 7650
 $Comp
 L Memory_EEPROM:28C256 IC?
@@
 	1    0    0    -1
 $EndComp
-Connection ~ 7900 7000
-Wire Bus Line
-	7900 7000 10000 7000
-Wire Bus Line
-	5750 7100 7450 7100
-Connection ~ 7450 7100
-Wire Bus Line
-	7450 7100 10150 7100
-Text HLabel 10050 1400 2    50   Input ~ 0
-LCD[0..7]
-Text Label 1700 4700 2    50   ~ 0
-~IRQ_VIA_2
-Wire Wire Line
-	1700 4700 1850 4700
-$Comp
-L Device:D_Schottky D14
-U 1 1 5DEA544B
-P 2000 4700
-F 0 "D14" H 2000 4916 50  0000 C CNN
-F 1 "SD103A" H 2000 4825 50  0000 C CNN
-F 2 "Diode_THT:D_DO-35_SOD27_P7.62mm_Horizontal" H 2000 4700 50  0001 C CNN
-F 3 "https://www.vishay.com/docs/85754/sd103a.pdf" H 2000 4700 50  0001 C CNN
-F 4 "Vishay Semiconductors" H 2000 4700 50  0001 C CNN "Mfr."
-F 5 "SD103A-TR" H 2000 4700 50  0001 C CNN "Mfr. No."
-F 6 "625-SD103A" H 2000 4700 50  0001 C CNN "Mouser"
-	1    2000 4700
-	1    0    0    -1
-$EndComp
-Wire Wire Line
-	2150 4700 2400 4700
-Connection ~ 2400 4700
-Wire Wire Line
-	2400 4700 2400 5050
-Wire Wire Line
-	2400 4350 2400 4700
-Wire Wire Line
-	2400 4700 3250 4700
-Wire Bus Line
-	10000 4550 10550 4550
-Connection ~ 10000 4550
-Wire Bus Line
-	10150 4700 10550 4700
-Connection ~ 10150 4700
-Text HLabel 10550 4700 2    50   Output ~ 0
-A[15..0]
-Text HLabel 10550 4550 2    50   BiDi ~ 0
-D[7..0]
-Text HLabel 4800 5400 2    50   Output ~ 0
-R~W
-Wire Wire Line
-	4350 5400 4800 5400
-Text HLabel 4800 4300 2    50   Output ~ 0
-1MHz
-Wire Wire Line
-	4350 4300 4800 4300
-Wire Wire Line
-	4350 7650 6800 7650
+Text HLabel 9900 2650 2    50   BiDi ~ 0
+PS2[0..1]
+Entry Wire Line
+	9700 3450 9800 3350
+Entry Wire Line
+	9700 3350 9800 3250
+Wire Wire Line
+	9700 3450 9300 3450
+Wire Wire Line
+	9300 3350 9700 3350
+Text Label 9450 3350 0    50   ~ 0
+PS20
+Text Label 9450 3450 0    50   ~ 0
+PS21
+Wire Bus Line
+	9800 2650 9900 2650
+Wire Bus Line
+	9750 1400 10050 1400
+Entry Wire Line
+	9650 1950 9750 1850
+Entry Wire Line
+	9650 2050 9750 1950
+Entry Wire Line
+	9650 2250 9750 2150
+Entry Wire Line
+	9650 2350 9750 2250
+Entry Wire Line
+	9650 2550 9750 2450
+Entry Wire Line
+	9650 2750 9750 2650
+Entry Wire Line
+	9650 2450 9750 2350
+Entry Wire Line
+	9650 2150 9750 2050
+Entry Wire Line
+	9650 1850 9750 1750
+Entry Wire Line
+	9650 2950 9750 2850
+Entry Wire Line
+	9650 2850 9750 2750
+Wire Wire Line
+	9650 1850 9300 1850
+Wire Wire Line
+	9300 1950 9650 1950
+Wire Wire Line
+	9650 2050 9300 2050
+Wire Wire Line
+	9300 2150 9650 2150
+Wire Wire Line
+	9650 2250 9300 2250
+Wire Wire Line
+	9300 2350 9650 2350
+Wire Wire Line
+	9650 2450 9300 2450
+Wire Wire Line
+	9300 2550 9650 2550
+Text Label 9400 1850 0    50   ~ 0
+LCD3
+Text Label 9400 1950 0    50   ~ 0
+LCD4
+Text Label 9400 2050 0    50   ~ 0
+LCD5
+Text Label 9400 2150 0    50   ~ 0
+LCD6
+Text Label 9400 2250 0    50   ~ 0
+LCD7
+Text Label 9400 2350 0    50   ~ 0
+LCD8
+Text Label 9400 2450 0    50   ~ 0
+LCD9
+Text Label 9400 2550 0    50   ~ 0
+LCD10
+Wire Wire Line
+	9300 2750 9650 2750
+Wire Wire Line
+	9650 2850 9300 2850
+Wire Wire Line
+	9300 2950 9650 2950
+Text Label 9400 2750 0    50   ~ 0
+LCD0
+Text Label 9400 2850 0    50   ~ 0
+LCD1
+Text Label 9400 2950 0    50   ~ 0
+LCD2
+Wire Wire Line
+	12550 7650 13900 7650
+Text HLabel 13900 7650 2    50   Output ~ 0
+~ReceiverReady
+Text HLabel 13900 7950 2    50   Input ~ 0
+~Carrier
+Wire Wire Line
+	12550 7950 13900 7950
+NoConn ~ 9300 3050
+NoConn ~ 9300 3150
+NoConn ~ 9300 3250
+NoConn ~ 9300 3600
+NoConn ~ 9300 3700
+NoConn ~ 9300 1600
+NoConn ~ 9300 1700
+Wire Bus Line
+	9800 2650 9800 3350
 Wire Bus Line
 	10150 4700 10150 7100
@@
 	2750 7100 2750 10300
 Wire Bus Line
+	9750 1400 9750 3100
+Wire Bus Line
 	7550 3100 7550 3850
 Wire Bus Line
 	10000 7000 10000 7850
 Wire Bus Line
+	10000 3550 10000 4550
+Wire Bus Line
 	4800 5800 4800 7000
 Wire Bus Line
-	10000 3550 10000 4550
-Wire Bus Line
 	2750 5000 2750 7100

Commit message: First version of the layout
Parts:
- IC10: Mfr. (none) -> Western Design Center; Mfr. No. (none) -> W65C22N6TPG-14; Mouser (none) -> 955-W65C22N6TPG-14
- IC3: symbol Retro-PC-rescue:74HC138-74xx -> 74xx:74HC138
- R1, R3: Mfr. Vishay / BC Components -> Yageo; Mfr. No. SFR25H0001002JR500 -> MFP-25BRD52-10K; Mouser 594-SFR25H0001002JR5 -> 603-MFP-25BRD52-10K
- R4: Mfr. Welwyn -> Yageo; Mfr. No. MFR3-1M0FC -> MFR-25FRE52-1M; Mouser 756-MFR3-1M0FC -> 603-MFR-25FRE52-1M
Changed lines of the file:
@@
 F 1 "10k" H 5120 5055 50  0000 L CNN
 F 2 "Resistor_THT:R_Axial_DIN0207_L6.3mm_D2.5mm_P7.62mm_Horizontal" V 4980 5100 50  0001 C CNN
-F 3 "https://www.mouser.de/datasheet/2/427/sfr16s25-239894.pdf" H 5050 5100 50  0001 C CNN
-F 4 "Vishay / BC Components" H 5050 5100 50  0001 C CNN "Mfr."
-F 5 "SFR25H0001002JR500" H 5050 5100 50  0001 C CNN "Mfr. No."
-F 6 "594-SFR25H0001002JR5" H 5050 5100 50  0001 C CNN "Mouser"
+F 3 "https://www.mouser.de/datasheet/2/447/Yageo%20LR_MFP_2013-594635.pdf" H 5050 5100 50  0001 C CNN
+F 4 "Yageo" H 5050 5100 50  0001 C CNN "Mfr."
+F 5 "MFP-25BRD52-10K" H 5050 5100 50  0001 C CNN "Mfr. No."
+F 6 "603-MFP-25BRD52-10K" H 5050 5100 50  0001 C CNN "Mouser"
 	1    5050 5100
 	0    1    1    0
@@
 F 1 "1M" H 12970 6105 50  0000 L CNN
 F 2 "Resistor_THT:R_Axial_DIN0207_L6.3mm_D2.5mm_P7.62mm_Horizontal" V 12830 6150 50  0001 C CNN
-F 3 "https://www.mouser.de/datasheet/2/414/MFR-1528371.pdf" H 12900 6150 50  0001 C CNN
-F 4 "Welwyn" H 12900 6150 50  0001 C CNN "Mfr."
-F 5 "MFR3-1M0FC" H 12900 6150 50  0001 C CNN "Mfr. No."
-F 6 "756-MFR3-1M0FC" H 12900 6150 50  0001 C CNN "Mouser"
+F 3 "https://www.mouser.de/datasheet/2/447/Yageo%20LR_MFR_2013-467719.pdf" H 12900 6150 50  0001 C CNN
+F 4 "Yageo" H 12900 6150 50  0001 C CNN "Mfr."
+F 5 "MFR-25FRE52-1M" H 12900 6150 50  0001 C CNN "Mfr. No."
+F 6 "603-MFR-25FRE52-1M" H 12900 6150 50  0001 C CNN "Mouser"
 	1    12900 6150
 	-1   0    0    1
@@
 ~CS_VIA_1
 $Comp
-L Retro-PC-rescue:74HC138-74xx IC3
+L 74xx:74HC138 IC3
 U 1 1 5DA01AB5
 P 3750 10000
@@
 F 2 "Package_DIP:DIP-40_W15.24mm_LongPads" H 8700 2650 50  0001 C CNN
 F 3 "https://www.westerndesigncenter.com/wdc/documentation/w65c22s.pdf" H 8700 2650 50  0001 C CNN
+F 4 "Western Design Center" H 8700 2650 50  0001 C CNN "Mfr."
+F 5 "W65C22N6TPG-14" H 8700 2650 50  0001 C CNN "Mfr. No."
+F 6 "955-W65C22N6TPG-14" H 8700 2650 50  0001 C CNN "Mouser"
 	1    8700 2650
 	1    0    0    -1
@@
 F 1 "10k" H 2470 3905 50  0000 L CNN
 F 2 "Resistor_THT:R_Axial_DIN0207_L6.3mm_D2.5mm_P7.62mm_Horizontal" V 2330 3950 50  0001 C CNN
-F 3 "https://www.mouser.de/datasheet/2/427/sfr16s25-239894.pdf" H 2400 3950 50  0001 C CNN
-F 4 "Vishay / BC Components" H 2400 3950 50  0001 C CNN "Mfr."
-F 5 "SFR25H0001002JR500" H 2400 3950 50  0001 C CNN "Mfr. No."
-F 6 "594-SFR25H0001002JR5" H 2400 3950 50  0001 C CNN "Mouser"
+F 3 "https://www.mouser.de/datasheet/2/447/Yageo%20LR_MFP_2013-594635.pdf" H 2400 3950 50  0001 C CNN
+F 4 "Yageo" H 2400 3950 50  0001 C CNN "Mfr."
+F 5 "MFP-25BRD52-10K" H 2400 3950 50  0001 C CNN "Mfr. No."
+F 6 "603-MFP-25BRD52-10K" H 2400 3950 50  0001 C CNN "Mouser"
 	1    2400 3950
 	-1   0    0    1

Commit message: Replace LCD
Parts:
- IC3: symbol 74xx:74HC138 -> Retro-PC-rescue:74HC138-74xx
- IC5: value AS6C62256A -> RAM
Changed lines of the file:
@@
 AR Path="/5EB09E21/5EBEAF84" Ref="IC5"  Part="1"
 F 0 "IC5" H 8500 6650 50  0000 C CNN
-F 1 "AS6C62256A" H 8650 6550 50  0000 C CNN
+F 1 "RAM" H 8650 6550 50  0000 C CNN
 F 2 "Package_DIP:DIP-28_W15.24mm_LongPads" H 8950 5700 50  0001 C CNN
 F 3 "https://www.alliancememory.com/wp-content/uploads/pdf/AS6C62256A.pdf" H 8950 5700 50  0001 C CNN
@@
 ~CS_VIA_1
 $Comp
-L 74xx:74HC138 IC3
+L Retro-PC-rescue:74HC138-74xx IC3
 U 1 1 5DA01AB5
 P 3750 10000
