File: hardware/Processor.sch (KiCad schematic (older format))
At the start: 22 parts, among them IC1 74HC138, IC2 W65C02, IC3 74HC00, IC4 SYSTEM ROM, IC5 W65C22, IC6 RAM, IC7 W65C22, IC8 W65C51, SW4 CLOCK INPUT, X5 EXT. CLOCK

Commit message: Update project
Parts:
- C1, C2, C3, C4, C5, C6, C7, C8: symbol Mainboard-rescue:C-Device -> Device:C
- IC1: symbol Mainboard-rescue:74HC138-Logic -> Logic:74HC138
- IC2: symbol Mainboard-rescue:W65C02-Western_Design_Center -> Western_Design_Center:W65C02
- IC3: symbol Mainboard-rescue:74HC00-74xx -> 74xx:74HC00
- IC4: symbol Mainboard-rescue:28C256-Memory_EEPROM -> Memory_EEPROM:28C256
- IC5, IC7: symbol Mainboard-rescue:W65C22-Western_Design_Center -> Western_Design_Center:W65C22
- IC6: symbol Mainboard-rescue:AS6C62256A-Alliance_Memory -> Alliance_Memory:AS6C62256A
- IC8: symbol Mainboard-rescue:W65C51-Western_Design_Center -> Western_Design_Center:W65C51
- R4, R5: symbol Mainboard-rescue:R-Device -> Device:R
- SW4: symbol Mainboard-rescue:SW_SPDT-Switch -> Switch:SW_SPDT
- X5: symbol Mainboard-rescue:Conn_01x02-Connector_Generic -> Connector_Generic:Conn_01x02
- XTAL1: symbol Mainboard-rescue:ECS-100X-ECS -> ECS:ECS-100X
- XTAL2: symbol Mainboard-rescue:Crystal-Device -> Device:Crystal
Other:
- note added: "- WDC recommends to use an oscillator for system time base instead of PHI1O and \nPHI2O, because the clock delay of PHI1O and PHI2O to PHI2 is no longer tested."
- note added: "Info"
Changed lines of the file:
@@
 Sheet 4 7
 Title "Processor system"
-Date "2021-05-10"
+Date "2020-10-11"
 Rev "1.0"
 Comp "https://www.kampis-elektroecke.de"
@@
 	4150 6500 4250 6400
 $Comp
-L Mainboard-rescue:GND-power #PWR?
+L power:GND #PWR?
 U 1 1 5EBEAFC0
 P 5200 6700
@@
 	6200 6500 6100 6400
 $Comp
-L Mainboard-rescue:C-Device C?
+L Device:C C?
 U 1 1 5EBEAFEE
 P 5350 3750
@@
 $EndComp
 $Comp
-L Mainboard-rescue:+5V-power #PWR?
+L power:+5V #PWR?
 U 1 1 5EBEAFF4
 P 5200 3525
@@
 $EndComp
 $Comp
-L Mainboard-rescue:GND-power #PWR?
+L power:GND #PWR?
 U 1 1 5EBEAFFA
 P 5350 3950
@@
 	4500 4300 4650 4300
 $Comp
-L Mainboard-rescue:+5V-power #PWR?
+L power:+5V #PWR?
 U 1 1 5F0A0D76
 P 13400 5325
@@
 $EndComp
 $Comp
-L Mainboard-rescue:C-Device C?
+L Device:C C?
 U 1 1 5F0A0D7C
 P 13550 5575
@@
 $EndComp
 $Comp
-L Mainboard-rescue:GND-power #PWR?
+L power:GND #PWR?
 U 1 1 5F0A0D82
 P 13550 5750
@@
 Connection ~ 13400 5375
 $Comp
-L Mainboard-rescue:GND-power #PWR?
+L power:GND #PWR?
 U 1 1 5F114440
 P 13400 8300
@@
 $EndComp
 $Comp
-L Mainboard-rescue:Crystal-Device XTAL2
+L Device:Crystal XTAL2
 U 1 1 5F163710
 P 14550 6150
@@
 	14550 6350 14550 6300
 $Comp
-L Mainboard-rescue:C-Device C?
+L Device:C C?
 U 1 1 5F17EFA5
 P 15250 6150
@@
 $EndComp
 $Comp
-L Mainboard-rescue:GND-power #PWR?
+L power:GND #PWR?
 U 1 1 5F17FE85
 P 15250 6350
@@
 Connection ~ 14550 5950
 $Comp
-L Mainboard-rescue:R-Device R?
+L Device:R R?
 U 1 1 5F1A8FA3
 P 14300 6150
@@
 	13400 1300 13550 1300
 $Comp
-L Mainboard-rescue:GND-power #PWR?
+L power:GND #PWR?
 U 1 1 5EBEB073
 P 13550 1700
@@
 $EndComp
 $Comp
-L Mainboard-rescue:C-Device C?
+L Device:C C?
 U 1 1 5EBEB06D
 P 13550 1500
@@
 $EndComp
 $Comp
-L Mainboard-rescue:+5V-power #PWR?
+L power:+5V #PWR?
 U 1 1 5EBEB067
 P 13400 1200
@@
 	11650 3450 12800 3450
 $Comp
-L Mainboard-rescue:GND-power #PWR?
+L power:GND #PWR?
 U 1 1 5EBEB024
 P 13400 4450
@@
 	13400 4350 13400 4450
 $Comp
-L Mainboard-rescue:W65C22-Western_Design_Center IC?
+L Western_Design_Center:W65C22 IC?
 U 1 1 5EBEAF7E
 P 13400 3100
@@
 	10350 4200 10350 4250
 $Comp
-L Mainboard-rescue:GND-power #PWR?
+L power:GND #PWR?
 U 1 1 5EBEB04C
 P 10500 4650
@@
 $EndComp
 $Comp
-L Mainboard-rescue:C-Device C?
+L Device:C C?
 U 1 1 5EBEB046
 P 10500 4450
@@
 $EndComp
 $Comp
-L Mainboard-rescue:+5V-power #PWR?
+L power:+5V #PWR?
 U 1 1 5EBEB040
 P 10350 4200
@@
 	10350 6700 10350 6600
 $Comp
-L Mainboard-rescue:GND-power #PWR?
+L power:GND #PWR?
 U 1 1 5EBEB01C
 P 10350 6700
@@
 $EndComp
 $Comp
-L Mainboard-rescue:AS6C62256A-Alliance_Memory IC?
+L Alliance_Memory:AS6C62256A IC?
 U 1 1 5EBEAF84
 P 10350 5700
@@
 Connection ~ 7150 7100
 $Comp
-L Mainboard-rescue:+5V-power #PWR?
+L power:+5V #PWR?
 U 1 1 5EBEB229
 P 7500 6200
@@
 	8400 4600 8650 4600
 $Comp
-L Mainboard-rescue:+5V-power #PWR?
+L power:+5V #PWR?
 U 1 1 5EBEB095
 P 6375 4875
@@
 $EndComp
 $Comp
-L Mainboard-rescue:+5V-power #PWR?
+L power:+5V #PWR?
 U 1 1 5EBEB02A
 P 8000 4200
@@
 $EndComp
 $Comp
-L Mainboard-rescue:GND-power #PWR?
+L power:GND #PWR?
 U 1 1 5EBEB016
 P 8000 6700
@@
 D0
 $Comp
-L Mainboard-rescue:W65C51-Western_Design_Center IC8
+L Western_Design_Center:W65C51 IC8
 U 1 1 5F08EFF6
 P 13400 7050
@@
 	11650 7250 11550 7150
 $Comp
-L Mainboard-rescue:74HC00-74xx IC3
+L 74xx:74HC00 IC3
 U 5 2 5DD62749
 P 10600 10200
-AR Path="/5DD62749" Ref="IC3"  Part="5"
-AR Path="/5EB09E21/5DD62749" Ref="IC3"  Part="5"
 F 0 "IC3" H 10658 10246 50  0000 L CNN
 F 1 "74HC00" H 10658 10155 50  0000 L CNN
@@
 $EndComp
 $Comp
-L Mainboard-rescue:C-Device C?
+L Device:C C?
 U 1 1 5DD67E33
 P 11200 10200
@@
 $EndComp
 $Comp
-L Mainboard-rescue:GND-power #PWR?
+L power:GND #PWR?
 U 1 1 5DD67E39
 P 11200 10725
@@
 $EndComp
 $Comp
-L Mainboard-rescue:+5V-power #PWR?
+L power:+5V #PWR?
 U 1 1 5DD7BAB1
 P 10600 9600
@@
 $EndComp
 $Comp
-L Mainboard-rescue:GND-power #PWR?
+L power:GND #PWR?
 U 1 1 5DD90602
 P 10600 10750
@@
 	8000 6600 8000 6700
 $Comp
-L Mainboard-rescue:GND-power #PWR?
+L power:GND #PWR?
 U 1 1 5DF4A850
 P 11250 6700
@@
 	5750 4800 5800 4800
 $Comp
-L Mainboard-rescue:W65C22-Western_Design_Center IC5
+L Western_Design_Center:W65C22 IC5
 U 1 1 5DA8CE2C
 P 10100 2650
@@
 	10100 850  10250 850
 $Comp
-L Mainboard-rescue:GND-power #PWR?
+L power:GND #PWR?
 U 1 1 5DA90421
 P 10250 1250
@@
 $EndComp
 $Comp
-L Mainboard-rescue:C-Device C?
+L Device:C C?
 U 1 1 5DA9042A
 P 10250 1050
@@
 $EndComp
 $Comp
-L Mainboard-rescue:+5V-power #PWR?
+L power:+5V #PWR?
 U 1 1 5DA90430
 P 10100 750
@@
 NoConn ~ 10700 1700
 $Comp
-L Mainboard-rescue:28C256-Memory_EEPROM IC?
+L Memory_EEPROM:28C256 IC?
 U 1 1 5EBEAFAB
 P 8000 5500
@@
 ~IRQ_CPU
 $Comp
-L Mainboard-rescue:R-Device R?
+L Device:R R?
 U 1 1 5EBEB08E
 P 6175 4875
@@
 NoConn ~ 5750 4400
 $Comp
-L Mainboard-rescue:W65C02-Western_Design_Center IC?
+L Western_Design_Center:W65C02 IC?
 U 1 1 5EBEAF78
 P 5200 5350
@@
 	4500 4700 4650 4700
 $Comp
-L Mainboard-rescue:+5V-power #PWR?
+L power:+5V #PWR?
 U 1 1 5DECCA6F
 P 5875 5250
@@
 	7475 6400 7600 6400
 $Comp
-L Mainboard-rescue:GND-power #PWR?
+L power:GND #PWR?
 U 1 1 5DEBFFC7
 P 7300 6700
@@
 	12700 2650 12800 2650
 $Comp
-L Mainboard-rescue:+5V-power #PWR?
+L power:+5V #PWR?
 U 1 1 5E1808C3
 P 12700 2650
@@
 	9400 2200 9500 2200
 $Comp
-L Mainboard-rescue:+5V-power #PWR?
+L power:+5V #PWR?
 U 1 1 5E1E7B71
 P 9400 2200
@@
 	12750 6750 12850 6750
 $Comp
-L Mainboard-rescue:+5V-power #PWR?
+L power:+5V #PWR?
 U 1 1 5E20A942
 P 12750 6750
@@
 	10100 4050 10100 3900
 $Comp
-L Mainboard-rescue:GND-power #PWR?
+L power:GND #PWR?
 U 1 1 5DAAA0A4
 P 10100 4050
@@
 	11525 1600 11450 1600
 $Comp
-L Mainboard-rescue:Conn_01x02-Connector_Generic X5
+L Connector_Generic:Conn_01x02 X5
 U 1 1 5E26AB5F
 P 700 900
@@
 	900  900  1125 900
 $Comp
-L Mainboard-rescue:GND-power #PWR?
+L power:GND #PWR?
 U 1 1 5DCE2807
 P 1125 1200
@@
 	1125 1000 1125 1200
 $Comp
-L Mainboard-rescue:SW_SPDT-Switch SW?
+L Switch:SW_SPDT SW?
 U 1 1 5E027064
 P 4650 1450
@@
 Clock
 $Comp
-L Mainboard-rescue:GND-power #PWR?
+L power:GND #PWR?
 U 1 1 5EBEB298
 P 2750 2150
@@
 $EndComp
 $Comp
-L Mainboard-rescue:+5V-power #PWR?
+L power:+5V #PWR?
 U 1 1 5EBEB292
 P 2750 800
@@
 	2750 1150 2750 800
 $Comp
-L Mainboard-rescue:ECS-100X-ECS XTAL?
+L ECS:ECS-100X XTAL?
 U 1 1 5EBEB282
 P 2750 1450
@@
 	5150 10700 5150 10750
 $Comp
-L Mainboard-rescue:C-Device C?
+L Device:C C?
 U 1 1 5DA77F99
 P 5300 9150
@@
 $EndComp
 $Comp
-L Mainboard-rescue:GND-power #PWR?
+L power:GND #PWR?
 U 1 1 5DA30F54
 P 5300 9350
@@
 	5150 8950 5300 8950
 $Comp
-L Mainboard-rescue:GND-power #PWR?
+L power:GND #PWR?
 U 1 1 5DA30F4B
 P 5150 10750
@@
 	5150 8950 5150 8900
 $Comp
-L Mainboard-rescue:+5V-power #PWR?
+L power:+5V #PWR?
 U 1 1 5DA30F43
 P 5150 8900
@@
 $EndComp
 $Comp
-L Mainboard-rescue:74HC138-Logic IC?
+L Logic:74HC138 IC?
 U 1 1 5DA01AB5
 P 5150 10000
@@
 	4150 8200 4250 8300
 $Comp
-L Mainboard-rescue:74HC00-74xx IC3
+L 74xx:74HC00 IC3
 U 3 1 5DE5C7B0
 P 5450 8200
-AR Path="/5DE5C7B0" Ref="IC3"  Part="3"
-AR Path="/5EB09E21/5DE5C7B0" Ref="IC3"  Part="3"
 F 0 "IC3" H 5450 8525 50  0000 C CNN
 F 1 "74HC00" H 5450 8434 50  0000 C CNN
@@
 	4150 8000 4250 8100
 $Comp
-L Mainboard-rescue:74HC00-74xx IC3
+L 74xx:74HC00 IC3
 U 2 1 5DE275DC
 P 8500 7550
-AR Path="/5DE275DC" Ref="IC3"  Part="2"
-AR Path="/5EB09E21/5DE275DC" Ref="IC3"  Part="2"
 F 0 "IC3" H 8500 7875 50  0000 C CNN
 F 1 "74HC00" H 8500 7784 50  0000 C CNN
@@
 $EndComp
 $Comp
-L Mainboard-rescue:74HC00-74xx IC3
+L 74xx:74HC00 IC3
 U 1 1 5DE24ADF
 P 5450 7650
-AR Path="/5DE24ADF" Ref="IC3"  Part="1"
-AR Path="/5EB09E21/5DE24ADF" Ref="IC3"  Part="1"
 F 0 "IC3" H 5450 7975 50  0000 C CNN
 F 1 "74HC00" H 5450 7884 50  0000 C CNN
@@
 Wire Bus Line
 	4150 7075 4150 7100
+Text Notes 11900 9200 0    100  ~ 20
+Info
+Wire Notes Line
+	11850 9000 11850 9900
+Wire Notes Line
+	16000 9000 11850 9000
+Wire Notes Line
+	16000 9900 16000 9000
+Wire Notes Line
+	11850 9900 16000 9900
+Text Notes 11950 9400 0    50   ~ 0
+- WDC recommends to use an oscillator for system time base instead of PHI1O and \nPHI2O, because the clock delay of PHI1O and PHI2O to PHI2 is no longer tested.
 Wire Bus Line
 	11300 1500 11300 3350

Commit message: Initialize branch
Parts:
- C1, C2, C3, C4, C5, C6, C7, C8: symbol Device:C -> Mainboard-rescue:C-Device
- IC1: symbol Logic:74HC138 -> Mainboard-rescue:74HC138-Logic
- IC2: symbol Western_Design_Center:W65C02 -> Mainboard-rescue:W65C02-Western_Design_Center
- IC3: symbol 74xx:74HC00 -> Mainboard-rescue:74HC00-74xx
- IC4: symbol Memory_EEPROM:28C256 -> Mainboard-rescue:28C256-Memory_EEPROM
- IC5, IC7: symbol Western_Design_Center:W65C22 -> Mainboard-rescue:W65C22-Western_Design_Center
- IC6: symbol Alliance_Memory:AS6C62256A -> Mainboard-rescue:AS6C62256A-Alliance_Memory
- IC8: symbol Western_Design_Center:W65C51 -> Mainboard-rescue:W65C51-Western_Design_Center
- R4, R5: symbol Device:R -> Mainboard-rescue:R-Device
- SW4: symbol Switch:SW_SPDT -> Mainboard-rescue:SW_SPDT-Switch
- X5: symbol Connector_Generic:Conn_01x02 -> Mainboard-rescue:Conn_01x02-Connector_Generic
- XTAL1: symbol ECS:ECS-100X -> Mainboard-rescue:ECS-100X-ECS
- XTAL2: symbol Device:Crystal -> Mainboard-rescue:Crystal-Device
Other:
- note removed: "- WDC recommends to use an oscillator for system time base instead of PHI1O and \nPHI2O, because the clock delay of PHI1O and PHI2O to PHI2 is no longer tested."
- note removed: "Info"
Changed lines of the file:
@@
 Sheet 4 7
 Title "Processor system"
-Date "2020-10-11"
+Date "2021-05-10"
 Rev "1.0"
 Comp "https://www.kampis-elektroecke.de"
@@
 	4150 6500 4250 6400
 $Comp
-L power:GND #PWR?
+L Mainboard-rescue:GND-power #PWR?
 U 1 1 5EBEAFC0
 P 5200 6700
@@
 	6200 6500 6100 6400
 $Comp
-L Device:C C?
+L Mainboard-rescue:C-Device C?
 U 1 1 5EBEAFEE
 P 5350 3750
@@
 $EndComp
 $Comp
-L power:+5V #PWR?
+L Mainboard-rescue:+5V-power #PWR?
 U 1 1 5EBEAFF4
 P 5200 3525
@@
 $EndComp
 $Comp
-L power:GND #PWR?
+L Mainboard-rescue:GND-power #PWR?
 U 1 1 5EBEAFFA
 P 5350 3950
@@
 	4500 4300 4650 4300
 $Comp
-L power:+5V #PWR?
+L Mainboard-rescue:+5V-power #PWR?
 U 1 1 5F0A0D76
 P 13400 5325
@@
 $EndComp
 $Comp
-L Device:C C?
+L Mainboard-rescue:C-Device C?
 U 1 1 5F0A0D7C
 P 13550 5575
@@
 $EndComp
 $Comp
-L power:GND #PWR?
+L Mainboard-rescue:GND-power #PWR?
 U 1 1 5F0A0D82
 P 13550 5750
@@
 Connection ~ 13400 5375
 $Comp
-L power:GND #PWR?
+L Mainboard-rescue:GND-power #PWR?
 U 1 1 5F114440
 P 13400 8300
@@
 $EndComp
 $Comp
-L Device:Crystal XTAL2
+L Mainboard-rescue:Crystal-Device XTAL2
 U 1 1 5F163710
 P 14550 6150
@@
 	14550 6350 14550 6300
 $Comp
-L Device:C C?
+L Mainboard-rescue:C-Device C?
 U 1 1 5F17EFA5
 P 15250 6150
@@
 $EndComp
 $Comp
-L power:GND #PWR?
+L Mainboard-rescue:GND-power #PWR?
 U 1 1 5F17FE85
 P 15250 6350
@@
 Connection ~ 14550 5950
 $Comp
-L Device:R R?
+L Mainboard-rescue:R-Device R?
 U 1 1 5F1A8FA3
 P 14300 6150
@@
 	13400 1300 13550 1300
 $Comp
-L power:GND #PWR?
+L Mainboard-rescue:GND-power #PWR?
 U 1 1 5EBEB073
 P 13550 1700
@@
 $EndComp
 $Comp
-L Device:C C?
+L Mainboard-rescue:C-Device C?
 U 1 1 5EBEB06D
 P 13550 1500
@@
 $EndComp
 $Comp
-L power:+5V #PWR?
+L Mainboard-rescue:+5V-power #PWR?
 U 1 1 5EBEB067
 P 13400 1200
@@
 	11650 3450 12800 3450
 $Comp
-L power:GND #PWR?
+L Mainboard-rescue:GND-power #PWR?
 U 1 1 5EBEB024
 P 13400 4450
@@
 	13400 4350 13400 4450
 $Comp
-L Western_Design_Center:W65C22 IC?
+L Mainboard-rescue:W65C22-Western_Design_Center IC?
 U 1 1 5EBEAF7E
 P 13400 3100
@@
 	10350 4200 10350 4250
 $Comp
-L power:GND #PWR?
+L Mainboard-rescue:GND-power #PWR?
 U 1 1 5EBEB04C
 P 10500 4650
@@
 $EndComp
 $Comp
-L Device:C C?
+L Mainboard-rescue:C-Device C?
 U 1 1 5EBEB046
 P 10500 4450
@@
 $EndComp
 $Comp
-L power:+5V #PWR?
+L Mainboard-rescue:+5V-power #PWR?
 U 1 1 5EBEB040
 P 10350 4200
@@
 	10350 6700 10350 6600
 $Comp
-L power:GND #PWR?
+L Mainboard-rescue:GND-power #PWR?
 U 1 1 5EBEB01C
 P 10350 6700
@@
 $EndComp
 $Comp
-L Alliance_Memory:AS6C62256A IC?
+L Mainboard-rescue:AS6C62256A-Alliance_Memory IC?
 U 1 1 5EBEAF84
 P 10350 5700
@@
 Connection ~ 7150 7100
 $Comp
-L power:+5V #PWR?
+L Mainboard-rescue:+5V-power #PWR?
 U 1 1 5EBEB229
 P 7500 6200
@@
 	8400 4600 8650 4600
 $Comp
-L power:+5V #PWR?
+L Mainboard-rescue:+5V-power #PWR?
 U 1 1 5EBEB095
 P 6375 4875
@@
 $EndComp
 $Comp
-L power:+5V #PWR?
+L Mainboard-rescue:+5V-power #PWR?
 U 1 1 5EBEB02A
 P 8000 4200
@@
 $EndComp
 $Comp
-L power:GND #PWR?
+L Mainboard-rescue:GND-power #PWR?
 U 1 1 5EBEB016
 P 8000 6700
@@
 D0
 $Comp
-L Western_Design_Center:W65C51 IC8
+L Mainboard-rescue:W65C51-Western_Design_Center IC8
 U 1 1 5F08EFF6
 P 13400 7050
@@
 	11650 7250 11550 7150
 $Comp
-L 74xx:74HC00 IC3
+L Mainboard-rescue:74HC00-74xx IC3
 U 5 2 5DD62749
 P 10600 10200
+AR Path="/5DD62749" Ref="IC3"  Part="5"
+AR Path="/5EB09E21/5DD62749" Ref="IC3"  Part="5"
 F 0 "IC3" H 10658 10246 50  0000 L CNN
 F 1 "74HC00" H 10658 10155 50  0000 L CNN
@@
 $EndComp
 $Comp
-L Device:C C?
+L Mainboard-rescue:C-Device C?
 U 1 1 5DD67E33
 P 11200 10200
@@
 $EndComp
 $Comp
-L power:GND #PWR?
+L Mainboard-rescue:GND-power #PWR?
 U 1 1 5DD67E39
 P 11200 10725
@@
 $EndComp
 $Comp
-L power:+5V #PWR?
+L Mainboard-rescue:+5V-power #PWR?
 U 1 1 5DD7BAB1
 P 10600 9600
@@
 $EndComp
 $Comp
-L power:GND #PWR?
+L Mainboard-rescue:GND-power #PWR?
 U 1 1 5DD90602
 P 10600 10750
@@
 	8000 6600 8000 6700
 $Comp
-L power:GND #PWR?
+L Mainboard-rescue:GND-power #PWR?
 U 1 1 5DF4A850
 P 11250 6700
@@
 	5750 4800 5800 4800
 $Comp
-L Western_Design_Center:W65C22 IC5
+L Mainboard-rescue:W65C22-Western_Design_Center IC5
 U 1 1 5DA8CE2C
 P 10100 2650
@@
 	10100 850  10250 850
 $Comp
-L power:GND #PWR?
+L Mainboard-rescue:GND-power #PWR?
 U 1 1 5DA90421
 P 10250 1250
@@
 $EndComp
 $Comp
-L Device:C C?
+L Mainboard-rescue:C-Device C?
 U 1 1 5DA9042A
 P 10250 1050
@@
 $EndComp
 $Comp
-L power:+5V #PWR?
+L Mainboard-rescue:+5V-power #PWR?
 U 1 1 5DA90430
 P 10100 750
@@
 NoConn ~ 10700 1700
 $Comp
-L Memory_EEPROM:28C256 IC?
+L Mainboard-rescue:28C256-Memory_EEPROM IC?
 U 1 1 5EBEAFAB
 P 8000 5500
@@
 ~IRQ_CPU
 $Comp
-L Device:R R?
+L Mainboard-rescue:R-Device R?
 U 1 1 5EBEB08E
 P 6175 4875
@@
 NoConn ~ 5750 4400
 $Comp
-L Western_Design_Center:W65C02 IC?
+L Mainboard-rescue:W65C02-Western_Design_Center IC?
 U 1 1 5EBEAF78
 P 5200 5350
@@
 	4500 4700 4650 4700
 $Comp
-L power:+5V #PWR?
+L Mainboard-rescue:+5V-power #PWR?
 U 1 1 5DECCA6F
 P 5875 5250
@@
 	7475 6400 7600 6400
 $Comp
-L power:GND #PWR?
+L Mainboard-rescue:GND-power #PWR?
 U 1 1 5DEBFFC7
 P 7300 6700
@@
 	12700 2650 12800 2650
 $Comp
-L power:+5V #PWR?
+L Mainboard-rescue:+5V-power #PWR?
 U 1 1 5E1808C3
 P 12700 2650
@@
 	9400 2200 9500 2200
 $Comp
-L power:+5V #PWR?
+L Mainboard-rescue:+5V-power #PWR?
 U 1 1 5E1E7B71
 P 9400 2200
@@
 	12750 6750 12850 6750
 $Comp
-L power:+5V #PWR?
+L Mainboard-rescue:+5V-power #PWR?
 U 1 1 5E20A942
 P 12750 6750
@@
 	10100 4050 10100 3900
 $Comp
-L power:GND #PWR?
+L Mainboard-rescue:GND-power #PWR?
 U 1 1 5DAAA0A4
 P 10100 4050
@@
 	11525 1600 11450 1600
 $Comp
-L Connector_Generic:Conn_01x02 X5
+L Mainboard-rescue:Conn_01x02-Connector_Generic X5
 U 1 1 5E26AB5F
 P 700 900
@@
 	900  900  1125 900
 $Comp
-L power:GND #PWR?
+L Mainboard-rescue:GND-power #PWR?
 U 1 1 5DCE2807
 P 1125 1200
@@
 	1125 1000 1125 1200
 $Comp
-L Switch:SW_SPDT SW?
+L Mainboard-rescue:SW_SPDT-Switch SW?
 U 1 1 5E027064
 P 4650 1450
@@
 Clock
 $Comp
-L power:GND #PWR?
+L Mainboard-rescue:GND-power #PWR?
 U 1 1 5EBEB298
 P 2750 2150
@@
 $EndComp
 $Comp
-L power:+5V #PWR?
+L Mainboard-rescue:+5V-power #PWR?
 U 1 1 5EBEB292
 P 2750 800
@@
 	2750 1150 2750 800
 $Comp
-L ECS:ECS-100X XTAL?
+L Mainboard-rescue:ECS-100X-ECS XTAL?
 U 1 1 5EBEB282
 P 2750 1450
@@
 	5150 10700 5150 10750
 $Comp
-L Device:C C?
+L Mainboard-rescue:C-Device C?
 U 1 1 5DA77F99
 P 5300 9150
@@
 $EndComp
 $Comp
-L power:GND #PWR?
+L Mainboard-rescue:GND-power #PWR?
 U 1 1 5DA30F54
 P 5300 9350
@@
 	5150 8950 5300 8950
 $Comp
-L power:GND #PWR?
+L Mainboard-rescue:GND-power #PWR?
 U 1 1 5DA30F4B
 P 5150 10750
@@
 	5150 8950 5150 8900
 $Comp
-L power:+5V #PWR?
+L Mainboard-rescue:+5V-power #PWR?
 U 1 1 5DA30F43
 P 5150 8900
@@
 $EndComp
 $Comp
-L Logic:74HC138 IC?
+L Mainboard-rescue:74HC138-Logic IC?
 U 1 1 5DA01AB5
 P 5150 10000
@@
 	4150 8200 4250 8300
 $Comp
-L 74xx:74HC00 IC3
+L Mainboard-rescue:74HC00-74xx IC3
 U 3 1 5DE5C7B0
 P 5450 8200
+AR Path="/5DE5C7B0" Ref="IC3"  Part="3"
+AR Path="/5EB09E21/5DE5C7B0" Ref="IC3"  Part="3"
 F 0 "IC3" H 5450 8525 50  0000 C CNN
 F 1 "74HC00" H 5450 8434 50  0000 C CNN
@@
 	4150 8000 4250 8100
 $Comp
-L 74xx:74HC00 IC3
+L Mainboard-rescue:74HC00-74xx IC3
 U 2 1 5DE275DC
 P 8500 7550
+AR Path="/5DE275DC" Ref="IC3"  Part="2"
+AR Path="/5EB09E21/5DE275DC" Ref="IC3"  Part="2"
 F 0 "IC3" H 8500 7875 50  0000 C CNN
 F 1 "74HC00" H 8500 7784 50  0000 C CNN
@@
 $EndComp
 $Comp
-L 74xx:74HC00 IC3
+L Mainboard-rescue:74HC00-74xx IC3
 U 1 1 5DE24ADF
 P 5450 7650
+AR Path="/5DE24ADF" Ref="IC3"  Part="1"
+AR Path="/5EB09E21/5DE24ADF" Ref="IC3"  Part="1"
 F 0 "IC3" H 5450 7975 50  0000 C CNN
 F 1 "74HC00" H 5450 7884 50  0000 C CNN
@@
 Wire Bus Line
 	4150 7075 4150 7100
-Text Notes 11900 9200 0    100  ~ 20
-Info
-Wire Notes Line
-	11850 9000 11850 9900
-Wire Notes Line
-	16000 9000 11850 9000
-Wire Notes Line
-	16000 9900 16000 9000
-Wire Notes Line
-	11850 9900 16000 9900
-Text Notes 11950 9400 0    50   ~ 0
-- WDC recommends to use an oscillator for system time base instead of PHI1O and \nPHI2O, because the clock delay of PHI1O and PHI2O to PHI2 is no longer tested.
 Wire Bus Line
 	11300 1500 11300 3350
