File: hardware/Retro PC.kicad_pcb (KiCad board)
At the start: 2 copper layers, 160 x 100 mm, 57 parts, among them IC1 74HC00, IC2 W65C02, IC3 74HC138, IC4 28C256, IC5 AS6C62256A, IC6 W65C22, IC7 W65C51, IC8 TL7702B, IC9 FT232RL, J1 Power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

Commit message: Working on layout
Parts:
- removed J3: Input, Connector_PinHeader_2.54mm:PinHeader_2x06_P2.54mm_Vertical
- removed J4: Output, Connector_PinHeader_2.54mm:PinHeader_2x06_P2.54mm_Vertical
- removed R2: 10k, Resistor_THT:R_Axial_DIN0207_L6.3mm_D2.5mm_P7.62mm_Horizontal
- added C17: 100nF, Capacitor_THT:C_Rect_L4.6mm_W2.0mm_P2.50mm_MKS02_FKP02, F.Cu at (130.8, 55.5)
- added D13: POWER, LED_THT:LED_D5.0mm, F.Cu at (71.1, 67.4)
- added R8: 470, Resistor_THT:R_Axial_DIN0207_L6.3mm_D2.5mm_P7.62mm_Horizontal, F.Cu at (78.3, 63.2)
- added R9: 10k, Resistor_THT:R_Axial_DIN0207_L6.3mm_D2.5mm_P7.62mm_Horizontal, F.Cu at (123.2, 52.2)
- added REF**: MountingHole_3.2mm_M3_Pad_Via, MountingHole:MountingHole_3.2mm_M3_Pad_Via, F.Cu at (223.2, 134.6)
- added REF**: MountingHole_3.2mm_M3_Pad_Via, MountingHole:MountingHole_3.2mm_M3_Pad_Via, F.Cu at (223.2, 44.6)
- added REF**: MountingHole_3.2mm_M3_Pad_Via, MountingHole:MountingHole_3.2mm_M3_Pad_Via, F.Cu at (73.2, 44.6)
- added REF**: MountingHole_3.2mm_M3_Pad_Via, MountingHole:MountingHole_3.2mm_M3_Pad_Via, F.Cu at (73.2, 134.6)
- added SW4: ~NMI, Button_Switch_THT:SW_PUSH_6mm_H4.3mm, F.Cu at (124.3, 44.1)
- D0: value LED -> LED0
- D1: value LED -> LED1
- D11: value Tx -> TX
- D12: value Rx -> RX
- D2: value LED -> LED2
- D3: value LED -> LED3
- D4: value LED -> LED4
- D5: value LED -> LED5
- D6: value LED -> LED6
- D7: value LED -> LED7
- D8, D9: value D_Schottky -> SD103A
- IC4: value 28C256 -> SYSTEM ROM; footprint Socket:DIP_Socket-28_W11.9_W12.7_W15.24_W17.78_W18.5_3M_228-1277-00-0602J -> Package_DIP:DIP-28_W15.24mm_LongPads
- IC8: value TL7702B -> TL7702
- J1: value Power -> 12V
- J2: value USB_A -> SERIAL
- XTAL1: value ECS-100X -> 1MHz
- moved SW1 46.1 mm to (110.5, 44.0), turned to 0 degrees
- moved C8 42.5 mm to (204.4, 159.0)
- moved XTAL2 42.5 mm to (209.4, 159.1)
- moved R4 42.5 mm to (215.5, 153.9)
- moved C11 32.5 mm to (117.0, 55.5), turned to 180 degrees
- moved C14 27.2 mm to (243.0, 116.4), turned to 0 degrees
- moved D11 26.5 mm to (200.9, 135.6)
- moved R6 23.7 mm to (200.9, 131.9)
- moved R5 23.0 mm to (109.4, 52.1), turned to 0 degrees
- moved D12 21.9 mm to (204.1, 135.6)
- moved R7 18.4 mm to (204.1, 131.9)
- moved R3 16.7 mm to (178.9, 101.2), turned to 90 degrees
- moved C15 16.2 mm to (224.0, 123.8), turned to 90 degrees
- moved U1 11.4 mm to (84.0, 47.0)
- moved C10 11.4 mm to (94.1, 47.0)
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Connections:
- net /IO/RDY renamed /Processor/RDY
- D11 pad 2: Net-(D11-Pad2) -> +5V
- D12 pad 2: Net-(D12-Pad2) -> +5V
- D9 pad 1: /IO/~IRQ -> /Processor/~IRQ
- IC2 pad 1: /IO/VPB -> /Processor/VPB
- IC2 pad 36: /IO/BE -> /Processor/BE
- IC2 pad 7: /IO/SYNC -> /Processor/SYNC
- IC7 pad 11: /IO/ACIAReady -> /Processor/ACIAReady
- IC9 pad 22: Net-(D12-Pad1) -> Net-(IC9-Pad22)
- IC9 pad 23: Net-(D11-Pad1) -> Net-(IC9-Pad23)
- R6 pad 1: +5V -> Net-(D11-Pad1)
- R6 pad 2: Net-(D11-Pad2) -> Net-(IC9-Pad23)
- R7 pad 1: +5V -> Net-(D12-Pad1)
- R7 pad 2: Net-(D12-Pad2) -> Net-(IC9-Pad22)
Routing:
- net /Processor/~RESET: track 248.7 -> 126.1 mm, vias 7 -> 5
- net /IO/VPB: track 115.6 -> 0.00 mm, vias 3 -> 0
- net /IO/SYNC: track 101.0 -> 0.00 mm, vias 1 -> 0
- net /IO/ACIAReady: track 79.4 -> 0.00 mm, vias 2 -> 0
- net /IO/~IRQ: track 53.2 -> 0.00 mm, vias 4 -> 0
- net /IO/BE: track 51.3 -> 0.00 mm, vias 2 -> 0
- net /Processor/RDY: track 59.4 -> 9.83 mm, vias 1 -> 0
- net /Processor/ModemReady: track 49.4 -> 0.00 mm, vias 3 -> 0
- net /IO/~NMI: track 59.3 -> 10.1 mm, vias 3 -> 0
- net /USB/D-: track 21.9 -> 0.00 mm
- net /USB/D+: track 21.2 -> 0.00 mm
- net /USB/CTS: track 19.7 -> 0.00 mm, vias 1 -> 0
- net Net-(C14-Pad2): track 13.8 -> 0.00 mm, vias 2 -> 0
- net +5V: track 50.2 -> 37.0 mm
- net /USB/RxD: track 12.7 -> 0.00 mm, vias 2 -> 0
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Other:
- outline, holes or cut-outs redrawn
- rule trace_min: 0.2 -> 0.09
- rule via_min_drill: 0.3 -> 0.2
- rule via_min_size: 0.4 -> 0.45

Commit message: Working on Schematic
Parts:
- removed the REF** at (223.2, 44.6)
- added C18: 100nF, Capacitor_THT:C_Rect_L4.0mm_W2.5mm_P2.50mm, F.Cu at (258.4, 205.0)
- added C19: 100nF, Capacitor_THT:C_Rect_L4.0mm_W2.5mm_P2.50mm, F.Cu at (258.4, 120.2)
- added IC10: W65C22, Package_DIP:DIP-40_W15.24mm_LongPads, F.Cu at (116.7, 186.0)
- added IC11: LCD-016N002L, Display:LCD-016N002L, F.Cu at (147.7, 156.6)
- added RV1: 10k, Potentiometer_THT:Potentiometer_Vishay_T73YP_Vertical, F.Cu at (203.5, 193.9)
- C1, C10, C11, C12, C13, C17, C2, C3, C4, C5, C6, C7, C8: footprint Capacitor_THT:C_Rect_L4.6mm_W2.0mm_P2.50mm_MKS02_FKP02 -> Capacitor_THT:C_Rect_L4.0mm_W2.5mm_P2.50mm
- moved REF** 60.0 mm to (223.2, 194.6)
- moved REF** 60.0 mm to (73.2, 194.6)
- moved IC7 51.3 mm to (212.6, 151.8), turned to 180 degrees
- moved J2 45.5 mm to (256.5, 136.8)
- moved R4 45.5 mm to (261.0, 155.5)
- moved C15 45.5 mm to (269.5, 125.4)
- moved C16 45.5 mm to (257.3, 122.8)
- moved C8 45.5 mm to (249.8, 160.5)
- moved D12 45.5 mm to (249.6, 137.2)
- moved R7 45.5 mm to (249.6, 133.4)
- moved XTAL2 45.5 mm to (254.9, 160.6)
- moved IC9 45.5 mm to (263.3, 124.1)
- moved D11 44.3 mm to (245.1, 137.9)
- moved R6 44.3 mm to (245.1, 134.2)
- moved D8 30.3 mm to (144.0, 80.1), turned to 270 degrees
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Connections:
- D9 pad 1: /Processor/~IRQ -> (no net)
- IC2 pad 1: /Processor/VPB -> (no net)
- IC2 pad 3: Net-(IC2-Pad3) -> (no net)
- IC2 pad 35: Net-(IC2-Pad35) -> (no net)
- IC2 pad 36: /Processor/BE -> (no net)
- IC2 pad 38: Net-(IC2-Pad38) -> (no net)
- IC2 pad 39: Net-(IC2-Pad39) -> (no net)
- IC2 pad 5: Net-(IC2-Pad5) -> (no net)
- IC2 pad 7: /Processor/SYNC -> (no net)
- IC3 pad 10: Net-(IC3-Pad10) -> (no net)
- IC3 pad 11: Net-(IC3-Pad11) -> (no net)
- IC3 pad 12: Net-(IC3-Pad12) -> (no net)
- IC3 pad 14: Net-(IC3-Pad14) -> /Processor/~CS_VIA_2
- IC3 pad 7: Net-(IC3-Pad7) -> (no net)
- IC3 pad 9: Net-(IC3-Pad9) -> (no net)
- IC6 pad 39: Net-(IC6-Pad39) -> (no net)
- IC6 pad 40: Net-(IC6-Pad40) -> (no net)
- IC7 pad 11: /Processor/ACIAReady -> (no net)
- IC7 pad 5: Net-(IC7-Pad5) -> (no net)
- IC8 pad 6: Net-(IC8-Pad6) -> (no net)
- IC9 pad 10: Net-(IC9-Pad10) -> (no net)
- IC9 pad 12: Net-(IC9-Pad12) -> (no net)
- IC9 pad 13: Net-(IC9-Pad13) -> (no net)
- IC9 pad 14: Net-(IC9-Pad14) -> (no net)
- IC9 pad 26: Net-(IC9-Pad26) -> (no net)
- IC9 pad 27: Net-(IC9-Pad27) -> (no net)
- IC9 pad 28: Net-(IC9-Pad28) -> (no net)
- IC9 pad 6: Net-(IC9-Pad6) -> (no net)
- IC9 pad 9: Net-(IC9-Pad9) -> (no net)
- XTAL1 pad 1: Net-(XTAL1-Pad1) -> (no net)
Routing:
- net /Processor/~RESET: track 126.1 -> 0.00 mm, vias 5 -> 0
- net /Processor/A1: track 241.4 -> 176.5 mm, vias 6 -> 3
- net /Processor/A0: track 244.5 -> 184.2 mm, vias 5 -> 3
- net /Processor/~CS_VIA_1: track 98.1 -> 39.7 mm, vias 5 -> 4
- net /Processor/A2: track 196.8 -> 142.3 mm, vias 6 -> 3
- net /Processor/A3: track 197.1 -> 143.0 mm, vias 3 -> 2
- net /Processor/~IRQ_ACIA: track 53.0 -> 24.0 mm
- net /Processor/R~W: track 133.8 -> 120.8 mm
- net /Processor/~IRQ_VIA_1: track 11.5 -> 0.00 mm
- net /Processor/D0: track 227.0 -> 217.2 mm
- net /Processor/1MHz: track 108.9 -> 100.3 mm
- net /Processor/D1: track 221.7 -> 214.4 mm
- net /Processor/D6: track 213.6 -> 206.9 mm
- net /Processor/D4: track 210.7 -> 204.0 mm
- net /Processor/D5: track 212.1 -> 205.5 mm
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Other:
- board size 160 x 100 mm -> 160 x 160 mm

Commit message: Working on layout
Parts:
- added D14: SD103A, Diode_THT:D_DO-35_SOD27_P7.62mm_Horizontal, F.Cu at (115.4, 71.2)
- J2: footprint Connector_USB:USB_Micro-B_Wuerth_629105150521 -> Connector_USB:USB_B_TE_5787834_Vertical
- moved R4 66.6 mm to (196.0, 141.0)
- moved C8 66.6 mm to (184.8, 146.1)
- moved XTAL2 66.6 mm to (189.9, 146.1)
- moved C15 59.7 mm to (223.5, 163.5)
- moved C16 59.7 mm to (211.3, 160.9)
- moved D11 59.7 mm to (199.1, 176.0)
- moved D12 59.7 mm to (203.6, 175.3)
- moved J2 59.7 mm to (210.5, 174.9)
- moved R6 59.7 mm to (199.1, 172.3)
- moved R7 59.7 mm to (203.6, 171.5)
- moved C14 59.7 mm to (197.0, 154.5)
- moved C19 59.7 mm to (212.5, 158.3)
- moved IC9 59.7 mm to (217.4, 162.2)
- moved C6 51.7 mm to (215.0, 145.0)
- moved IC7 38.4 mm to (177.7, 135.8), turned to 90 degrees
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Connections:
- net /Processor/1MHz renamed /IO/1MHz
- net /Processor/A0 renamed /IO/A0
- net /Processor/A1 renamed /IO/A1
- net /Processor/A10 renamed /IO/A10
- net /Processor/A11 renamed /IO/A11
- net /Processor/A12 renamed /IO/A12
- net /Processor/A13 renamed /IO/A13
- net /Processor/A14 renamed /IO/A14
- net /Processor/A15 renamed /IO/A15
- net /Processor/A2 renamed /IO/A2
- net /Processor/A3 renamed /IO/A3
- net /Processor/A4 renamed /IO/A4
- net /Processor/A5 renamed /IO/A5
- net /Processor/A6 renamed /IO/A6
- net /Processor/A7 renamed /IO/A7
- net /Processor/A8 renamed /IO/A8
- net /Processor/A9 renamed /IO/A9
- net /Processor/D0 renamed /IO/D0
- net /Processor/D1 renamed /IO/D1
- net /Processor/D2 renamed /IO/D2
- net /Processor/D3 renamed /IO/D3
- net /Processor/D4 renamed /IO/D4
- net /Processor/D5 renamed /IO/D5
- net /Processor/D6 renamed /IO/D6
- net /Processor/D7 renamed /IO/D7
- net /Processor/R~W renamed /IO/R~W
- net /Processor/~RESET renamed /IO/~RESET
- D9 pad 1: (no net) -> /Processor/~IRQ
- IC10 pad 10: (no net) -> Net-(IC10-Pad10)
- IC10 pad 11: (no net) -> Net-(IC10-Pad11)
- IC10 pad 12: (no net) -> Net-(IC10-Pad12)
- IC10 pad 13: (no net) -> Net-(IC10-Pad13)
- IC10 pad 14: (no net) -> Net-(IC10-Pad14)
- IC10 pad 15: (no net) -> Net-(IC10-Pad15)
- IC10 pad 16: (no net) -> Net-(IC10-Pad16)
- IC10 pad 17: (no net) -> Net-(IC10-Pad17)
- IC10 pad 18: (no net) -> Net-(IC10-Pad18)
- IC10 pad 19: (no net) -> Net-(IC10-Pad19)
- IC10 pad 2: (no net) -> Net-(IC10-Pad2)
- IC10 pad 21: (no net) -> /Processor/~IRQ_VIA_2
- IC10 pad 3: (no net) -> Net-(IC10-Pad3)
- IC10 pad 39: (no net) -> Net-(IC10-Pad39)
- IC10 pad 4: (no net) -> Net-(IC10-Pad4)
- IC10 pad 40: (no net) -> Net-(IC10-Pad40)
- IC10 pad 5: (no net) -> Net-(IC10-Pad5)
- IC10 pad 6: (no net) -> Net-(IC10-Pad6)
- IC10 pad 7: (no net) -> Net-(IC10-Pad7)
- IC10 pad 8: (no net) -> Net-(IC10-Pad8)
- IC10 pad 9: (no net) -> Net-(IC10-Pad9)
- IC11 pad 10: (no net) -> Net-(IC11-Pad10)
- IC11 pad 11: (no net) -> Net-(IC11-Pad11)
- IC11 pad 12: (no net) -> Net-(IC11-Pad12)
- IC11 pad 13: (no net) -> Net-(IC11-Pad13)
- IC11 pad 14: (no net) -> Net-(IC11-Pad14)
- IC11 pad 4: (no net) -> Net-(IC11-Pad4)
- IC11 pad 5: (no net) -> Net-(IC11-Pad5)
- IC11 pad 6: (no net) -> Net-(IC11-Pad6)
- IC11 pad 7: (no net) -> Net-(IC11-Pad7)
- IC11 pad 8: (no net) -> Net-(IC11-Pad8)
- IC11 pad 9: (no net) -> Net-(IC11-Pad9)
- IC11 pad A1: (no net) -> Net-(IC11-PadA1)
- IC11 pad A2: (no net) -> Net-(IC11-PadA2)
- IC11 pad K1: (no net) -> Net-(IC11-PadK1)
- IC11 pad K2: (no net) -> Net-(IC11-PadK2)
- IC2 pad 1: (no net) -> /Processor/VPB
- IC2 pad 3: (no net) -> Net-(IC2-Pad3)
- IC2 pad 35: (no net) -> Net-(IC2-Pad35)
- IC2 pad 36: (no net) -> /Processor/BE
- IC2 pad 38: (no net) -> Net-(IC2-Pad38)
- IC2 pad 39: (no net) -> Net-(IC2-Pad39)
- IC2 pad 5: (no net) -> Net-(IC2-Pad5)
- IC2 pad 7: (no net) -> /Processor/SYNC
- IC3 pad 10: (no net) -> Net-(IC3-Pad10)
- IC3 pad 11: (no net) -> Net-(IC3-Pad11)
- IC3 pad 12: (no net) -> Net-(IC3-Pad12)
- IC3 pad 7: (no net) -> Net-(IC3-Pad7)
- IC3 pad 9: (no net) -> Net-(IC3-Pad9)
- IC6 pad 39: (no net) -> Net-(IC6-Pad39)
- IC6 pad 40: (no net) -> Net-(IC6-Pad40)
- IC7 pad 11: (no net) -> /Processor/ACIAReady
- IC7 pad 5: (no net) -> Net-(IC7-Pad5)
- IC8 pad 6: (no net) -> Net-(IC8-Pad6)
- IC9 pad 10: (no net) -> Net-(IC9-Pad10)
- IC9 pad 12: (no net) -> Net-(IC9-Pad12)
- IC9 pad 13: (no net) -> Net-(IC9-Pad13)
- IC9 pad 14: (no net) -> Net-(IC9-Pad14)
- IC9 pad 26: (no net) -> Net-(IC9-Pad26)
- IC9 pad 27: (no net) -> Net-(IC9-Pad27)
- IC9 pad 28: (no net) -> Net-(IC9-Pad28)
- IC9 pad 6: (no net) -> Net-(IC9-Pad6)
- IC9 pad 9: (no net) -> Net-(IC9-Pad9)
- RV1 pad 3: (no net) -> Net-(RV1-Pad3)
- XTAL1 pad 1: (no net) -> Net-(XTAL1-Pad1)
Routing:
- net /IO/~RESET: track 0.00 -> 189.6 mm, vias 0 -> 5
- net /IO/A1: track 176.5 -> 346.2 mm, vias 3 -> 6
- net /IO/A0: track 184.2 -> 342.6 mm, vias 3 -> 6
- net /IO/D0: track 217.2 -> 372.3 mm, vias 1 -> 11
- net /IO/A3: track 143.0 -> 294.0 mm, vias 2 -> 4
- net /IO/A2: track 142.3 -> 291.9 mm, vias 3 -> 5
- net /IO/D1: track 214.4 -> 361.7 mm, vias 1 -> 11
- net /IO/D2: track 211.2 -> 352.6 mm, vias 1 -> 11
- net /IO/D3: track 199.3 -> 335.2 mm, vias 3 -> 13
- net /IO/D4: track 204.0 -> 334.6 mm, vias 3 -> 13
- net /IO/D5: track 205.5 -> 330.9 mm, vias 3 -> 13
- net /IO/D6: track 206.9 -> 327.4 mm, vias 3 -> 13
- net /IO/D7: track 208.4 -> 323.7 mm, vias 2 -> 12
- net /Processor/~CS_VIA_2: track 0.00 -> 76.0 mm, vias 0 -> 4
- net /Processor/~CS_VIA_1: track 39.7 -> 101.2 mm, vias 4 -> 3
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
Commit message: Working on layout
Parts:
- added J3: Conn_02x20_Odd_Even, Connector_PinHeader_2.54mm:PinHeader_2x20_P2.54mm_Horizontal, F.Cu at (221.1, 72.3)
- J1: footprint Connector_BarrelJack:BarrelJack_Wuerth_6941xx301002 -> Wuerth:BarrelJack_Wuerth_6941xx301002
- J2: footprint Connector_USB:USB_B_TE_5787834_Vertical -> TE_Connectivity:USB_B_TE_2923042_Horizontal
- moved C19 53.4 mm to (159.4, 164.3)
- moved D11 38.3 mm to (222.9, 145.9), turned to 0 degrees
- moved D12 33.2 mm to (222.9, 148.2), turned to 0 degrees
- moved R6 33.1 mm to (219.1, 145.9), turned to 180 degrees
- moved C6 28.3 mm to (210.7, 117.0), turned to 180 degrees
- moved R7 28.0 mm to (219.1, 148.2), turned to 180 degrees
- moved J2 18.9 mm to (220.2, 158.7), turned to 90 degrees
- moved C15 18.2 mm to (209.3, 152.1), turned to 180 degrees
- moved C14 17.0 mm to (214.0, 153.6), turned to 180 degrees
- moved IC9 9.75 mm to (208.0, 159.5), turned to 90 degrees
- moved C16 6.60 mm to (206.7, 165.5), turned to 0 degrees
- moved C8 0.56 mm to (184.3, 146.2)
- moved XTAL2 0.10 mm to (189.9, 146.2)
Connections:
- D9 pad 1: /Processor/~IRQ -> (no net)
- IC10 pad 10: Net-(IC10-Pad10) -> (no net)
- IC10 pad 11: Net-(IC10-Pad11) -> (no net)
- IC10 pad 12: Net-(IC10-Pad12) -> (no net)
- IC10 pad 13: Net-(IC10-Pad13) -> (no net)
- IC10 pad 14: Net-(IC10-Pad14) -> (no net)
- IC10 pad 15: Net-(IC10-Pad15) -> (no net)
- IC10 pad 16: Net-(IC10-Pad16) -> (no net)
- IC10 pad 17: Net-(IC10-Pad17) -> (no net)
- IC10 pad 18: Net-(IC10-Pad18) -> (no net)
- IC10 pad 19: Net-(IC10-Pad19) -> (no net)
- IC10 pad 2: Net-(IC10-Pad2) -> (no net)
- IC10 pad 21: /Processor/~IRQ_VIA_2 -> (no net)
- IC10 pad 3: Net-(IC10-Pad3) -> (no net)
- IC10 pad 39: Net-(IC10-Pad39) -> (no net)
- IC10 pad 4: Net-(IC10-Pad4) -> (no net)
- IC10 pad 40: Net-(IC10-Pad40) -> (no net)
- IC10 pad 5: Net-(IC10-Pad5) -> (no net)
- IC10 pad 6: Net-(IC10-Pad6) -> (no net)
- IC10 pad 7: Net-(IC10-Pad7) -> (no net)
- IC10 pad 8: Net-(IC10-Pad8) -> (no net)
- IC10 pad 9: Net-(IC10-Pad9) -> (no net)
- IC11 pad 10: Net-(IC11-Pad10) -> (no net)
- IC11 pad 11: Net-(IC11-Pad11) -> (no net)
- IC11 pad 12: Net-(IC11-Pad12) -> (no net)
- IC11 pad 13: Net-(IC11-Pad13) -> (no net)
- IC11 pad 14: Net-(IC11-Pad14) -> (no net)
- IC11 pad 4: Net-(IC11-Pad4) -> (no net)
- IC11 pad 5: Net-(IC11-Pad5) -> (no net)
- IC11 pad 6: Net-(IC11-Pad6) -> (no net)
- IC11 pad 7: Net-(IC11-Pad7) -> (no net)
- IC11 pad 8: Net-(IC11-Pad8) -> (no net)
- IC11 pad 9: Net-(IC11-Pad9) -> (no net)
- IC11 pad A1: Net-(IC11-PadA1) -> (no net)
- IC11 pad A2: Net-(IC11-PadA2) -> (no net)
- IC11 pad K1: Net-(IC11-PadK1) -> (no net)
- IC11 pad K2: Net-(IC11-PadK2) -> (no net)
- IC2 pad 1: /Processor/VPB -> (no net)
- IC2 pad 3: Net-(IC2-Pad3) -> (no net)
- IC2 pad 35: Net-(IC2-Pad35) -> (no net)
- IC2 pad 36: /Processor/BE -> (no net)
- IC2 pad 38: Net-(IC2-Pad38) -> (no net)
- IC2 pad 39: Net-(IC2-Pad39) -> (no net)
- IC2 pad 5: Net-(IC2-Pad5) -> (no net)
- IC2 pad 7: /Processor/SYNC -> (no net)
- IC3 pad 10: Net-(IC3-Pad10) -> (no net)
- IC3 pad 11: Net-(IC3-Pad11) -> (no net)
- IC3 pad 12: Net-(IC3-Pad12) -> (no net)
- IC3 pad 7: Net-(IC3-Pad7) -> (no net)
- IC3 pad 9: Net-(IC3-Pad9) -> (no net)
- IC6 pad 39: Net-(IC6-Pad39) -> (no net)
- IC6 pad 40: Net-(IC6-Pad40) -> (no net)
- IC7 pad 11: /Processor/ACIAReady -> (no net)
- IC7 pad 5: Net-(IC7-Pad5) -> (no net)
- IC8 pad 6: Net-(IC8-Pad6) -> (no net)
- IC9 pad 10: Net-(IC9-Pad10) -> (no net)
- IC9 pad 12: Net-(IC9-Pad12) -> (no net)
- IC9 pad 13: Net-(IC9-Pad13) -> (no net)
- IC9 pad 14: Net-(IC9-Pad14) -> (no net)
- IC9 pad 26: Net-(IC9-Pad26) -> (no net)
- IC9 pad 27: Net-(IC9-Pad27) -> (no net)
- IC9 pad 28: Net-(IC9-Pad28) -> (no net)
- IC9 pad 6: Net-(IC9-Pad6) -> (no net)
- IC9 pad 9: Net-(IC9-Pad9) -> (no net)
- RV1 pad 3: Net-(RV1-Pad3) -> (no net)
- XTAL1 pad 1: Net-(XTAL1-Pad1) -> (no net)
Routing:
- net /IO/~RESET: track 189.6 -> 356.8 mm, vias 5 -> 8
- net /Processor/ModemReady: track 0.00 -> 76.8 mm, vias 0 -> 4
- net /USB/CTS: track 0.00 -> 37.2 mm, vias 0 -> 4
- net /Processor/RxD: track 0.00 -> 33.6 mm
- net /Processor/CTS: track 0.00 -> 30.2 mm, vias 0 -> 2
- net /USB/RxD: track 0.00 -> 29.7 mm, vias 0 -> 2
- net Net-(IC9-Pad23): track 0.00 -> 20.3 mm
- net Net-(IC9-Pad22): track 0.00 -> 18.8 mm
- net GND: track 27.6 -> 42.4 mm, vias 2 -> 5
- net /USB/D-: track 0.00 -> 14.3 mm
- net /USB/D+: track 0.00 -> 14.3 mm
- net Net-(IC7-Pad7): track 5.65 -> 12.7 mm
- net Net-(C8-Pad1): track 10.9 -> 17.4 mm
- net +5V: track 33.8 -> 38.6 mm
- net Net-(C14-Pad2): track 0.00 -> 4.26 mm
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
Commit message: Working on layout
Parts:
- removed J2: SERIAL, TE_Connectivity:USB_B_TE_2923042_Horizontal
- added REF**: MountingHole_3.2mm_M3_Pad_Via, MountingHole:MountingHole_3.2mm_M3_Pad_Via, F.Cu at (223.2, 44.6)
- added X1: ConBarrel, Wuerth:BarrelJack_Wuerth_6941xx301002, F.Cu at (77.4, 55.5)
- J1: value 12V -> USB_B; footprint Wuerth:BarrelJack_Wuerth_6941xx301002 -> TE_Connectivity:USB_B_TE_2923042_Horizontal
- moved J1 176.3 mm to (220.2, 158.6), turned to 90 degrees
- moved D14 106.7 mm to (149.2, 172.4), turned to 0 degrees
- moved D9 31.7 mm to (153.8, 73.1), turned to 90 degrees
- moved D8 31.6 mm to (163.7, 81.0), turned to 90 degrees
- moved R1 29.6 mm to (159.5, 73.3), turned to 270 degrees
- moved R3 10.4 mm to (163.6, 94.4), turned to 0 degrees
- moved C2 0.52 mm to (156.0, 93.8), turned to 0 degrees
- moved J3 0.25 mm to (221.1, 72.6)
- moved IC10 0.13 mm to (96.3, 187.6)
Connections:
- D14 pad 1: /Processor/~IRQ_VIA_1 -> /Processor/~IRQ_VIA_2
- D9 pad 1: (no net) -> /Processor/~IRQ
- IC10 pad 10: (no net) -> Net-(IC10-Pad10)
- IC10 pad 11: (no net) -> Net-(IC10-Pad11)
- IC10 pad 12: (no net) -> Net-(IC10-Pad12)
- IC10 pad 13: (no net) -> Net-(IC10-Pad13)
- IC10 pad 14: (no net) -> Net-(IC10-Pad14)
- IC10 pad 15: (no net) -> Net-(IC10-Pad15)
- IC10 pad 16: (no net) -> Net-(IC10-Pad16)
- IC10 pad 17: (no net) -> Net-(IC10-Pad17)
- IC10 pad 18: (no net) -> Net-(IC10-Pad18)
- IC10 pad 19: (no net) -> Net-(IC10-Pad19)
- IC10 pad 2: (no net) -> Net-(IC10-Pad2)
- IC10 pad 21: (no net) -> /Processor/~IRQ_VIA_2
- IC10 pad 3: (no net) -> Net-(IC10-Pad3)
- IC10 pad 39: (no net) -> Net-(IC10-Pad39)
- IC10 pad 4: (no net) -> Net-(IC10-Pad4)
- IC10 pad 40: (no net) -> Net-(IC10-Pad40)
- IC10 pad 5: (no net) -> Net-(IC10-Pad5)
- IC10 pad 6: (no net) -> Net-(IC10-Pad6)
- IC10 pad 7: (no net) -> Net-(IC10-Pad7)
- IC10 pad 8: (no net) -> Net-(IC10-Pad8)
- IC10 pad 9: (no net) -> Net-(IC10-Pad9)
- IC11 pad 10: (no net) -> Net-(IC11-Pad10)
- IC11 pad 11: (no net) -> Net-(IC11-Pad11)
- IC11 pad 12: (no net) -> Net-(IC11-Pad12)
- IC11 pad 13: (no net) -> Net-(IC11-Pad13)
- IC11 pad 14: (no net) -> Net-(IC11-Pad14)
- IC11 pad 4: (no net) -> Net-(IC11-Pad4)
- IC11 pad 5: (no net) -> Net-(IC11-Pad5)
- IC11 pad 6: (no net) -> Net-(IC11-Pad6)
- IC11 pad 7: (no net) -> Net-(IC11-Pad7)
- IC11 pad 8: (no net) -> Net-(IC11-Pad8)
- IC11 pad 9: (no net) -> Net-(IC11-Pad9)
- IC11 pad A1: (no net) -> Net-(IC11-PadA1)
- IC11 pad A2: (no net) -> Net-(IC11-PadA2)
- IC11 pad K1: (no net) -> Net-(IC11-PadK1)
- IC11 pad K2: (no net) -> Net-(IC11-PadK2)
- IC2 pad 1: (no net) -> /Processor/VPB
- IC2 pad 3: (no net) -> Net-(IC2-Pad3)
- IC2 pad 35: (no net) -> Net-(IC2-Pad35)
- IC2 pad 36: (no net) -> /Processor/BE
- IC2 pad 38: (no net) -> Net-(IC2-Pad38)
- IC2 pad 39: (no net) -> Net-(IC2-Pad39)
- IC2 pad 5: (no net) -> Net-(IC2-Pad5)
- IC2 pad 7: (no net) -> /Processor/SYNC
- IC3 pad 10: (no net) -> Net-(IC3-Pad10)
- IC3 pad 11: (no net) -> Net-(IC3-Pad11)
- IC3 pad 12: (no net) -> Net-(IC3-Pad12)
- IC3 pad 7: (no net) -> Net-(IC3-Pad7)
- IC3 pad 9: (no net) -> Net-(IC3-Pad9)
- IC6 pad 39: (no net) -> Net-(IC6-Pad39)
- IC6 pad 40: (no net) -> Net-(IC6-Pad40)
- IC7 pad 11: (no net) -> /Processor/ACIAReady
- IC7 pad 5: (no net) -> Net-(IC7-Pad5)
- IC8 pad 6: (no net) -> Net-(IC8-Pad6)
- IC9 pad 10: (no net) -> Net-(IC9-Pad10)
- IC9 pad 12: (no net) -> Net-(IC9-Pad12)
- IC9 pad 13: (no net) -> Net-(IC9-Pad13)
- IC9 pad 14: (no net) -> Net-(IC9-Pad14)
- IC9 pad 26: (no net) -> Net-(IC9-Pad26)
- IC9 pad 27: (no net) -> Net-(IC9-Pad27)
- IC9 pad 28: (no net) -> Net-(IC9-Pad28)
- IC9 pad 6: (no net) -> Net-(IC9-Pad6)
- IC9 pad 9: (no net) -> Net-(IC9-Pad9)
- J1 pad 1: Net-(D10-Pad2) -> +5V
- J1 pad 2: GND -> /USB/D-
- J1 pad 3: (no net) -> /USB/D+
- J3 pad 24: (no net) -> Net-(J3-Pad24)
- J3 pad 26: (no net) -> Net-(J3-Pad26)
- J3 pad 28: (no net) -> Net-(J3-Pad28)
- J3 pad 30: (no net) -> Net-(J3-Pad30)
- J3 pad 32: (no net) -> Net-(J3-Pad32)
- J3 pad 33: (no net) -> Net-(J3-Pad33)
- J3 pad 34: (no net) -> Net-(J3-Pad34)
- J3 pad 35: (no net) -> Net-(J3-Pad35)
- J3 pad 36: (no net) -> Net-(J3-Pad36)
- J3 pad 37: (no net) -> Net-(J3-Pad37)
- J3 pad 38: (no net) -> Net-(J3-Pad38)
- RV1 pad 3: (no net) -> Net-(RV1-Pad3)
- XTAL1 pad 1: (no net) -> Net-(XTAL1-Pad1)
Routing:
- net /IO/A11: track 139.6 -> 254.8 mm, vias 4 -> 8
- net /IO/A10: track 135.0 -> 247.1 mm, vias 4 -> 7
- net /IO/A9: track 115.2 -> 225.5 mm, vias 3 -> 6
- net /IO/A8: track 119.2 -> 228.8 mm, vias 3 -> 6
- net /IO/A4: track 130.2 -> 237.5 mm, vias 1 -> 4
- net /IO/A5: track 129.3 -> 236.4 mm, vias 1 -> 4
- net /IO/A12: track 131.3 -> 237.8 mm, vias 2 -> 6
- net /IO/A6: track 128.1 -> 233.6 mm, vias 1 -> 4
- net /IO/A7: track 126.5 -> 230.9 mm, vias 1 -> 4
- net /IO/A14: track 142.1 -> 240.7 mm, vias 2 -> 6
- net /IO/A15: track 48.6 -> 143.7 mm, vias 2 -> 6
- net /IO/A13: track 161.1 -> 253.0 mm, vias 4 -> 8
- net /IO/~NMI: track 13.5 -> 85.3 mm, vias 0 -> 1
- net /IO/A0: track 343.1 -> 357.9 mm
- net /IO/A1: track 346.6 -> 358.7 mm, vias 6 -> 5
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