File: hardware/IO.sch (KiCad schematic (older format))
At the start: 15 parts, among them SW1 CARRIER, SW2 PORT B, SW3 INTERRUPT, X1 PORT B, X2 EXPANSION

Commit message: Update project
Parts:
- D1, D2, D3, D4, D5, D6, D7, D8: symbol Mainboard-rescue:LED-Device -> Device:LED
- RN1: symbol Mainboard-rescue:R_Network10-Device -> Device:R_Network10
- RN2: symbol Mainboard-rescue:R_Network08-Device -> Device:R_Network08
- SW1: symbol Mainboard-rescue:SW_SPDT-Switch -> Switch:SW_SPDT
- SW2: symbol Mainboard-rescue:SW_DIP_x08-Switch -> Switch:SW_DIP_x08
- SW3: symbol Mainboard-rescue:SW_DIP_x02-Switch -> Switch:SW_DIP_x02
- X1: symbol Mainboard-rescue:Conn_01x10-Connector_Generic -> Connector_Generic:Conn_01x10
- X2: symbol Mainboard-rescue:Conn_02x20_Odd_Even-Connector_Generic -> Connector_Generic:Conn_02x20_Odd_Even
Other:
- note added: "- The W65C22N I/O lines of PB have internal current limiting resistors."
- note added: "Info"
Changed lines of the file:
@@
 Sheet 2 7
 Title "I/O"
-Date "2021-05-10"
+Date "2020-10-11"
 Rev "1.0"
 Comp "https://www.kampis-elektroecke.de"
@@
 	1900 1650 1800 1550
 $Comp
-L Mainboard-rescue:LED-Device D?
+L Device:LED D?
 U 1 1 5ED5BEAF
 P 3600 4250
@@
 $EndComp
 $Comp
-L Mainboard-rescue:LED-Device D?
+L Device:LED D?
 U 1 1 5ED5BEB8
 P 3500 4250
@@
 $EndComp
 $Comp
-L Mainboard-rescue:LED-Device D?
+L Device:LED D?
 U 1 1 5ED5BEA6
 P 3700 4250
@@
 $EndComp
 $Comp
-L Mainboard-rescue:LED-Device D?
+L Device:LED D?
 U 1 1 5ED5BE9D
 P 3800 4250
@@
 $EndComp
 $Comp
-L Mainboard-rescue:LED-Device D?
+L Device:LED D?
 U 1 1 5ED5BE94
 P 3900 4250
@@
 $EndComp
 $Comp
-L Mainboard-rescue:LED-Device D?
+L Device:LED D?
 U 1 1 5ED5BE8B
 P 4000 4250
@@
 $EndComp
 $Comp
-L Mainboard-rescue:LED-Device D?
+L Device:LED D?
 U 1 1 5ED5BE82
 P 4100 4250
@@
 $EndComp
 $Comp
-L Mainboard-rescue:R_Network08-Device RN?
+L Device:R_Network08 RN?
 U 1 1 5ED5BED1
 P 3800 4650
@@
 $EndComp
 $Comp
-L Mainboard-rescue:LED-Device D?
+L Device:LED D?
 U 1 1 5ED5BE79
 P 4200 4250
@@
 $EndComp
 $Comp
-L Mainboard-rescue:GND-power #PWR?
+L power:GND #PWR?
 U 1 1 5DDAB6B1
 P 4200 4900
@@
 	4100 3450 4100 4100
 $Comp
-L Mainboard-rescue:SW_DIP_x02-Switch SW?
+L Switch:SW_DIP_x02 SW?
 U 1 1 5EE8631D
 P 3800 2500
@@
 $EndComp
 $Comp
-L Mainboard-rescue:SW_DIP_x08-Switch SW?
+L Switch:SW_DIP_x08 SW?
 U 1 1 5EE69B10
 P 3800 1850
@@
 D7
 $Comp
-L Mainboard-rescue:Conn_02x20_Odd_Even-Connector_Generic X2
+L Connector_Generic:Conn_02x20_Odd_Even X2
 U 1 1 5DBDED7E
 P 9950 2250
@@
 Wire Wire Line
 	10350 2150 10250 2150
+$Comp
+L power:GND #PWR?
+U 1 1 5DC0914B
+P 9650 3400
+AR Path="/5DC0914B" Ref="#PWR?"  Part="1"
+AR Path="/5EB09E21/5DC0914B" Ref="#PWR?"  Part="1"
+AR Path="/5EC67F7B/5DC0914B" Ref="#PWR06"  Part="1"
+F 0 "#PWR06" H 9650 3150 50  0001 C CNN
+F 1 "GND" H 9655 3227 50  0000 C CNN
+F 2 "" H 9650 3400 50  0001 C CNN
+F 3 "" H 9650 3400 50  0001 C CNN
+	1    9650 3400
+	1    0    0    -1
+$EndComp
 Wire Wire Line
 	9650 3400 9650 3250
@@
 	9750 3250 9650 3250
 $Comp
-L Mainboard-rescue:+5V-power #PWR?
+L power:+5V #PWR?
 U 1 1 5DC11208
 P 10450 3150
@@
 	1800 6300 1900 6300
 $Comp
-L Mainboard-rescue:+5V-power #PWR?
+L power:+5V #PWR?
 U 1 1 5E24E58E
 P 1900 6250
@@
 $EndComp
 $Comp
-L Mainboard-rescue:GND-power #PWR?
+L power:GND #PWR?
 U 1 1 5E24E594
 P 1900 6625
@@
 $EndComp
 $Comp
-L Mainboard-rescue:SW_SPDT-Switch SW1
+L Switch:SW_SPDT SW1
 U 1 1 5E24E59D
 P 1600 6400
@@
 	1400 6400 925  6400
 $Comp
-L Mainboard-rescue:GND-power #PWR?
+L power:GND #PWR?
 U 1 1 5E75385F
 P 4200 3100
@@
 Wire Wire Line
 	1900 1450 2550 1450
-$Comp
-L Mainboard-rescue:Conn_01x10-Connector_Generic X1
+Text Notes 7100 5850 0    50   ~ 0
+- The W65C22N I/O lines of PB have internal current limiting resistors.
+$Comp
+L Connector_Generic:Conn_01x10 X1
 U 1 1 5E73E8FD
 P 2750 2900
@@
 Wire Wire Line
 	2350 2400 3500 2400
+Wire Notes Line
+	7000 6450 11150 6450
+Wire Notes Line
+	11150 6450 11150 5550
+Wire Notes Line
+	11150 5550 7000 5550
+Wire Notes Line
+	7000 5550 7000 6450
+Text Notes 7050 5750 0    100  ~ 20
+Info
 Wire Wire Line
 	1900 2500 2450 2500
@@
 	2350 800  2350 950
 $Comp
-L Mainboard-rescue:+5V-power #PWR?
+L power:+5V #PWR?
 U 1 1 5FB069AF
 P 2350 800
@@
 $EndComp
 $Comp
-L Mainboard-rescue:R_Network10-Device RN?
+L Device:R_Network10 RN?
 U 1 1 5FB069BA
 P 2850 1150

Commit message: Initialize branch
Parts:
- D1, D2, D3, D4, D5, D6, D7, D8: symbol Device:LED -> Mainboard-rescue:LED-Device
- RN1: symbol Device:R_Network10 -> Mainboard-rescue:R_Network10-Device
- RN2: symbol Device:R_Network08 -> Mainboard-rescue:R_Network08-Device
- SW1: symbol Switch:SW_SPDT -> Mainboard-rescue:SW_SPDT-Switch
- SW2: symbol Switch:SW_DIP_x08 -> Mainboard-rescue:SW_DIP_x08-Switch
- SW3: symbol Switch:SW_DIP_x02 -> Mainboard-rescue:SW_DIP_x02-Switch
- X1: symbol Connector_Generic:Conn_01x10 -> Mainboard-rescue:Conn_01x10-Connector_Generic
- X2: symbol Connector_Generic:Conn_02x20_Odd_Even -> Mainboard-rescue:Conn_02x20_Odd_Even-Connector_Generic
Other:
- note removed: "- The W65C22N I/O lines of PB have internal current limiting resistors."
- note removed: "Info"
Changed lines of the file:
@@
 Sheet 2 7
 Title "I/O"
-Date "2020-10-11"
+Date "2021-05-10"
 Rev "1.0"
 Comp "https://www.kampis-elektroecke.de"
@@
 	1900 1650 1800 1550
 $Comp
-L Device:LED D?
+L Mainboard-rescue:LED-Device D?
 U 1 1 5ED5BEAF
 P 3600 4250
@@
 $EndComp
 $Comp
-L Device:LED D?
+L Mainboard-rescue:LED-Device D?
 U 1 1 5ED5BEB8
 P 3500 4250
@@
 $EndComp
 $Comp
-L Device:LED D?
+L Mainboard-rescue:LED-Device D?
 U 1 1 5ED5BEA6
 P 3700 4250
@@
 $EndComp
 $Comp
-L Device:LED D?
+L Mainboard-rescue:LED-Device D?
 U 1 1 5ED5BE9D
 P 3800 4250
@@
 $EndComp
 $Comp
-L Device:LED D?
+L Mainboard-rescue:LED-Device D?
 U 1 1 5ED5BE94
 P 3900 4250
@@
 $EndComp
 $Comp
-L Device:LED D?
+L Mainboard-rescue:LED-Device D?
 U 1 1 5ED5BE8B
 P 4000 4250
@@
 $EndComp
 $Comp
-L Device:LED D?
+L Mainboard-rescue:LED-Device D?
 U 1 1 5ED5BE82
 P 4100 4250
@@
 $EndComp
 $Comp
-L Device:R_Network08 RN?
+L Mainboard-rescue:R_Network08-Device RN?
 U 1 1 5ED5BED1
 P 3800 4650
@@
 $EndComp
 $Comp
-L Device:LED D?
+L Mainboard-rescue:LED-Device D?
 U 1 1 5ED5BE79
 P 4200 4250
@@
 $EndComp
 $Comp
-L power:GND #PWR?
+L Mainboard-rescue:GND-power #PWR?
 U 1 1 5DDAB6B1
 P 4200 4900
@@
 	4100 3450 4100 4100
 $Comp
-L Switch:SW_DIP_x02 SW?
+L Mainboard-rescue:SW_DIP_x02-Switch SW?
 U 1 1 5EE8631D
 P 3800 2500
@@
 $EndComp
 $Comp
-L Switch:SW_DIP_x08 SW?
+L Mainboard-rescue:SW_DIP_x08-Switch SW?
 U 1 1 5EE69B10
 P 3800 1850
@@
 D7
 $Comp
-L Connector_Generic:Conn_02x20_Odd_Even X2
+L Mainboard-rescue:Conn_02x20_Odd_Even-Connector_Generic X2
 U 1 1 5DBDED7E
 P 9950 2250
@@
 Wire Wire Line
 	10350 2150 10250 2150
-$Comp
-L power:GND #PWR?
-U 1 1 5DC0914B
-P 9650 3400
-AR Path="/5DC0914B" Ref="#PWR?"  Part="1"
-AR Path="/5EB09E21/5DC0914B" Ref="#PWR?"  Part="1"
-AR Path="/5EC67F7B/5DC0914B" Ref="#PWR06"  Part="1"
-F 0 "#PWR06" H 9650 3150 50  0001 C CNN
-F 1 "GND" H 9655 3227 50  0000 C CNN
-F 2 "" H 9650 3400 50  0001 C CNN
-F 3 "" H 9650 3400 50  0001 C CNN
-	1    9650 3400
-	1    0    0    -1
-$EndComp
 Wire Wire Line
 	9650 3400 9650 3250
@@
 	9750 3250 9650 3250
 $Comp
-L power:+5V #PWR?
+L Mainboard-rescue:+5V-power #PWR?
 U 1 1 5DC11208
 P 10450 3150
@@
 	1800 6300 1900 6300
 $Comp
-L power:+5V #PWR?
+L Mainboard-rescue:+5V-power #PWR?
 U 1 1 5E24E58E
 P 1900 6250
@@
 $EndComp
 $Comp
-L power:GND #PWR?
+L Mainboard-rescue:GND-power #PWR?
 U 1 1 5E24E594
 P 1900 6625
@@
 $EndComp
 $Comp
-L Switch:SW_SPDT SW1
+L Mainboard-rescue:SW_SPDT-Switch SW1
 U 1 1 5E24E59D
 P 1600 6400
@@
 	1400 6400 925  6400
 $Comp
-L power:GND #PWR?
+L Mainboard-rescue:GND-power #PWR?
 U 1 1 5E75385F
 P 4200 3100
@@
 Wire Wire Line
 	1900 1450 2550 1450
-Text Notes 7100 5850 0    50   ~ 0
-- The W65C22N I/O lines of PB have internal current limiting resistors.
-$Comp
-L Connector_Generic:Conn_01x10 X1
+$Comp
+L Mainboard-rescue:Conn_01x10-Connector_Generic X1
 U 1 1 5E73E8FD
 P 2750 2900
@@
 Wire Wire Line
 	2350 2400 3500 2400
-Wire Notes Line
-	7000 6450 11150 6450
-Wire Notes Line
-	11150 6450 11150 5550
-Wire Notes Line
-	11150 5550 7000 5550
-Wire Notes Line
-	7000 5550 7000 6450
-Text Notes 7050 5750 0    100  ~ 20
-Info
 Wire Wire Line
 	1900 2500 2450 2500
@@
 	2350 800  2350 950
 $Comp
-L power:+5V #PWR?
+L Mainboard-rescue:+5V-power #PWR?
 U 1 1 5FB069AF
 P 2350 800
@@
 $EndComp
 $Comp
-L Device:R_Network10 RN?
+L Mainboard-rescue:R_Network10-Device RN?
 U 1 1 5FB069BA
 P 2850 1150
