File: hardware/Supply.sch (KiCad schematic (older format))
At the start: 20 parts, among them IC11 TL7702A, SW6 FT232 RESET, SW7 RESET, U1 R-785.0-1.0, X7 GND, X8 DC IN

Commit message: Update project
Parts:
- C13, C14, C15, C16, C17, C18: symbol Mainboard-rescue:C-Device -> Device:C
- D11: symbol Mainboard-rescue:1N4148W-Diode -> Diode:1N4148W
- D12: symbol Mainboard-rescue:LED-Device -> Device:LED
- IC11: symbol Mainboard-rescue:TL7702B-Power_Supervisor -> Power_Supervisor:TL7702B
- R10, R11, R12, R13, R14, R15: symbol Mainboard-rescue:R-Device -> Device:R
- SW6, SW7: symbol Mainboard-rescue:SW_Push-Switch -> Switch:SW_Push
- U1: symbol Mainboard-rescue:R-785.0-1.0-Regulator_Switching -> Regulator_Switching:R-785.0-1.0
- X7: symbol Mainboard-rescue:Conn_01x01-Connector_Generic -> Connector_Generic:Conn_01x01
- X8: symbol Mainboard-rescue:ConBarrel-Wuerth -> Wuerth:ConBarrel
Changed lines of the file:
@@
 Sheet 7 7
 Title "Power Supply & Reset"
-Date "2021-05-10"
+Date "2020-10-11"
 Rev "1.0"
 Comp "https://www.kampis-elektroecke.de"
@@
 	2375 4600 2375 4650
 $Comp
-L Mainboard-rescue:GND-power #PWR?
+L power:GND #PWR?
 U 1 1 5E234E9F
 P 2375 4650
@@
 $EndComp
 $Comp
-L Mainboard-rescue:Conn_01x01-Connector_Generic X7
+L Connector_Generic:Conn_01x01 X7
 U 1 1 5E232D80
 P 2375 4400
@@
 	2725 5975 2925 5975
 $Comp
-L Mainboard-rescue:SW_Push-Switch SW?
+L Switch:SW_Push SW?
 U 1 1 5E27BBF0
 P 2725 6250
@@
 	3450 6400 3450 6500
 $Comp
-L Mainboard-rescue:GND-power #PWR?
+L power:GND #PWR?
 U 1 1 5E27BBE6
 P 3450 6500
@@
 $EndComp
 $Comp
-L Mainboard-rescue:C-Device C?
+L Device:C C?
 U 1 1 5E27BBE0
 P 3450 6250
@@
 	2725 5900 2725 5975
 $Comp
-L Mainboard-rescue:GND-power #PWR?
+L power:GND #PWR?
 U 1 1 5E27BBD2
 P 2725 6500
@@
 	2725 5575 2725 5600
 $Comp
-L Mainboard-rescue:+5V-power #PWR?
+L power:+5V #PWR?
 U 1 1 5E27BBCB
 P 2725 5575
@@
 $EndComp
 $Comp
-L Mainboard-rescue:R-Device R?
+L Device:R R?
 U 1 1 5E27BBC5
 P 2725 5750
@@
 	8050 3050 8050 3450
 $Comp
-L Mainboard-rescue:+5V-power #PWR?
+L power:+5V #PWR?
 U 1 1 5DC3430D
 P 8050 3050
@@
 $EndComp
 $Comp
-L Mainboard-rescue:R-Device R?
+L Device:R R?
 U 1 1 5DC34307
 P 8050 3600
@@
 $EndComp
 $Comp
-L Mainboard-rescue:ConBarrel-Wuerth X8
+L Wuerth:ConBarrel X8
 U 1 1 5DA7C8DA
 P 2400 3850
@@
 	4750 4650 4750 4500
 $Comp
-L Mainboard-rescue:GND-power #PWR?
+L power:GND #PWR?
 U 1 1 5D9EC35B
 P 4750 4650
@@
 	4750 4150 4750 4200
 $Comp
-L Mainboard-rescue:R-Device R?
+L Device:R R?
 U 1 1 5D9EA844
 P 4750 4000
@@
 $EndComp
 $Comp
-L Mainboard-rescue:LED-Device D?
+L Device:LED D?
 U 1 1 5D9EA3B0
 P 4750 4350
@@
 ~Reset
 $Comp
-L Mainboard-rescue:TL7702B-Power_Supervisor IC?
+L Power_Supervisor:TL7702B IC?
 U 1 1 5E9AA51D
 P 7300 4000
@@
 	7900 4650 7900 4550
 $Comp
-L Mainboard-rescue:GND-power #PWR?
+L power:GND #PWR?
 U 1 1 5E9AA50B
 P 7900 4650
@@
 $EndComp
 $Comp
-L Mainboard-rescue:C-Device C?
+L Device:C C?
 U 1 1 5E9AA505
 P 7900 4400
@@
 	6550 4550 6550 4650
 $Comp
-L Mainboard-rescue:GND-power #PWR?
+L power:GND #PWR?
 U 1 1 5E9AA4FC
 P 6550 4650
@@
 $EndComp
 $Comp
-L Mainboard-rescue:C-Device C?
+L Device:C C?
 U 1 1 5E9AA4F6
 P 6550 4400
@@
 	7300 4400 7300 4650
 $Comp
-L Mainboard-rescue:GND-power #PWR?
+L power:GND #PWR?
 U 1 1 5E9AA4EE
 P 7300 4650
@@
 $EndComp
 $Comp
-L Mainboard-rescue:+VDC-power #PWR?
+L power:+VDC #PWR?
 U 1 1 5E9AA4E8
 P 7300 3150
@@
 	3250 3150 3250 3750
 $Comp
-L Mainboard-rescue:+VDC-power #PWR?
+L power:+VDC #PWR?
 U 1 1 5E9AA4E1
 P 3250 3150
@@
 $EndComp
 $Comp
-L Mainboard-rescue:R-785.0-1.0-Regulator_Switching U?
+L Regulator_Switching:R-785.0-1.0 U?
 U 1 1 5E9AA4DB
 P 3750 3750
@@
 	2700 3950 2750 3950
 $Comp
-L Mainboard-rescue:GND-power #PWR?
+L power:GND #PWR?
 U 1 1 5E9AA4CF
 P 2750 4650
@@
 	3750 4050 3750 4650
 $Comp
-L Mainboard-rescue:GND-power #PWR?
+L power:GND #PWR?
 U 1 1 5E9AA4BF
 P 3750 4650
@@
 	3150 3750 3250 3750
 $Comp
-L Mainboard-rescue:1N4148W-Diode D?
+L Diode:1N4148W D?
 U 1 1 5E9AA4B5
 P 3000 3750
@@
 	3450 3750 3250 3750
 $Comp
-L Mainboard-rescue:+5V-power #PWR?
+L power:+5V #PWR?
 U 1 1 5E9AA4A9
 P 4200 3050
@@
 $EndComp
 $Comp
-L Mainboard-rescue:GND-power #PWR?
+L power:GND #PWR?
 U 1 1 5E9AA4A3
 P 4200 4650
@@
 $EndComp
 $Comp
-L Mainboard-rescue:GND-power #PWR?
+L power:GND #PWR?
 U 1 1 5E9AA49D
 P 3250 4650
@@
 $EndComp
 $Comp
-L Mainboard-rescue:C-Device C?
+L Device:C C?
 U 1 1 5E9AA497
 P 4200 4200
@@
 $EndComp
 $Comp
-L Mainboard-rescue:C-Device C?
+L Device:C C?
 U 1 1 5E9AA491
 P 3250 4200
@@
 	6100 4550 6100 4650
 $Comp
-L Mainboard-rescue:GND-power #PWR?
+L power:GND #PWR?
 U 1 1 5E9AA487
 P 6100 4650
@@
 	6100 4000 6100 4250
 $Comp
-L Mainboard-rescue:C-Device C?
+L Device:C C?
 U 1 1 5E9AA47C
 P 6100 4400
@@
 $EndComp
 $Comp
-L Mainboard-rescue:GND-power #PWR?
+L power:GND #PWR?
 U 1 1 5E9AA476
 P 5650 4650
@@
 	5650 3050 5650 3150
 $Comp
-L Mainboard-rescue:+5V-power #PWR?
+L power:+5V #PWR?
 U 1 1 5E9AA46F
 P 5650 3050
@@
 $EndComp
 $Comp
-L Mainboard-rescue:R-Device R?
+L Device:R R?
 U 1 1 5E9AA460
 P 5650 3300
@@
 Connection ~ 6100 4000
 $Comp
-L Mainboard-rescue:R-Device R?
+L Device:R R?
 U 1 1 5E74121A
 P 3075 5975
@@
 	5650 4450 5650 4650
 $Comp
-L Mainboard-rescue:SW_Push-Switch SW?
+L Switch:SW_Push SW?
 U 1 1 5E9AA469
 P 5650 4250
@@
 	5650 3600 6100 3600
 $Comp
-L Mainboard-rescue:R-Device R?
+L Device:R R?
 U 1 1 5E734C17
 P 5650 3850

Commit message: Initialize branch
Parts:
- C13, C14, C15, C16, C17, C18: symbol Device:C -> Mainboard-rescue:C-Device
- D11: symbol Diode:1N4148W -> Mainboard-rescue:1N4148W-Diode
- D12: symbol Device:LED -> Mainboard-rescue:LED-Device
- IC11: symbol Power_Supervisor:TL7702B -> Mainboard-rescue:TL7702B-Power_Supervisor
- R10, R11, R12, R13, R14, R15: symbol Device:R -> Mainboard-rescue:R-Device
- SW6, SW7: symbol Switch:SW_Push -> Mainboard-rescue:SW_Push-Switch
- U1: symbol Regulator_Switching:R-785.0-1.0 -> Mainboard-rescue:R-785.0-1.0-Regulator_Switching
- X7: symbol Connector_Generic:Conn_01x01 -> Mainboard-rescue:Conn_01x01-Connector_Generic
- X8: symbol Wuerth:ConBarrel -> Mainboard-rescue:ConBarrel-Wuerth
Changed lines of the file:
@@
 Sheet 7 7
 Title "Power Supply & Reset"
-Date "2020-10-11"
+Date "2021-05-10"
 Rev "1.0"
 Comp "https://www.kampis-elektroecke.de"
@@
 	2375 4600 2375 4650
 $Comp
-L power:GND #PWR?
+L Mainboard-rescue:GND-power #PWR?
 U 1 1 5E234E9F
 P 2375 4650
@@
 $EndComp
 $Comp
-L Connector_Generic:Conn_01x01 X7
+L Mainboard-rescue:Conn_01x01-Connector_Generic X7
 U 1 1 5E232D80
 P 2375 4400
@@
 	2725 5975 2925 5975
 $Comp
-L Switch:SW_Push SW?
+L Mainboard-rescue:SW_Push-Switch SW?
 U 1 1 5E27BBF0
 P 2725 6250
@@
 	3450 6400 3450 6500
 $Comp
-L power:GND #PWR?
+L Mainboard-rescue:GND-power #PWR?
 U 1 1 5E27BBE6
 P 3450 6500
@@
 $EndComp
 $Comp
-L Device:C C?
+L Mainboard-rescue:C-Device C?
 U 1 1 5E27BBE0
 P 3450 6250
@@
 	2725 5900 2725 5975
 $Comp
-L power:GND #PWR?
+L Mainboard-rescue:GND-power #PWR?
 U 1 1 5E27BBD2
 P 2725 6500
@@
 	2725 5575 2725 5600
 $Comp
-L power:+5V #PWR?
+L Mainboard-rescue:+5V-power #PWR?
 U 1 1 5E27BBCB
 P 2725 5575
@@
 $EndComp
 $Comp
-L Device:R R?
+L Mainboard-rescue:R-Device R?
 U 1 1 5E27BBC5
 P 2725 5750
@@
 	8050 3050 8050 3450
 $Comp
-L power:+5V #PWR?
+L Mainboard-rescue:+5V-power #PWR?
 U 1 1 5DC3430D
 P 8050 3050
@@
 $EndComp
 $Comp
-L Device:R R?
+L Mainboard-rescue:R-Device R?
 U 1 1 5DC34307
 P 8050 3600
@@
 $EndComp
 $Comp
-L Wuerth:ConBarrel X8
+L Mainboard-rescue:ConBarrel-Wuerth X8
 U 1 1 5DA7C8DA
 P 2400 3850
@@
 	4750 4650 4750 4500
 $Comp
-L power:GND #PWR?
+L Mainboard-rescue:GND-power #PWR?
 U 1 1 5D9EC35B
 P 4750 4650
@@
 	4750 4150 4750 4200
 $Comp
-L Device:R R?
+L Mainboard-rescue:R-Device R?
 U 1 1 5D9EA844
 P 4750 4000
@@
 $EndComp
 $Comp
-L Device:LED D?
+L Mainboard-rescue:LED-Device D?
 U 1 1 5D9EA3B0
 P 4750 4350
@@
 ~Reset
 $Comp
-L Power_Supervisor:TL7702B IC?
+L Mainboard-rescue:TL7702B-Power_Supervisor IC?
 U 1 1 5E9AA51D
 P 7300 4000
@@
 	7900 4650 7900 4550
 $Comp
-L power:GND #PWR?
+L Mainboard-rescue:GND-power #PWR?
 U 1 1 5E9AA50B
 P 7900 4650
@@
 $EndComp
 $Comp
-L Device:C C?
+L Mainboard-rescue:C-Device C?
 U 1 1 5E9AA505
 P 7900 4400
@@
 	6550 4550 6550 4650
 $Comp
-L power:GND #PWR?
+L Mainboard-rescue:GND-power #PWR?
 U 1 1 5E9AA4FC
 P 6550 4650
@@
 $EndComp
 $Comp
-L Device:C C?
+L Mainboard-rescue:C-Device C?
 U 1 1 5E9AA4F6
 P 6550 4400
@@
 	7300 4400 7300 4650
 $Comp
-L power:GND #PWR?
+L Mainboard-rescue:GND-power #PWR?
 U 1 1 5E9AA4EE
 P 7300 4650
@@
 $EndComp
 $Comp
-L power:+VDC #PWR?
+L Mainboard-rescue:+VDC-power #PWR?
 U 1 1 5E9AA4E8
 P 7300 3150
@@
 	3250 3150 3250 3750
 $Comp
-L power:+VDC #PWR?
+L Mainboard-rescue:+VDC-power #PWR?
 U 1 1 5E9AA4E1
 P 3250 3150
@@
 $EndComp
 $Comp
-L Regulator_Switching:R-785.0-1.0 U?
+L Mainboard-rescue:R-785.0-1.0-Regulator_Switching U?
 U 1 1 5E9AA4DB
 P 3750 3750
@@
 	2700 3950 2750 3950
 $Comp
-L power:GND #PWR?
+L Mainboard-rescue:GND-power #PWR?
 U 1 1 5E9AA4CF
 P 2750 4650
@@
 	3750 4050 3750 4650
 $Comp
-L power:GND #PWR?
+L Mainboard-rescue:GND-power #PWR?
 U 1 1 5E9AA4BF
 P 3750 4650
@@
 	3150 3750 3250 3750
 $Comp
-L Diode:1N4148W D?
+L Mainboard-rescue:1N4148W-Diode D?
 U 1 1 5E9AA4B5
 P 3000 3750
@@
 	3450 3750 3250 3750
 $Comp
-L power:+5V #PWR?
+L Mainboard-rescue:+5V-power #PWR?
 U 1 1 5E9AA4A9
 P 4200 3050
@@
 $EndComp
 $Comp
-L power:GND #PWR?
+L Mainboard-rescue:GND-power #PWR?
 U 1 1 5E9AA4A3
 P 4200 4650
@@
 $EndComp
 $Comp
-L power:GND #PWR?
+L Mainboard-rescue:GND-power #PWR?
 U 1 1 5E9AA49D
 P 3250 4650
@@
 $EndComp
 $Comp
-L Device:C C?
+L Mainboard-rescue:C-Device C?
 U 1 1 5E9AA497
 P 4200 4200
@@
 $EndComp
 $Comp
-L Device:C C?
+L Mainboard-rescue:C-Device C?
 U 1 1 5E9AA491
 P 3250 4200
@@
 	6100 4550 6100 4650
 $Comp
-L power:GND #PWR?
+L Mainboard-rescue:GND-power #PWR?
 U 1 1 5E9AA487
 P 6100 4650
@@
 	6100 4000 6100 4250
 $Comp
-L Device:C C?
+L Mainboard-rescue:C-Device C?
 U 1 1 5E9AA47C
 P 6100 4400
@@
 $EndComp
 $Comp
-L power:GND #PWR?
+L Mainboard-rescue:GND-power #PWR?
 U 1 1 5E9AA476
 P 5650 4650
@@
 	5650 3050 5650 3150
 $Comp
-L power:+5V #PWR?
+L Mainboard-rescue:+5V-power #PWR?
 U 1 1 5E9AA46F
 P 5650 3050
@@
 $EndComp
 $Comp
-L Device:R R?
+L Mainboard-rescue:R-Device R?
 U 1 1 5E9AA460
 P 5650 3300
@@
 Connection ~ 6100 4000
 $Comp
-L Device:R R?
+L Mainboard-rescue:R-Device R?
 U 1 1 5E74121A
 P 3075 5975
@@
 	5650 4450 5650 4650
 $Comp
-L Switch:SW_Push SW?
+L Mainboard-rescue:SW_Push-Switch SW?
 U 1 1 5E9AA469
 P 5650 4250
@@
 	5650 3600 6100 3600
 $Comp
-L Device:R R?
+L Mainboard-rescue:R-Device R?
 U 1 1 5E734C17
 P 5650 3850
