File: hardware/USB.sch (KiCad schematic (older format))
At the start: 9 parts, among them IC10 FT232RL, X6 SERIAL

Commit message: Update project
Parts:
- C10, C11, C12: symbol Mainboard-rescue:C-Device -> Device:C
- D10, D9: symbol Mainboard-rescue:LED-Device -> Device:LED
- IC10: symbol Mainboard-rescue:FT232RL-Interface_USB -> Interface_USB:FT232RL
- R8, R9: symbol Mainboard-rescue:R-Device -> Device:R
- X6: symbol Mainboard-rescue:USB-B-Connector_Custom -> Connector_Custom:USB-B
Changed lines of the file:
@@
 Sheet 6 7
 Title "USB-Serial"
-Date "2021-05-10"
+Date "2020-10-11"
 Rev "1.0"
 Comp "https://www.kampis-elektroecke.de"
@@
 $EndDescr
 $Comp
-L Mainboard-rescue:FT232RL-Interface_USB IC?
+L Interface_USB:FT232RL IC?
 U 1 1 5E95D1D6
 P 5650 3850
@@
 $EndComp
 $Comp
-L Mainboard-rescue:C-Device C?
+L Device:C C?
 U 1 1 5E95D20C
 P 4650 3150
@@
 $EndComp
 $Comp
-L Mainboard-rescue:GND-power #PWR?
+L power:GND #PWR?
 U 1 1 5E95D212
 P 4500 3150
@@
 Connection ~ 5750 4950
 $Comp
-L Mainboard-rescue:+5V-power #PWR?
+L power:+5V #PWR?
 U 1 1 5E95D229
 P 7600 3250
@@
 	3150 3900 3200 3900
 $Comp
-L Mainboard-rescue:GND-power #PWR?
+L power:GND #PWR?
 U 1 1 5E95D244
 P 3150 3950
@@
 NoConn ~ 6450 3750
 $Comp
-L Mainboard-rescue:+5V-power #PWR?
+L power:+5V #PWR?
 U 1 1 5ECF03CA
 P 5550 2000
@@
 $EndComp
 $Comp
-L Mainboard-rescue:GND-power #PWR?
+L power:GND #PWR?
 U 1 1 5ECF08BF
 P 5650 5050
@@
 	5750 2100 5750 2850
 $Comp
-L Mainboard-rescue:+5V-power #PWR?
+L power:+5V #PWR?
 U 1 1 5D9D8F30
 P 5750 2000
@@
 Connection ~ 5750 2100
 $Comp
-L Mainboard-rescue:USB-B-Connector_Custom X?
+L Connector_Custom:USB-B X?
 U 1 1 5DA7E5BF
 P 3200 3450
@@
 	6450 4150 7450 4150
 $Comp
-L Mainboard-rescue:R-Device R?
+L Device:R R?
 U 1 1 5E95D1EC
 P 7450 3950
@@
 $EndComp
 $Comp
-L Mainboard-rescue:LED-Device D?
+L Device:LED D?
 U 1 1 5E95D1E6
 P 7450 3500
@@
 	5400 2550 5400 2650
 $Comp
-L Mainboard-rescue:GND-power #PWR?
+L power:GND #PWR?
 U 1 1 5E2B8CA7
 P 5400 2650
@@
 $EndComp
 $Comp
-L Mainboard-rescue:C-Device C?
+L Device:C C?
 U 1 1 5E2B4DFA
 P 5400 2400
@@
 	5900 2100 5900 2250
 $Comp
-L Mainboard-rescue:GND-power #PWR?
+L power:GND #PWR?
 U 1 1 5E2BDF14
 P 5900 2650
@@
 $EndComp
 $Comp
-L Mainboard-rescue:C-Device C?
+L Device:C C?
 U 1 1 5E2BDF0E
 P 5900 2400
@@
 	7750 3800 7750 3650
 $Comp
-L Mainboard-rescue:LED-Device D?
+L Device:LED D?
 U 1 1 5E95D1F8
 P 7750 3500
@@
 $EndComp
 $Comp
-L Mainboard-rescue:R-Device R?
+L Device:R R?
 U 1 1 5E95D1F2
 P 7750 3950

Commit message: Initialize branch
Parts:
- C10, C11, C12: symbol Device:C -> Mainboard-rescue:C-Device
- D10, D9: symbol Device:LED -> Mainboard-rescue:LED-Device
- IC10: symbol Interface_USB:FT232RL -> Mainboard-rescue:FT232RL-Interface_USB
- R8, R9: symbol Device:R -> Mainboard-rescue:R-Device
- X6: symbol Connector_Custom:USB-B -> Mainboard-rescue:USB-B-Connector_Custom
Changed lines of the file:
@@
 Sheet 6 7
 Title "USB-Serial"
-Date "2020-10-11"
+Date "2021-05-10"
 Rev "1.0"
 Comp "https://www.kampis-elektroecke.de"
@@
 $EndDescr
 $Comp
-L Interface_USB:FT232RL IC?
+L Mainboard-rescue:FT232RL-Interface_USB IC?
 U 1 1 5E95D1D6
 P 5650 3850
@@
 $EndComp
 $Comp
-L Device:C C?
+L Mainboard-rescue:C-Device C?
 U 1 1 5E95D20C
 P 4650 3150
@@
 $EndComp
 $Comp
-L power:GND #PWR?
+L Mainboard-rescue:GND-power #PWR?
 U 1 1 5E95D212
 P 4500 3150
@@
 Connection ~ 5750 4950
 $Comp
-L power:+5V #PWR?
+L Mainboard-rescue:+5V-power #PWR?
 U 1 1 5E95D229
 P 7600 3250
@@
 	3150 3900 3200 3900
 $Comp
-L power:GND #PWR?
+L Mainboard-rescue:GND-power #PWR?
 U 1 1 5E95D244
 P 3150 3950
@@
 NoConn ~ 6450 3750
 $Comp
-L power:+5V #PWR?
+L Mainboard-rescue:+5V-power #PWR?
 U 1 1 5ECF03CA
 P 5550 2000
@@
 $EndComp
 $Comp
-L power:GND #PWR?
+L Mainboard-rescue:GND-power #PWR?
 U 1 1 5ECF08BF
 P 5650 5050
@@
 	5750 2100 5750 2850
 $Comp
-L power:+5V #PWR?
+L Mainboard-rescue:+5V-power #PWR?
 U 1 1 5D9D8F30
 P 5750 2000
@@
 Connection ~ 5750 2100
 $Comp
-L Connector_Custom:USB-B X?
+L Mainboard-rescue:USB-B-Connector_Custom X?
 U 1 1 5DA7E5BF
 P 3200 3450
@@
 	6450 4150 7450 4150
 $Comp
-L Device:R R?
+L Mainboard-rescue:R-Device R?
 U 1 1 5E95D1EC
 P 7450 3950
@@
 $EndComp
 $Comp
-L Device:LED D?
+L Mainboard-rescue:LED-Device D?
 U 1 1 5E95D1E6
 P 7450 3500
@@
 	5400 2550 5400 2650
 $Comp
-L power:GND #PWR?
+L Mainboard-rescue:GND-power #PWR?
 U 1 1 5E2B8CA7
 P 5400 2650
@@
 $EndComp
 $Comp
-L Device:C C?
+L Mainboard-rescue:C-Device C?
 U 1 1 5E2B4DFA
 P 5400 2400
@@
 	5900 2100 5900 2250
 $Comp
-L power:GND #PWR?
+L Mainboard-rescue:GND-power #PWR?
 U 1 1 5E2BDF14
 P 5900 2650
@@
 $EndComp
 $Comp
-L Device:C C?
+L Mainboard-rescue:C-Device C?
 U 1 1 5E2BDF0E
 P 5900 2400
@@
 	7750 3800 7750 3650
 $Comp
-L Device:LED D?
+L Mainboard-rescue:LED-Device D?
 U 1 1 5E95D1F8
 P 7750 3500
@@
 $EndComp
 $Comp
-L Device:R R?
+L Mainboard-rescue:R-Device R?
 U 1 1 5E95D1F2
 P 7750 3950
