File: hardware/IRQ.sch (KiCad schematic (older format))
At the start: 6 parts, among them IC9 74HC148, SW5 NMI

Commit message: Initialize branch
Parts:
- C9: symbol Device:C -> Mainboard-rescue:C-Device
- IC9: symbol Logic:74HC148 -> Mainboard-rescue:74HC148-Logic
- R6, R7: symbol Device:R -> Mainboard-rescue:R-Device
- RN3: symbol Device:R_Network08 -> Mainboard-rescue:R_Network08-Device
- SW5: symbol Switch:SW_Push -> Mainboard-rescue:SW_Push-Switch
Other:
- note removed: "- The W65C22N does need external pull up resistors for the IRQB line, because \nof the open collector IRQ output."
- note removed: "Info"
Changed lines of the file:
@@
 Sheet 5 7
 Title "Interrupt logic"
-Date "2020-10-11"
+Date "2021-05-10"
 Rev "1.0"
 Comp "https://www.kampis-elektroecke.de"
@@
 ~IRQ
 $Comp
-L power:+5V #PWR?
+L Mainboard-rescue:+5V-power #PWR?
 U 1 1 5E717796
 P 6350 2100
@@
 $EndComp
 $Comp
-L power:GND #PWR?
+L Mainboard-rescue:GND-power #PWR?
 U 1 1 5E7177A8
 P 6350 4300
@@
 	6350 4300 6350 3950
 $Comp
-L power:GND #PWR?
+L Mainboard-rescue:GND-power #PWR?
 U 1 1 5E7177AF
 P 5900 4300
@@
 Connection ~ 5600 3550
 $Comp
-L Device:R R?
+L Mainboard-rescue:R-Device R?
 U 1 1 5DE0C707
 P 900 900
@@
 $EndComp
 $Comp
-L power:+5V #PWR?
+L Mainboard-rescue:+5V-power #PWR?
 U 1 1 5DE0C716
 P 900 725
@@
 	900  725  900  750
 $Comp
-L power:GND #PWR?
+L Mainboard-rescue:GND-power #PWR?
 U 1 1 5DE0C71D
 P 900 1925
@@
 $EndComp
 $Comp
-L Device:C C?
+L Mainboard-rescue:C-Device C?
 U 1 1 5DE0C726
 P 1300 1600
@@
 Connection ~ 900  1250
 $Comp
-L power:GND #PWR?
+L Mainboard-rescue:GND-power #PWR?
 U 1 1 5DE0C731
 P 1300 1925
@@
 	900  1250 950  1250
 $Comp
-L Switch:SW_Push SW?
+L Mainboard-rescue:SW_Push-Switch SW?
 U 1 1 5DE0C710
 P 900 1600
@@
 NoConn ~ 6750 3150
 NoConn ~ 6750 3250
-Text Notes 7100 5950 0    50   ~ 0
-- The W65C22N does need external pull up resistors for the IRQB line, because \nof the open collector IRQ output.
 Wire Wire Line
 	5100 2100 5100 2250
 $Comp
-L power:+5V #PWR?
+L Mainboard-rescue:+5V-power #PWR?
 U 1 1 5E7177C0
 P 5100 2100
@@
 $EndComp
 $Comp
-L Device:R_Network08 RN?
+L Mainboard-rescue:R_Network08-Device RN?
 U 1 1 5E7177BA
 P 5500 2450
@@
 	5700 3450 5700 2650
 $Comp
-L Logic:74HC148 IC?
+L Mainboard-rescue:74HC148-Logic IC?
 U 1 1 5E7177D6
 P 6350 3350
@@
 	6750 3600 7400 3600
 $Comp
-L Device:R R?
+L Mainboard-rescue:R-Device R?
 U 1 1 5E72F959
 P 1100 1250
@@
 Wire Wire Line
 	900  1250 900  1400
-Wire Notes Line
-	7000 6450 11150 6450
-Wire Notes Line
-	11150 6450 11150 5550
-Wire Notes Line
-	11125 5550 6975 5550
-Wire Notes Line
-	6975 5550 6975 6450
-Text Notes 7050 5750 0    100  ~ 20
-Info
 $EndSCHEMATC

Commit message: Update project
Parts:
- C9: symbol Mainboard-rescue:C-Device -> Device:C
- IC9: symbol Mainboard-rescue:74HC148-Logic -> Logic:74HC148
- R6, R7: symbol Mainboard-rescue:R-Device -> Device:R
- RN3: symbol Mainboard-rescue:R_Network08-Device -> Device:R_Network08
- SW5: symbol Mainboard-rescue:SW_Push-Switch -> Switch:SW_Push
Other:
- note added: "- The W65C22N does need external pull up resistors for the IRQB line, because \nof the open collector IRQ output."
- note added: "Info"
Changed lines of the file:
@@
 Sheet 5 7
 Title "Interrupt logic"
-Date "2021-05-10"
+Date "2020-10-11"
 Rev "1.0"
 Comp "https://www.kampis-elektroecke.de"
@@
 ~IRQ
 $Comp
-L Mainboard-rescue:+5V-power #PWR?
+L power:+5V #PWR?
 U 1 1 5E717796
 P 6350 2100
@@
 $EndComp
 $Comp
-L Mainboard-rescue:GND-power #PWR?
+L power:GND #PWR?
 U 1 1 5E7177A8
 P 6350 4300
@@
 	6350 4300 6350 3950
 $Comp
-L Mainboard-rescue:GND-power #PWR?
+L power:GND #PWR?
 U 1 1 5E7177AF
 P 5900 4300
@@
 Connection ~ 5600 3550
 $Comp
-L Mainboard-rescue:R-Device R?
+L Device:R R?
 U 1 1 5DE0C707
 P 900 900
@@
 $EndComp
 $Comp
-L Mainboard-rescue:+5V-power #PWR?
+L power:+5V #PWR?
 U 1 1 5DE0C716
 P 900 725
@@
 	900  725  900  750
 $Comp
-L Mainboard-rescue:GND-power #PWR?
+L power:GND #PWR?
 U 1 1 5DE0C71D
 P 900 1925
@@
 $EndComp
 $Comp
-L Mainboard-rescue:C-Device C?
+L Device:C C?
 U 1 1 5DE0C726
 P 1300 1600
@@
 Connection ~ 900  1250
 $Comp
-L Mainboard-rescue:GND-power #PWR?
+L power:GND #PWR?
 U 1 1 5DE0C731
 P 1300 1925
@@
 	900  1250 950  1250
 $Comp
-L Mainboard-rescue:SW_Push-Switch SW?
+L Switch:SW_Push SW?
 U 1 1 5DE0C710
 P 900 1600
@@
 NoConn ~ 6750 3150
 NoConn ~ 6750 3250
+Text Notes 7100 5950 0    50   ~ 0
+- The W65C22N does need external pull up resistors for the IRQB line, because \nof the open collector IRQ output.
 Wire Wire Line
 	5100 2100 5100 2250
 $Comp
-L Mainboard-rescue:+5V-power #PWR?
+L power:+5V #PWR?
 U 1 1 5E7177C0
 P 5100 2100
@@
 $EndComp
 $Comp
-L Mainboard-rescue:R_Network08-Device RN?
+L Device:R_Network08 RN?
 U 1 1 5E7177BA
 P 5500 2450
@@
 	5700 3450 5700 2650
 $Comp
-L Mainboard-rescue:74HC148-Logic IC?
+L Logic:74HC148 IC?
 U 1 1 5E7177D6
 P 6350 3350
@@
 	6750 3600 7400 3600
 $Comp
-L Mainboard-rescue:R-Device R?
+L Device:R R?
 U 1 1 5E72F959
 P 1100 1250
@@
 Wire Wire Line
 	900  1250 900  1400
+Wire Notes Line
+	7000 6450 11150 6450
+Wire Notes Line
+	11150 6450 11150 5550
+Wire Notes Line
+	11125 5550 6975 5550
+Wire Notes Line
+	6975 5550 6975 6450
+Text Notes 7050 5750 0    100  ~ 20
+Info
 $EndSCHEMATC
