File: hardware/LCD_PS2.sch (KiCad schematic (older format))
At the start: 8 parts, among them T1 BC546, X3 TIMER, X4 KEYBOARD

Commit message: Initialize branch
Parts:
- DS1: symbol Display_Character:WC1602A -> Mainboard-rescue:WC1602A-Display_Character
- R1, R2, R3: symbol Device:R -> Mainboard-rescue:R-Device
- RV1: symbol Device:R_POT -> Mainboard-rescue:R_POT-Device
- T1: symbol Transistor_BJT:BC546 -> Mainboard-rescue:BC546-Transistor_BJT
- X3: symbol Connector_Generic:Conn_01x04 -> Mainboard-rescue:Conn_01x04-Connector_Generic
- X4: symbol Connector_Custom:Mini-DIN-6 -> Mainboard-rescue:Mini-DIN-6-Connector_Custom
Changed lines of the file:
@@
 Sheet 3 7
 Title "LCD, P2/2 & Timer"
-Date "2020-10-11"
+Date "2021-05-10"
 Rev "1.0"
 Comp "https://www.kampis-elektroecke.de"
@@
 	5075 3575 5075 3625
 $Comp
-L power:GND #PWR?
+L Mainboard-rescue:GND-power #PWR?
 U 1 1 5DAE0AEC
 P 5075 3625
@@
 NoConn ~ 6125 2025
 $Comp
-L power:GND #PWR?
+L Mainboard-rescue:GND-power #PWR?
 U 1 1 5DE9A843
 P 6125 2400
@@
 	5475 2475 5625 2475
 $Comp
-L power:+5V #PWR?
+L Mainboard-rescue:+5V-power #PWR?
 U 1 1 5DE9C02E
 P 5625 2425
@@
 	5475 2175 5975 2175
 $Comp
-L power:+5V #PWR?
+L Mainboard-rescue:+5V-power #PWR?
 U 1 1 5DADFE9B
 P 5075 1875
@@
 LCD[0..11]
 $Comp
-L Connector_Custom:Mini-DIN-6 X4
+L Mainboard-rescue:Mini-DIN-6-Connector_Custom X4
 U 1 1 5DD571A9
 P 5550 5550
@@
 $EndComp
 $Comp
-L power:+5V #PWR?
+L Mainboard-rescue:+5V-power #PWR?
 U 1 1 5DD5A54C
 P 5075 5450
@@
 	5550 5850 5550 5900
 $Comp
-L power:GND #PWR?
+L Mainboard-rescue:GND-power #PWR?
 U 1 1 5DA8A71B
 P 5550 5900
@@
 $EndComp
 $Comp
-L Device:R_POT RV1
+L Mainboard-rescue:R_POT-Device RV1
 U 1 1 5DE99AEE
 P 6125 2175
@@
 $EndComp
 $Comp
-L Display_Character:WC1602A DS1
+L Mainboard-rescue:WC1602A-Display_Character DS1
 U 1 1 5DAA1FEA
 P 5075 2775
@@
 $EndComp
 $Comp
-L power:GND #PWR?
+L Mainboard-rescue:GND-power #PWR?
 U 1 1 5DDCDE4D
 P 6125 5900
@@
 NoConn ~ 5250 5650
 $Comp
-L Device:R R?
+L Mainboard-rescue:R-Device R?
 U 1 1 5E36C0FD
 P 4975 6100
@@
 $EndComp
 $Comp
-L Device:R R?
+L Mainboard-rescue:R-Device R?
 U 1 1 5E36C658
 P 5075 6100
@@
 	5025 5900 5075 5900
 $Comp
-L power:+5V #PWR?
+L Mainboard-rescue:+5V-power #PWR?
 U 1 1 5E36F16F
 P 5025 5850
@@
 $EndComp
 $Comp
-L Transistor_BJT:BC546 T1
+L Mainboard-rescue:BC546-Transistor_BJT T1
 U 1 1 5E3A14A2
 P 5525 4400
@@
 	6125 2325 6125 2400
 $Comp
-L power:GND #PWR?
+L Mainboard-rescue:GND-power #PWR?
 U 1 1 5E3B1822
 P 5625 4725
@@
 	5625 2575 5625 4200
 $Comp
-L Device:R R?
+L Mainboard-rescue:R-Device R?
 U 1 1 5E3B3B17
 P 4650 4225
@@
 $EndComp
 $Comp
-L power:+5V #PWR?
+L Mainboard-rescue:+5V-power #PWR?
 U 1 1 5E3B5DDD
 P 4650 4000
@@
 Timer[0..1]
 $Comp
-L power:GND #PWR?
+L Mainboard-rescue:GND-power #PWR?
 U 1 1 5E772A75
 P 2925 1475
@@
 	1975 1175 2275 1175
 $Comp
-L Connector_Generic:Conn_01x04 X3
+L Mainboard-rescue:Conn_01x04-Connector_Generic X3
 U 1 1 5E783A1F
 P 3200 1275
@@
 	2925 1475 3000 1475
 $Comp
-L power:GND #PWR?
+L Mainboard-rescue:GND-power #PWR?
 U 1 1 5E78679F
 P 2925 1175
@@
 Wire Wire Line
 	2375 1375 3000 1375
-Text Notes 4150 5850 0    50   ~ 0
+Text Notes 4300 5650 0    50   ~ 0
 PS/2 Connector\n\n1\n2\n3\n4\n5\n6
-Text Notes 4375 5850 0    50   ~ 0
+Text Notes 4525 5650 0    50   ~ 0
 Data\nNC\nGND\n+5V\nClock\nNC
 Wire Bus Line

Commit message: Update project
Parts:
- DS1: symbol Mainboard-rescue:WC1602A-Display_Character -> Display_Character:WC1602A
- R1, R2, R3: symbol Mainboard-rescue:R-Device -> Device:R
- RV1: symbol Mainboard-rescue:R_POT-Device -> Device:R_POT
- T1: symbol Mainboard-rescue:BC546-Transistor_BJT -> Transistor_BJT:BC546
- X3: symbol Mainboard-rescue:Conn_01x04-Connector_Generic -> Connector_Generic:Conn_01x04
- X4: symbol Mainboard-rescue:Mini-DIN-6-Connector_Custom -> Connector_Custom:Mini-DIN-6
Changed lines of the file:
@@
 Sheet 3 7
 Title "LCD, P2/2 & Timer"
-Date "2021-05-10"
+Date "2020-10-11"
 Rev "1.0"
 Comp "https://www.kampis-elektroecke.de"
@@
 	5075 3575 5075 3625
 $Comp
-L Mainboard-rescue:GND-power #PWR?
+L power:GND #PWR?
 U 1 1 5DAE0AEC
 P 5075 3625
@@
 NoConn ~ 6125 2025
 $Comp
-L Mainboard-rescue:GND-power #PWR?
+L power:GND #PWR?
 U 1 1 5DE9A843
 P 6125 2400
@@
 	5475 2475 5625 2475
 $Comp
-L Mainboard-rescue:+5V-power #PWR?
+L power:+5V #PWR?
 U 1 1 5DE9C02E
 P 5625 2425
@@
 	5475 2175 5975 2175
 $Comp
-L Mainboard-rescue:+5V-power #PWR?
+L power:+5V #PWR?
 U 1 1 5DADFE9B
 P 5075 1875
@@
 LCD[0..11]
 $Comp
-L Mainboard-rescue:Mini-DIN-6-Connector_Custom X4
+L Connector_Custom:Mini-DIN-6 X4
 U 1 1 5DD571A9
 P 5550 5550
@@
 $EndComp
 $Comp
-L Mainboard-rescue:+5V-power #PWR?
+L power:+5V #PWR?
 U 1 1 5DD5A54C
 P 5075 5450
@@
 	5550 5850 5550 5900
 $Comp
-L Mainboard-rescue:GND-power #PWR?
+L power:GND #PWR?
 U 1 1 5DA8A71B
 P 5550 5900
@@
 $EndComp
 $Comp
-L Mainboard-rescue:R_POT-Device RV1
+L Device:R_POT RV1
 U 1 1 5DE99AEE
 P 6125 2175
@@
 $EndComp
 $Comp
-L Mainboard-rescue:WC1602A-Display_Character DS1
+L Display_Character:WC1602A DS1
 U 1 1 5DAA1FEA
 P 5075 2775
@@
 $EndComp
 $Comp
-L Mainboard-rescue:GND-power #PWR?
+L power:GND #PWR?
 U 1 1 5DDCDE4D
 P 6125 5900
@@
 NoConn ~ 5250 5650
 $Comp
-L Mainboard-rescue:R-Device R?
+L Device:R R?
 U 1 1 5E36C0FD
 P 4975 6100
@@
 $EndComp
 $Comp
-L Mainboard-rescue:R-Device R?
+L Device:R R?
 U 1 1 5E36C658
 P 5075 6100
@@
 	5025 5900 5075 5900
 $Comp
-L Mainboard-rescue:+5V-power #PWR?
+L power:+5V #PWR?
 U 1 1 5E36F16F
 P 5025 5850
@@
 $EndComp
 $Comp
-L Mainboard-rescue:BC546-Transistor_BJT T1
+L Transistor_BJT:BC546 T1
 U 1 1 5E3A14A2
 P 5525 4400
@@
 	6125 2325 6125 2400
 $Comp
-L Mainboard-rescue:GND-power #PWR?
+L power:GND #PWR?
 U 1 1 5E3B1822
 P 5625 4725
@@
 	5625 2575 5625 4200
 $Comp
-L Mainboard-rescue:R-Device R?
+L Device:R R?
 U 1 1 5E3B3B17
 P 4650 4225
@@
 $EndComp
 $Comp
-L Mainboard-rescue:+5V-power #PWR?
+L power:+5V #PWR?
 U 1 1 5E3B5DDD
 P 4650 4000
@@
 Timer[0..1]
 $Comp
-L Mainboard-rescue:GND-power #PWR?
+L power:GND #PWR?
 U 1 1 5E772A75
 P 2925 1475
@@
 	1975 1175 2275 1175
 $Comp
-L Mainboard-rescue:Conn_01x04-Connector_Generic X3
+L Connector_Generic:Conn_01x04 X3
 U 1 1 5E783A1F
 P 3200 1275
@@
 	2925 1475 3000 1475
 $Comp
-L Mainboard-rescue:GND-power #PWR?
+L power:GND #PWR?
 U 1 1 5E78679F
 P 2925 1175
@@
 Wire Wire Line
 	2375 1375 3000 1375
-Text Notes 4300 5650 0    50   ~ 0
+Text Notes 4150 5850 0    50   ~ 0
 PS/2 Connector\n\n1\n2\n3\n4\n5\n6
-Text Notes 4525 5650 0    50   ~ 0
+Text Notes 4375 5850 0    50   ~ 0
 Data\nNC\nGND\n+5V\nClock\nNC
 Wire Bus Line
