File: hardware/IO Board/IO.sch (KiCad schematic (older format))
At the start: 25 parts, among them IC3 74HC138, IC6 W65C22

Commit message: Working on hardware
Parts:
- removed C1: 100nF, Capacitor_THT:C_Rect_L4.0mm_W2.5mm_P2.50mm, symbol Device:C
- removed IC? (x4): 74HC00, Package_DIP:DIP-14_W7.62mm_LongPads, symbol 74xx:74HC00
- removed X?: BUS, Connector_PinHeader_2.54mm:PinHeader_2x20_P2.54mm_Horizontal, symbol Connector_Generic:Conn_02x20_Odd_Even
- added X?: BUS, Connector_PinHeader_2.54mm:PinHeader_2x20_P2.54mm_Horizontal, symbol Connector_Generic:Conn_02x20_Odd_Even
Connections:
- net ~IRQ_VIA_1 is gone; now on net ~IRQ: IC6.21 (~IRQ)
- net +5V: now also X?.40 (Pin_40)
- net A0: now also X?.1 (Pin_1)
- net A1: now also X?.3 (Pin_3)
- net A10: now also X?.21 (Pin_21)
- net A11: now also X?.23 (Pin_23)
- net A12: now also X?.25 (Pin_25)
- net A13: now also X?.27 (Pin_27)
- net A14: now also X?.29 (Pin_29)
- net A15: now also X?.31 (Pin_31)
- net A2: now also X?.5 (Pin_5)
- net A3: now also X?.7 (Pin_7)
- net A4: now also X?.9 (Pin_9)
- net A5: now also X?.11 (Pin_11)
- net A6: now also X?.13 (Pin_13)
- net A7: now also X?.15 (Pin_15)
- net A8: now also X?.17 (Pin_17)
- net A9: now also X?.19 (Pin_19)
- net Clock: now also X?.20 (Pin_20)
- net D0: now also X?.2 (Pin_2)
- net D1: now also X?.4 (Pin_4)
- net D2: now also X?.6 (Pin_6)
- net D3: now also X?.8 (Pin_8)
- net D4: now also X?.10 (Pin_10)
- net D5: now also X?.12 (Pin_12)
- net D6: now also X?.14 (Pin_14)
- net D7: now also X?.16 (Pin_16)
- net GND: now also X?.39 (Pin_39)
- net RDY: now also X?.28 (Pin_28)
- net R~W: now also X?.18 (Pin_18), X?.33 (Pin_33)
- net Sync: now also X?.30 (Pin_30)
- net ~IRQ: now also X?.24 (Pin_24)
- net ~Reset: now also X?.22 (Pin_22); no longer IC6.34 (~RESET)
- net ~TerminalReady: now also X?.26 (Pin_26)
- net CLOCK_INT renamed CLOCK
- net CLOCK: now also X?.35 (Pin_35)
- new net ~RESET: IC6.34 (~RESET), X?.37 (Pin_37)
- no-connect marks 14 -> 11
Other:
- moved on the sheet: C7, IC6
