File: hardware/IO Board/IOBoard.kicad_pcb (KiCad board)
At the start: 2 copper layers, 160 x 160 mm, 77 parts, among them IC1 74HC00, IC10 W65C22, IC11 74HC148, IC12 74HC273, IC2 W65C02, IC3 74HC138, IC4 SYSTEM ROM, IC5 RAM, IC6 W65C22, IC7 W65C51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

Commit message: Working on hardware
Parts:
- removed C1, C10, C11, C12, C13, C17, C18, C19, C2, C3, C4, C5, C6, C7: 100nF, Capacitor_THT:C_Rect_L4.0mm_W2.5mm_P2.50mm
- removed C14, C15, C16: 100nF, Capacitor_SMD:C_0805_2012Metric
- removed C8: 30pF, Capacitor_THT:C_Rect_L4.0mm_W2.5mm_P2.50mm
- removed C9: 330nF, Capacitor_THT:C_Rect_L4.0mm_W2.5mm_P2.50mm
- removed D0: LED0, LED_THT:LED_D5.0mm
- removed D1: LED1, LED_THT:LED_D5.0mm
- removed D10: 1N4148, Diode_THT:D_DO-35_SOD27_P7.62mm_Horizontal
- removed D11: TX, LED_SMD:LED_0805_2012Metric
- removed D12: RX, LED_SMD:LED_0805_2012Metric
- removed D13: POWER, LED_THT:LED_D5.0mm
- removed D2: LED2, LED_THT:LED_D5.0mm
- removed D3: LED3, LED_THT:LED_D5.0mm
- removed D4: LED4, LED_THT:LED_D5.0mm
- removed D5: LED5, LED_THT:LED_D5.0mm
- removed D6: LED6, LED_THT:LED_D5.0mm
- removed D7: LED7, LED_THT:LED_D5.0mm
- removed DS1: DISPLAY, Display:WC1602A
- removed IC1: 74HC00, Package_DIP:DIP-14_W7.62mm_LongPads
- removed IC10, IC6: W65C22, Package_DIP:DIP-40_W15.24mm_LongPads
- removed IC11: 74HC148, Package_DIP:DIP-16_W7.62mm_LongPads
- removed IC12: 74HC273, Package_DIP:DIP-20_W7.62mm_LongPads
- removed IC2: W65C02, Package_DIP:DIP-40_W15.24mm_LongPads
- removed IC3: 74HC138, Package_DIP:DIP-16_W7.62mm_LongPads
- removed IC4: SYSTEM ROM, Package_DIP:DIP-28_W15.24mm_LongPads
- removed IC5: RAM, Package_DIP:DIP-28_W15.24mm_LongPads
- removed IC7: W65C51, Package_DIP:DIP-28_W15.24mm_LongPads
- removed IC8: TL7702A, Package_DIP:DIP-8_W7.62mm_LongPads
- removed IC9: FT232RL, Package_SO:SSOP-28_5.3x10.2mm_P0.65mm
- removed R1, R10, R11, R2, R3, R5, R9: 10k, Resistor_THT:R_Axial_DIN0207_L6.3mm_D2.5mm_P7.62mm_Horizontal
- removed R4: 1M, Resistor_THT:R_Axial_DIN0207_L6.3mm_D2.5mm_P7.62mm_Horizontal
- removed R6, R7: 1k, Resistor_SMD:R_0805_2012Metric
- removed R8: 470, Resistor_THT:R_Axial_DIN0207_L6.3mm_D2.5mm_P7.62mm_Horizontal
- removed RN1: 10k, Resistor_THT:R_Array_SIP11
- removed RN2: 470, Resistor_THT:R_Array_SIP9
- removed RN3: 4k7, Resistor_THT:R_Array_SIP9
- removed RV1: 10k, Potentiometer:Bourns_3386T_Vertical
- removed SW1: RESET, Button_Switch_THT:SW_PUSH_6mm_H4.3mm
- removed SW2: Interrupt, Button_Switch_THT:SW_DIP_SPSTx02_Slide_9.78x7.26mm_W7.62mm_P2.54mm
- removed SW3: Port B, Button_Switch_THT:SW_DIP_SPSTx08_Slide_9.78x22.5mm_W7.62mm_P2.54mm
- removed SW4: NMI, Button_Switch_THT:SW_PUSH_6mm_H4.3mm
- removed SW5: CARRIER, Button_Switch_THT:SW_E-Switch_EG1224_SPDT_Angled
- removed SW6: CLOCK, Button_Switch_THT:SW_PUSH_6mm_H4.3mm
- removed SW7: CLOCK INPUT, Switches:SW_E-Switch_EG1271_DPDT
- removed U1: R-785.0-1.0, Converter_DCDC:Converter_DCDC_RECOM_R-78E-0.5_THT
- removed X1: DC IN, Connector_Custom:BarrelJack_Wuerth_6941xx301002
- removed X3: EXPANSION, Connector_PinHeader_2.54mm:PinHeader_2x20_P2.54mm_Horizontal
- removed X4: KEYBOARD, Connector_Custom:Mini-DIN_TE_Female_6Pin_2rows
- removed XTAL1: 1MHz, Oscillator:Oscillator_DIP-14
- removed XTAL2: 1.8432MHz, Crystal:Crystal_HC49-U_Vertical
- X2: value SERIAL -> BUS; footprint Connector_Custom:USB-B_TE_2923042_Horizontal -> Connector_PinHeader_2.54mm:PinHeader_2x20_P2.54mm_Horizontal
- moved X2 60.0 mm to (307.8, 113.0), turned to 0 degrees
- moved REF** 39.5 mm to (309.8, 92.1)
- moved REF** 39.5 mm to (159.8, 92.1)
- moved REF** 29.4 mm to (309.8, 182.1)
- moved REF** 29.4 mm to (159.8, 182.1)
Connections:
- X2 pad 2: /USB/D- -> (no net)
- X2 pad 3: /USB/D+ -> (no net)
- X2 pad 4: GND -> (no net)
- X2 pad 5: GND -> (no net)
Routing:
- net /IO/A1: track 423.9 -> 0.00 mm, vias 6 -> 0
- net /IO/A0: track 419.1 -> 0.00 mm, vias 8 -> 0
- net /IO/D4: track 404.1 -> 0.00 mm, vias 9 -> 0
- net /IO/D5: track 397.8 -> 0.00 mm, vias 9 -> 0
- net /IO/D6: track 397.1 -> 0.00 mm, vias 9 -> 0
- net /IO/D1: track 396.9 -> 0.00 mm, vias 6 -> 0
- net /IO/D2: track 396.0 -> 0.00 mm, vias 6 -> 0
- net /IO/D3: track 394.0 -> 0.00 mm, vias 8 -> 0
- net /IO/D0: track 391.5 -> 0.00 mm, vias 6 -> 0
- net /IO/D7: track 389.8 -> 0.00 mm, vias 8 -> 0
- net /IO/A3: track 363.9 -> 0.00 mm, vias 5 -> 0
- net /IO/A2: track 361.0 -> 0.00 mm, vias 5 -> 0
- net /IO/~Reset: track 348.5 -> 0.00 mm, vias 7 -> 0
- net /IO/Clock: track 336.6 -> 0.00 mm, vias 13 -> 0
- net /IO/R~W: track 263.7 -> 0.00 mm, vias 9 -> 0
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Other:
- board size 160 x 160 mm -> 160 x 100 mm
- net class USB removed
- board text added: "IO Board 1.0"
- board text removed: "BTN"
- board text removed: "Baseboard 1.1"
- board text removed: "OFF"
- board text removed: "ON"
- board text removed: "OSC"
