File: hardware/IO Board/IOBoard.sch (KiCad schematic (older format))
At the start: 0 parts

Commit message: Working on hardware
Changed lines of the file:
@@
 1K
 $Sheet
-S 8250 6250 1600 1550
+S 7325 4750 2675 2800
 U 5EB09E21
 F0 "IO" 50
 F1 "IO.sch" 50
-F2 "PA[0..7]" O R 9850 7550 50
-F3 "PB[0..7]" I R 9850 7650 50
-F4 "TxD" O R 9850 6350 50
-F5 "RxD" I R 9850 6450 50
-F6 "RTS" O R 9850 6550 50
-F7 "CTS" I R 9850 6650 50
-F8 "~NMI" I L 8250 7475 50
-F9 "R~W" O R 9850 7250 50
-F10 "LCD[0..10]" B L 8250 6700 50
-F11 "PS2[0..1]" B L 8250 6800 50
-F12 "~ModemReady" I R 9850 6750 50
-F13 "Clock" O R 9850 7350 50
-F14 "~TerminalReady" O R 9850 6850 50
-F15 "~CarrierDetect" I R 9850 6950 50
-F16 "~Reset" I L 8250 6350 50
-F17 "~IRQ_VIA_2" O L 8250 7175 50
-F18 "~IRQ_VIA_1" O L 8250 7075 50
-F19 "~IRQ_ACIA" O L 8250 7275 50
-F20 "~IRQ_CPU" I L 8250 7375 50
-F21 "CB[0..1]" I R 9850 7750 50
-F22 "A[0..15]" O R 9850 7050 50
-F23 "D[0..7]" B R 9850 7150 50
-F24 "RDY" I L 8250 7650 50
-F25 "Sync" O L 8250 7750 50
 $EndSheet
 Wire Notes Line width 18 style solid
