File: hardware/Baseboard/IO.sch (KiCad schematic (older format))
At the start: 17 parts, among them SW2 Interrupt, SW3 Port B, SW4 ~NMI, SW5 CARRIER, X3 EXPANSION

Commit message: Rework hardware for IRQ, change some routing
Connections:
- net CB2 is gone; now on net CB1: RN1.2 (R1), SW2.1
- net CB1: no longer RN1.3 (R2), SW2.2
- new net CB0: RN1.3 (R2), SW2.2
Other:
- moved on the sheet: SW5
Changed lines of the file:
@@
 $Descr A4 11693 8268
 encoding utf-8
-Sheet 3 6
+Sheet 3 7
 Title "Baseboard"
-Date "2019-10-08"
-Rev "1.0"
+Date "2019-11-24"
+Rev "1.1"
 Comp "https://www.kampis-elektroecke.de"
 Comment1 "Author: Daniel Kampert"
@@
 Entry Wire Line
 	1900 2050 1800 1950
-Text Label 2000 2050 0    50   ~ 0
-CB2
-Text Label 2000 2150 0    50   ~ 0
-CB1
 Wire Bus Line
 	1800 1950 950  1950
 Text HLabel 950  1950 0    50   Output ~ 0
-CB[1..2]
+CB[0..1]
 Wire Bus Line
 	1800 1950 1800 2050
@@
 R~W
 Text HLabel 8800 1150 0    50   Input ~ 0
-A[15..0]
+A[0..15]
 Text HLabel 8800 1050 0    50   BiDi ~ 0
-D[7..0]
+D[0..7]
 Entry Wire Line
 	9250 1550 9350 1450
@@
 Wire Wire Line
 	10350 2550 10250 2550
-Text HLabel 3850 6200 0    50   Output ~ 0
+Text HLabel 2500 6825 0    50   Output ~ 0
 ~CarrierDetect
 $Comp
 L Switch:SW_SPDT SW5
 U 1 1 5DC04457
-P 4050 6200
-F 0 "SW5" H 4050 6485 50  0000 C CNN
-F 1 "CARRIER" H 4050 6394 50  0000 C CNN
-F 2 "Button_Switch_THT:SW_E-Switch_EG1224_SPDT_Angled" H 4050 6200 50  0001 C CNN
-F 3 "https://www.mouser.de/datasheet/2/140/EG-345873.pdf" H 4050 6200 50  0001 C CNN
-F 4 "E-Switch" H 4050 6200 50  0001 C CNN "Mfr."
-F 5 "EG1224" H 4050 6200 50  0001 C CNN "Mfr. No."
-F 6 "612-EG1224" H 4050 6200 50  0001 C CNN "Mouser"
-	1    4050 6200
+P 2700 6825
+F 0 "SW5" H 2700 7110 50  0000 C CNN
+F 1 "CARRIER" H 2700 7019 50  0000 C CNN
+F 2 "Button_Switch_THT:SW_E-Switch_EG1224_SPDT_Angled" H 2700 6825 50  0001 C CNN
+F 3 "https://www.mouser.de/datasheet/2/140/EG-345873.pdf" H 2700 6825 50  0001 C CNN
+F 4 "E-Switch" H 2700 6825 50  0001 C CNN "Mfr."
+F 5 "EG1224" H 2700 6825 50  0001 C CNN "Mfr. No."
+F 6 "612-EG1224" H 2700 6825 50  0001 C CNN "Mouser"
+	1    2700 6825
 	1    0    0    -1
 $EndComp
@@
 L power:GND #PWR?
 U 1 1 5DC0FBD8
-P 4350 6400
+P 3000 7050
 AR Path="/5DC0FBD8" Ref="#PWR?"  Part="1"
 AR Path="/5EB09E21/5DC0FBD8" Ref="#PWR?"  Part="1"
 AR Path="/5EC67F7B/5DC0FBD8" Ref="#PWR048"  Part="1"
-F 0 "#PWR048" H 4350 6150 50  0001 C CNN
-F 1 "GND" H 4355 6227 50  0000 C CNN
-F 2 "" H 4350 6400 50  0001 C CNN
-F 3 "" H 4350 6400 50  0001 C CNN
-	1    4350 6400
+F 0 "#PWR048" H 3000 6800 50  0001 C CNN
+F 1 "GND" H 3005 6877 50  0000 C CNN
+F 2 "" H 3000 7050 50  0001 C CNN
+F 3 "" H 3000 7050 50  0001 C CNN
+	1    3000 7050
 	1    0    0    -1
 $EndComp
@@
 L power:+5V #PWR?
 U 1 1 5DC13EF2
-P 4350 6050
+P 3000 6675
 AR Path="/5DC13EF2" Ref="#PWR?"  Part="1"
 AR Path="/5E9728CC/5DC13EF2" Ref="#PWR?"  Part="1"
 AR Path="/5EC67F7B/5DC13EF2" Ref="#PWR032"  Part="1"
-F 0 "#PWR032" H 4350 5900 50  0001 C CNN
-F 1 "+5V" H 4365 6223 50  0000 C CNN
-F 2 "" H 4350 6050 50  0001 C CNN
-F 3 "" H 4350 6050 50  0001 C CNN
-	1    4350 6050
-	1    0    0    -1
-$EndComp
-Wire Wire Line
-	4250 6100 4350 6100
-Wire Wire Line
-	4350 6100 4350 6050
-Wire Wire Line
-	4250 6300 4350 6300
-Wire Wire Line
-	4350 6300 4350 6400
+F 0 "#PWR032" H 3000 6525 50  0001 C CNN
+F 1 "+5V" H 3015 6848 50  0000 C CNN
+F 2 "" H 3000 6675 50  0001 C CNN
+F 3 "" H 3000 6675 50  0001 C CNN
+	1    3000 6675
+	1    0    0    -1
+$EndComp
+Wire Wire Line
+	2900 6725 3000 6725
+Wire Wire Line
+	3000 6725 3000 6675
+Wire Wire Line
+	2900 6925 3000 6925
+Text Label 2000 2150 0    50   ~ 0
+CB0
+Text Label 2000 2050 0    50   ~ 0
+CB1
+Wire Wire Line
+	3000 6925 3000 7050
 Wire Bus Line
 	2850 3450 2850 4150

Commit message: Improve routing, add some datasheet recommendations
Parts:
- removed C17: 100nF, Capacitor_THT:C_Rect_L4.0mm_W2.5mm_P2.50mm, symbol Device:C
- removed R9: 10k, Resistor_THT:R_Axial_DIN0207_L6.3mm_D2.5mm_P7.62mm_Horizontal, symbol Device:R
- removed SW4: ~NMI, Button_Switch_THT:SW_PUSH_6mm_H4.3mm, symbol Switch:SW_Push
Changed lines of the file:
@@
 Wire Wire Line
 	4200 2050 4300 2050
-$Comp
-L Device:R R?
-U 1 1 5D9FD99A
-P 850 6050
-AR Path="/5D9FD99A" Ref="R?"  Part="1"
-AR Path="/5E9728CC/5D9FD99A" Ref="R?"  Part="1"
-AR Path="/5EC67F7B/5D9FD99A" Ref="R9"  Part="1"
-F 0 "R9" H 920 6096 50  0000 L CNN
-F 1 "10k" H 920 6005 50  0000 L CNN
-F 2 "Resistor_THT:R_Axial_DIN0207_L6.3mm_D2.5mm_P7.62mm_Horizontal" V 780 6050 50  0001 C CNN
-F 3 "https://www.mouser.de/datasheet/2/447/Yageo%20LR_MFP_2013-594635.pdf" H 850 6050 50  0001 C CNN
-F 4 "Yageo" H 850 6050 50  0001 C CNN "Mfr."
-F 5 "MFP-25BRD52-10K" H 850 6050 50  0001 C CNN "Mfr. No."
-F 6 "603-MFP-25BRD52-10K" H 850 6050 50  0001 C CNN "Mouser"
-	1    850  6050
-	1    0    0    -1
-$EndComp
-$Comp
-L Switch:SW_Push SW?
-U 1 1 5D9FD9A3
-P 850 6650
-AR Path="/5D9FD9A3" Ref="SW?"  Part="1"
-AR Path="/5E9728CC/5D9FD9A3" Ref="SW?"  Part="1"
-AR Path="/5EC67F7B/5D9FD9A3" Ref="SW4"  Part="1"
-F 0 "SW4" V 896 6602 50  0000 R CNN
-F 1 "~NMI" V 805 6602 50  0000 R CNN
-F 2 "Button_Switch_THT:SW_PUSH_6mm_H4.3mm" H 850 6850 50  0001 C CNN
-F 3 "https://www.te.com/commerce/DocumentDelivery/DDEController?Action=showdoc&DocId=Customer+Drawing%7F1825910%7FC10%7Fpdf%7FEnglish%7FENG_CD_1825910_C10.pdf%7F2-1825910-7" H 850 6850 50  0001 C CNN
-F 4 "TE Connectivity / Alcoswitch" H 850 6650 50  0001 C CNN "Mfr."
-F 5 "2-1825910-7" H 850 6650 50  0001 C CNN "Mfr. No."
-F 6 "506-2-1825910-7" H 850 6650 50  0001 C CNN "Mouser"
-	1    850  6650
-	0    -1   -1   0
-$EndComp
-$Comp
-L power:+5V #PWR?
-U 1 1 5D9FD9A9
-P 850 5700
-AR Path="/5D9FD9A9" Ref="#PWR?"  Part="1"
-AR Path="/5E9728CC/5D9FD9A9" Ref="#PWR?"  Part="1"
-AR Path="/5EC67F7B/5D9FD9A9" Ref="#PWR057"  Part="1"
-F 0 "#PWR057" H 850 5550 50  0001 C CNN
-F 1 "+5V" H 865 5873 50  0000 C CNN
-F 2 "" H 850 5700 50  0001 C CNN
-F 3 "" H 850 5700 50  0001 C CNN
-	1    850  5700
-	1    0    0    -1
-$EndComp
-Wire Wire Line
-	850  5700 850  5900
-$Comp
-L power:GND #PWR?
-U 1 1 5D9FD9B0
-P 850 7050
-AR Path="/5D9FD9B0" Ref="#PWR?"  Part="1"
-AR Path="/5E9728CC/5D9FD9B0" Ref="#PWR?"  Part="1"
-AR Path="/5EC67F7B/5D9FD9B0" Ref="#PWR058"  Part="1"
-F 0 "#PWR058" H 850 6800 50  0001 C CNN
-F 1 "GND" H 855 6877 50  0000 C CNN
-F 2 "" H 850 7050 50  0001 C CNN
-F 3 "" H 850 7050 50  0001 C CNN
-	1    850  7050
-	1    0    0    -1
-$EndComp
-$Comp
-L Device:C C?
-U 1 1 5D9FD9B9
-P 1300 6800
-AR Path="/5D9FD9B9" Ref="C?"  Part="1"
-AR Path="/5E9728CC/5D9FD9B9" Ref="C?"  Part="1"
-AR Path="/5EC67F7B/5D9FD9B9" Ref="C17"  Part="1"
-F 0 "C17" H 1415 6846 50  0000 L CNN
-F 1 "100nF" H 1415 6755 50  0000 L CNN
-F 2 "Capacitor_THT:C_Rect_L4.0mm_W2.5mm_P2.50mm" H 1338 6650 50  0001 C CNN
-F 3 "https://www.mouser.de/datasheet/2/400/eadmlcc_halogenfree_fa150_en-890480.pdf" H 1300 6800 50  0001 C CNN
-F 4 "TDK" H 1300 6800 50  0001 C CNN "Mfr."
-F 5 "FA18X8R1H104KRU06" H 1300 6800 50  0001 C CNN "Mfr. No."
-F 6 "810-FA18X8R1H104KRU6" H 1300 6800 50  0001 C CNN "Mouser"
-	1    1300 6800
-	1    0    0    -1
-$EndComp
-Wire Wire Line
-	850  6200 850  6400
-Wire Wire Line
-	850  6400 1300 6400
-Wire Wire Line
-	1300 6400 1300 6650
-Connection ~ 850  6400
-Wire Wire Line
-	850  6400 850  6450
-$Comp
-L power:GND #PWR?
-U 1 1 5D9FD9C4
-P 1300 7050
-AR Path="/5D9FD9C4" Ref="#PWR?"  Part="1"
-AR Path="/5E9728CC/5D9FD9C4" Ref="#PWR?"  Part="1"
-AR Path="/5EC67F7B/5D9FD9C4" Ref="#PWR065"  Part="1"
-F 0 "#PWR065" H 1300 6800 50  0001 C CNN
-F 1 "GND" H 1305 6877 50  0000 C CNN
-F 2 "" H 1300 7050 50  0001 C CNN
-F 3 "" H 1300 7050 50  0001 C CNN
-	1    1300 7050
-	1    0    0    -1
-$EndComp
-Connection ~ 1300 6400
-Wire Wire Line
-	850  6850 850  7050
-Wire Wire Line
-	1300 6950 1300 7050
-Wire Wire Line
-	1300 6400 1600 6400
-Text HLabel 1600 6400 2    50   Output ~ 0
-~NMI
-Text HLabel 10350 2150 2    50   Input ~ 0
-R~W
 Text HLabel 8800 1150 0    50   Input ~ 0
 A[0..15]
@@
 Text Label 9450 1450 0    50   ~ 0
 A1
-Text HLabel 10350 2250 2    50   Input ~ 0
-Clock
 Wire Wire Line
 	10350 2250 10250 2250
@@
 Wire Wire Line
 	3000 6925 3000 7050
+Text HLabel 10350 2150 2    50   Input ~ 0
+R~W
+Text HLabel 10350 2250 2    50   Input ~ 0
+Clock
 Wire Bus Line
 	2850 3450 2850 4150

Commit message: Optimize routing, add RDY and SYNC to expansion header
Connections:
- net RDY: now reaches X3.28 (Pin_28)
- net Sync: now reaches X3.30 (Pin_30)
- no-connect marks 9 -> 7
Changed lines of the file:
@@
 NoConn ~ 10250 2950
 NoConn ~ 10250 2850
-NoConn ~ 10250 2750
-NoConn ~ 10250 2650
 Text HLabel 10350 2550 2    50   Input ~ 0
 ~TerminalReady
@@
 Text HLabel 10350 2250 2    50   Input ~ 0
 Clock
+Text HLabel 10350 2650 2    50   Output ~ 0
+RDY
+Wire Wire Line
+	10350 2650 10250 2650
+Text HLabel 10350 2750 2    50   Input ~ 0
+Sync
+Wire Wire Line
+	10350 2750 10250 2750
 Wire Bus Line
 	2850 3450 2850 4150

Commit message: Rename PortB and the interrupt DIP switch
Parts:
- SW2: value Interrupt -> INTERRUPT
- SW3: value Port B -> PORT B
Changed lines of the file:
@@
 AR Path="/5EC67F7B/5EE8631D" Ref="SW2"  Part="1"
 F 0 "SW2" H 4600 2000 50  0000 C CNN
-F 1 "Interrupt" H 4650 1900 50  0000 C CNN
+F 1 "INTERRUPT" H 4650 1900 50  0000 C CNN
 F 2 "Button_Switch_THT:SW_DIP_SPSTx02_Slide_9.78x7.26mm_W7.62mm_P2.54mm" H 4600 2150 50  0001 C CNN
 F 3 "https://www.weltroniker.de/DB-Pool/DIP_NDI.pdf" H 4600 2150 50  0001 C CNN
@@
 AR Path="/5EC67F7B/5EE69B10" Ref="SW3"  Part="1"
 F 0 "SW3" H 4600 2167 50  0000 C CNN
-F 1 "Port B" H 4600 2076 50  0000 C CNN
+F 1 "PORT B" H 4600 2076 50  0000 C CNN
 F 2 "Button_Switch_THT:SW_DIP_SPSTx08_Slide_9.78x22.5mm_W7.62mm_P2.54mm" H 4600 1500 50  0001 C CNN
 F 3 "https://www.weltroniker.de/DB-Pool/DIP_NDI.pdf" H 4600 1500 50  0001 C CNN

Commit message: Replace RN2 with 390 Ohms restistor network
Parts:
- RN2: value 470 -> 390; Mfr. No. 4608M-102-471LF -> 4609X-101-391LF; Mouser 652-4608M-2LF-470 -> 652-4609X-1LF-390
Changed lines of the file:
@@
 AR Path="/5EC67F7B/5ED5BED1" Ref="RN2"  Part="1"
 F 0 "RN2" H 4188 4696 50  0000 L CNN
-F 1 "470" H 4188 4605 50  0000 L CNN
+F 1 "390" H 4188 4605 50  0000 L CNN
 F 2 "Resistor_THT:R_Array_SIP9" V 4275 4650 50  0001 C CNN
-F 3 "http://www.vishay.com/docs/31509/csc.pdf" H 3800 4650 50  0001 C CNN
+F 3 "https://www.mouser.de/datasheet/2/54/4600x-776645.pdf" H 3800 4650 50  0001 C CNN
 F 4 "Bourns" H 3800 4650 50  0001 C CNN "Mfr."
-F 5 "4608M-102-471LF" H 3800 4650 50  0001 C CNN "Mfr. No."
-F 6 "652-4608M-2LF-470" H 3800 4650 50  0001 C CNN "Mouser"
+F 5 "4609X-101-391LF" H 3800 4650 50  0001 C CNN "Mfr. No."
+F 6 "652-4609X-1LF-390" H 3800 4650 50  0001 C CNN "Mouser"
 	1    3800 4650
 	-1   0    0    1

Commit message: Add VP signal to expansion header, optimize routing
Connections:
- net ~VP: now reaches X3.32 (Pin_32)
- no-connect marks 7 -> 6
Changed lines of the file:
@@
 NoConn ~ 10250 3050
 NoConn ~ 10250 2950
-NoConn ~ 10250 2850
 Text HLabel 10350 2550 2    50   Input ~ 0
 ~TerminalReady
@@
 Wire Wire Line
 	10350 2750 10250 2750
+Text HLabel 10350 2850 2    50   Input ~ 0
+~VP
+Wire Wire Line
+	10350 2850 10250 2850
 Wire Bus Line
 	2850 3450 2850 4150

Commit message: Working on PCB
Connections:
- net ~TerminalReady is gone; now on net RDY: X3.26 (Pin_26)
- net RDY: no longer X3.28 (Pin_28)
- net Sync: now also X3.28 (Pin_28); no longer X3.30 (Pin_30)
- net ~CarrierDetect renamed ~DCD
- no-connect marks 6 -> 7
Changed lines of the file:
@@
 Sheet 3 7
 Title "Baseboard"
-Date "2019-11-24"
-Rev "1.1"
+Date "2020-01-17"
+Rev "1.0"
 Comp "https://www.kampis-elektroecke.de"
 Comment1 "Author: Daniel Kampert"
@@
 NoConn ~ 10250 3050
 NoConn ~ 10250 2950
-Text HLabel 10350 2550 2    50   Input ~ 0
-~TerminalReady
-Wire Wire Line
-	10350 2550 10250 2550
-Text HLabel 2500 6825 0    50   Output ~ 0
-~CarrierDetect
-$Comp
-L Switch:SW_SPDT SW5
-U 1 1 5DC04457
-P 2700 6825
-F 0 "SW5" H 2700 7110 50  0000 C CNN
-F 1 "CARRIER" H 2700 7019 50  0000 C CNN
-F 2 "Button_Switch_THT:SW_E-Switch_EG1224_SPDT_Angled" H 2700 6825 50  0001 C CNN
-F 3 "https://www.mouser.de/datasheet/2/140/EG-345873.pdf" H 2700 6825 50  0001 C CNN
-F 4 "E-Switch" H 2700 6825 50  0001 C CNN "Mfr."
-F 5 "EG1224" H 2700 6825 50  0001 C CNN "Mfr. No."
-F 6 "612-EG1224" H 2700 6825 50  0001 C CNN "Mouser"
-	1    2700 6825
-	1    0    0    -1
-$EndComp
-$Comp
-L power:GND #PWR?
-U 1 1 5DC0FBD8
-P 3000 7050
-AR Path="/5DC0FBD8" Ref="#PWR?"  Part="1"
-AR Path="/5EB09E21/5DC0FBD8" Ref="#PWR?"  Part="1"
-AR Path="/5EC67F7B/5DC0FBD8" Ref="#PWR048"  Part="1"
-F 0 "#PWR048" H 3000 6800 50  0001 C CNN
-F 1 "GND" H 3005 6877 50  0000 C CNN
-F 2 "" H 3000 7050 50  0001 C CNN
-F 3 "" H 3000 7050 50  0001 C CNN
-	1    3000 7050
-	1    0    0    -1
-$EndComp
-$Comp
-L power:+5V #PWR?
-U 1 1 5DC13EF2
-P 3000 6675
-AR Path="/5DC13EF2" Ref="#PWR?"  Part="1"
-AR Path="/5E9728CC/5DC13EF2" Ref="#PWR?"  Part="1"
-AR Path="/5EC67F7B/5DC13EF2" Ref="#PWR032"  Part="1"
-F 0 "#PWR032" H 3000 6525 50  0001 C CNN
-F 1 "+5V" H 3015 6848 50  0000 C CNN
-F 2 "" H 3000 6675 50  0001 C CNN
-F 3 "" H 3000 6675 50  0001 C CNN
-	1    3000 6675
-	1    0    0    -1
-$EndComp
-Wire Wire Line
-	2900 6725 3000 6725
-Wire Wire Line
-	3000 6725 3000 6675
-Wire Wire Line
-	2900 6925 3000 6925
 Text Label 2000 2150 0    50   ~ 0
 CB0
 Text Label 2000 2050 0    50   ~ 0
 CB1
-Wire Wire Line
-	3000 6925 3000 7050
 Text HLabel 10350 2150 2    50   Input ~ 0
 R~W
 Text HLabel 10350 2250 2    50   Input ~ 0
 Clock
-Text HLabel 10350 2650 2    50   Output ~ 0
-RDY
-Wire Wire Line
-	10350 2650 10250 2650
-Text HLabel 10350 2750 2    50   Input ~ 0
-Sync
-Wire Wire Line
-	10350 2750 10250 2750
 Text HLabel 10350 2850 2    50   Input ~ 0
 ~VP
 Wire Wire Line
 	10350 2850 10250 2850
+Text HLabel 10350 2550 2    50   Output ~ 0
+RDY
+Wire Wire Line
+	10350 2550 10250 2550
+Text HLabel 10350 2650 2    50   Input ~ 0
+Sync
+Wire Wire Line
+	10350 2650 10250 2650
+NoConn ~ 10250 2750
+Wire Wire Line
+	1925 6475 1925 6600
+Wire Wire Line
+	1825 6475 1925 6475
+Wire Wire Line
+	1925 6275 1925 6225
+Wire Wire Line
+	1825 6275 1925 6275
+$Comp
+L power:+5V #PWR?
+U 1 1 5E24E58E
+P 1925 6225
+AR Path="/5E24E58E" Ref="#PWR?"  Part="1"
+AR Path="/5E9728CC/5E24E58E" Ref="#PWR?"  Part="1"
+AR Path="/5EC67F7B/5E24E58E" Ref="#PWR013"  Part="1"
+F 0 "#PWR013" H 1925 6075 50  0001 C CNN
+F 1 "+5V" H 1940 6398 50  0000 C CNN
+F 2 "" H 1925 6225 50  0001 C CNN
+F 3 "" H 1925 6225 50  0001 C CNN
+	1    1925 6225
+	1    0    0    -1
+$EndComp
+$Comp
+L power:GND #PWR?
+U 1 1 5E24E594
+P 1925 6600
+AR Path="/5E24E594" Ref="#PWR?"  Part="1"
+AR Path="/5EB09E21/5E24E594" Ref="#PWR?"  Part="1"
+AR Path="/5EC67F7B/5E24E594" Ref="#PWR024"  Part="1"
+F 0 "#PWR024" H 1925 6350 50  0001 C CNN
+F 1 "GND" H 1930 6427 50  0000 C CNN
+F 2 "" H 1925 6600 50  0001 C CNN
+F 3 "" H 1925 6600 50  0001 C CNN
+	1    1925 6600
+	1    0    0    -1
+$EndComp
+$Comp
+L Switch:SW_SPDT SW5
+U 1 1 5E24E59D
+P 1625 6375
+F 0 "SW5" H 1625 6660 50  0000 C CNN
+F 1 "CARRIER" H 1625 6569 50  0000 C CNN
+F 2 "Button_Switch_THT:SW_E-Switch_EG1224_SPDT_Angled" H 1625 6375 50  0001 C CNN
+F 3 "https://www.mouser.de/datasheet/2/140/EG-345873.pdf" H 1625 6375 50  0001 C CNN
+F 4 "E-Switch" H 1625 6375 50  0001 C CNN "Mfr."
+F 5 "EG1224" H 1625 6375 50  0001 C CNN "Mfr. No."
+F 6 "612-EG1224" H 1625 6375 50  0001 C CNN "Mouser"
+	1    1625 6375
+	1    0    0    -1
+$EndComp
+Text HLabel 950  6375 0    50   Output ~ 0
+~DCD
+Wire Wire Line
+	1425 6375 950  6375
 Wire Bus Line
 	2850 3450 2850 4150
