File: hardware/Baseboard/Processor.sch (KiCad schematic (older format))
At the start: 29 parts, among them IC1 74HC00, IC10 W65C22, IC2 W65C02, IC3 74HC138, IC4 SYSTEM ROM, IC5 RAM, IC6 W65C22, IC7 W65C51, SW6 CLOCK, SW7 CLOCK INPUT

Commit message: Rework hardware for IRQ, change some routing
Parts:
- removed D14, D8, D9: SD103A, Diode_THT:D_DO-35_SOD27_P7.62mm_Horizontal, symbol Device:D_Schottky
Connections:
- net labels added: A[0..15], CB0, CB[0..1], CLOCK_INT, D[0..7], IRQ_Sync, ~IRQ_CPU, ~IRQ_Read
- net labels removed: A[15..0], CB2, CB[1..2], Clock_Int, D[7..0], ~IRQ
- wire segments 286 -> 281
- no-connect marks 23 -> 21
Other:
- moved on the sheet: C1, C18, C19, C2, C3, C4, C5, C6, C7, C8, IC10, IC1A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

Commit message: Improve routing, add some datasheet recommendations
Parts:
- removed R1: 10k, Resistor_THT:R_Axial_DIN0207_L6.3mm_D2.5mm_P7.62mm_Horizontal, symbol Device:R
Connections:
- net +5V: now also IC2.36 (BE), IC2.38 (~SO)
- net IRQ_Sync: no longer names the net of IC2.39 (PHI2O)
- no-connect marks 21 -> 20
Other:
- note added: "NOTE: WDC recommends to use an oscillator for system time base \ninstead of PHI1O and PHI2O, because the clock delay of PHI1O \nand PHI2O to PHI2 is no longer tested."
- moved on the sheet: SW7
Changed lines of the file:
@@
 Comment4 "Processor and Bus"
 $EndDescr
-$Comp
-L Western_Design_Center:W65C02 IC?
-U 1 1 5EBEAF78
-P 5200 5375
-AR Path="/5EBEAF78" Ref="IC?"  Part="1"
-AR Path="/5EB09E21/5EBEAF78" Ref="IC2"  Part="1"
-F 0 "IC2" H 4800 6575 50  0000 C CNN
-F 1 "W65C02" H 4890 4175 50  0000 C CNN
-F 2 "Package_DIP:DIP-40_W15.24mm_LongPads" H 5200 5075 50  0001 C CNN
-F 3 "https://www.westerndesigncenter.com/wdc/documentation/w65c02s.pdf" H 5200 5375 50  0001 C CNN
-F 4 "Western Design Center" H 5200 5375 50  0001 C CNN "Mfr."
-F 5 "W65C02S6TPG-14" H 5200 5375 50  0001 C CNN "Mfr. No."
-F 6 "955-W65C02S6TPG-14" H 5200 5375 50  0001 C CNN "Mouser"
-	1    5200 5375
-	1    0    0    -1
-$EndComp
 Entry Wire Line
 	4150 5125 4250 5025
@@
 	5450 3925 5450 3975
 NoConn ~ 5750 4525
-NoConn ~ 5750 5225
 NoConn ~ 5750 4925
 Wire Wire Line
@@
 	2750 1175 2750 825
 Wire Wire Line
-	4650 1075 4800 1075
+	4850 1500 5400 1500
 Wire Wire Line
 	2750 1775 2750 2175
@@
 	1    0    0    -1
 $EndComp
-Text Label 4800 1075 0    50   ~ 0
+Text Label 4900 1500 0    50   ~ 0
 CLOCK_INT
-Text Label 5800 4325 0    50   ~ 0
+Text Label 6200 4325 0    50   ~ 0
 CLOCK_INT
 Text Label 12700 6125 2    50   ~ 0
@@
 NoConn ~ 10700 1625
 NoConn ~ 10700 1725
-Text HLabel 6200 4325 2    50   Output ~ 0
+Text HLabel 5400 1500 2    50   Output ~ 0
 Clock
 $Comp
@@
 	1    0    0    -1
 $EndComp
-NoConn ~ 5750 5325
 NoConn ~ 5750 4725
 Wire Wire Line
@@
 Text Label 1500 1575 0    50   ~ 0
 CLOCK_BTN
-Text Label 4150 975  2    50   ~ 0
+Text Label 4350 1400 2    50   ~ 0
 CLOCK_BTN
 Text Label 3250 1475 0    50   ~ 0
@@
 Wire Wire Line
 	3250 1475 3150 1475
-Text Label 4150 1175 2    50   ~ 0
+Text Label 4350 1600 2    50   ~ 0
 CLOCK_OSC
 Wire Wire Line
-	4150 1175 4250 1175
-Wire Wire Line
-	4250 975  4150 975
+	4350 1600 4450 1600
+Wire Wire Line
+	4450 1400 4350 1400
 $Comp
 L Switch:SW_SPDT SW?
 U 1 1 5E027064
-P 4450 1075
+P 4650 1500
 AR Path="/5EC67F7B/5E027064" Ref="SW?"  Part="1"
 AR Path="/5EB09E21/5E027064" Ref="SW7"  Part="1"
-F 0 "SW7" H 4450 1425 50  0000 C CNN
-F 1 "CLOCK INPUT" H 4450 1325 50  0000 C CNN
-F 2 "Switches:SW_E-Switch_EG1271_DPDT" H 4450 1075 50  0001 C CNN
-F 3 "https://www.mouser.de/datasheet/2/140/EG-345873.pdf" H 4450 1075 50  0001 C CNN
-F 4 "E-Switch" H 4450 1075 50  0001 C CNN "Mfr."
-F 5 "EG1271" H 4450 1075 50  0001 C CNN "Mfr. No."
-F 6 "612-EG1271" H 4450 1075 50  0001 C CNN "Mouser"
-	1    4450 1075
+F 0 "SW7" H 4650 1850 50  0000 C CNN
+F 1 "CLOCK INPUT" H 4650 1750 50  0000 C CNN
+F 2 "Switches:SW_E-Switch_EG1271_DPDT" H 4650 1500 50  0001 C CNN
+F 3 "https://www.mouser.de/datasheet/2/140/EG-345873.pdf" H 4650 1500 50  0001 C CNN
+F 4 "E-Switch" H 4650 1500 50  0001 C CNN "Mfr."
+F 5 "EG1271" H 4650 1500 50  0001 C CNN "Mfr. No."
+F 6 "612-EG1271" H 4650 1500 50  0001 C CNN "Mouser"
+	1    4650 1500
 	-1   0    0    1
 $EndComp
@@
 Entry Wire Line
 	11100 3625 11200 3525
-Wire Wire Line
-	5750 4425 6200 4425
 Text HLabel 9350 1825 0    50   Output ~ 0
 ~IRQ_VIA_2
@@
 Text HLabel 4500 4725 0    50   Input ~ 0
 ~IRQ_CPU
-Wire Wire Line
-	4650 4725 4575 4725
-Text HLabel 6200 4425 2    50   Output ~ 0
-IRQ_Sync
 NoConn ~ 10700 3375
-$Comp
-L Device:R R?
-U 1 1 5E83B12B
-P 4325 4575
-AR Path="/5E83B12B" Ref="R?"  Part="1"
-AR Path="/5EB09E21/5E83B12B" Ref="R1"  Part="1"
-F 0 "R1" V 4325 4525 50  0000 L CNN
-F 1 "10k" V 4425 4525 50  0000 L CNN
-F 2 "Resistor_THT:R_Axial_DIN0207_L6.3mm_D2.5mm_P7.62mm_Horizontal" V 4255 4575 50  0001 C CNN
-F 3 "https://www.mouser.de/datasheet/2/447/Yageo%20LR_MFP_2013-594635.pdf" H 4325 4575 50  0001 C CNN
-F 4 "Yageo" H 4325 4575 50  0001 C CNN "Mfr."
-F 5 "MFP-25BRD52-10K" H 4325 4575 50  0001 C CNN "Mfr. No."
-F 6 "603-MFP-25BRD52-10K" H 4325 4575 50  0001 C CNN "Mouser"
-	1    4325 4575
-	0    -1   -1   0
-$EndComp
-Wire Wire Line
-	4475 4575 4575 4575
-Wire Wire Line
-	4575 4575 4575 4725
-Connection ~ 4575 4725
-Wire Wire Line
-	4575 4725 4500 4725
-$Comp
-L power:+5V #PWR?
-U 1 1 5E87D7A7
-P 4075 4575
-AR Path="/5E87D7A7" Ref="#PWR?"  Part="1"
-AR Path="/5EB09E21/5E87D7A7" Ref="#PWR079"  Part="1"
-F 0 "#PWR079" H 4075 4425 50  0001 C CNN
-F 1 "+5V" H 4090 4748 50  0000 C CNN
-F 2 "" H 4075 4575 50  0001 C CNN
-F 3 "" H 4075 4575 50  0001 C CNN
-	1    4075 4575
-	0    -1   -1   0
-$EndComp
-Wire Wire Line
-	4075 4575 4175 4575
 NoConn ~ 10700 3075
 Text HLabel 6200 5125 2    50   Output ~ 0
@@
 Wire Wire Line
 	6150 5025 6550 5025
+NoConn ~ 5750 4425
+Text Notes 3875 1125 0    50   ~ 0
+NOTE: WDC recommends to use an oscillator for system time base \ninstead of PHI1O and PHI2O, because the clock delay of PHI1O \nand PHI2O to PHI2 is no longer tested.
+$Comp
+L Western_Design_Center:W65C02 IC?
+U 1 1 5EBEAF78
+P 5200 5375
+AR Path="/5EBEAF78" Ref="IC?"  Part="1"
+AR Path="/5EB09E21/5EBEAF78" Ref="IC2"  Part="1"
+F 0 "IC2" H 4800 6575 50  0000 C CNN
+F 1 "W65C02" H 4890 4175 50  0000 C CNN
+F 2 "Package_DIP:DIP-40_W15.24mm_LongPads" H 5200 5075 50  0001 C CNN
+F 3 "https://www.westerndesigncenter.com/wdc/documentation/w65c02s.pdf" H 5200 5375 50  0001 C CNN
+F 4 "Western Design Center" H 5200 5375 50  0001 C CNN "Mfr."
+F 5 "W65C02S6TPG-14" H 5200 5375 50  0001 C CNN "Mfr. No."
+F 6 "955-W65C02S6TPG-14" H 5200 5375 50  0001 C CNN "Mouser"
+	1    5200 5375
+	1    0    0    -1
+$EndComp
+Wire Wire Line
+	4500 4725 4650 4725
+$Comp
+L power:+5V #PWR?
+U 1 1 5DECCA6F
+P 6200 5275
+AR Path="/5DECCA6F" Ref="#PWR?"  Part="1"
+AR Path="/5EB09E21/5DECCA6F" Ref="#PWR0107"  Part="1"
+F 0 "#PWR0107" H 6200 5125 50  0001 C CNN
+F 1 "+5V" H 6215 5448 50  0000 C CNN
+F 2 "" H 6200 5275 50  0001 C CNN
+F 3 "" H 6200 5275 50  0001 C CNN
+	1    6200 5275
+	0    1    1    0
+$EndComp
+Wire Wire Line
+	5750 5225 5825 5225
+Wire Wire Line
+	5825 5225 5825 5275
+Wire Wire Line
+	5825 5325 5750 5325
+Wire Wire Line
+	5825 5275 6200 5275
 Wire Bus Line
 	11200 2675 11200 3525
@@
 Wire Bus Line
 	7150 4725 7150 7125
+Connection ~ 5825 5275
+Wire Wire Line
+	5825 5275 5825 5325
 $EndSCHEMATC

Commit message: Optimize routing, add RDY and SYNC to expansion header
Connections:
- net RDY: now reaches IC2.2 (RDY), R3.2
- net Sync: now reaches IC2.7 (SYNC)
- net ~IRQ_Read: no longer names the net of IC2.1 (VPB)
Other:
- moved on the sheet: R3
Changed lines of the file:
@@
 NoConn ~ 5750 4925
-Wire Wire Line
-	5750 5025 5850 5025
 Wire Wire Line
 	4250 4925 4650 4925
@@
 Text Label 12700 6625 2    50   ~ 0
 R~W
-Text Label 6000 5425 0    50   ~ 0
+Text Label 5825 5425 0    50   ~ 0
 R~W
 Text HLabel 15300 7175 2    50   Output ~ 0
@@
 L power:+5V #PWR?
 U 1 1 5EBEB095
-P 6550 4950
+P 6550 4900
 AR Path="/5EBEB095" Ref="#PWR?"  Part="1"
 AR Path="/5EB09E21/5EBEB095" Ref="#PWR014"  Part="1"
-F 0 "#PWR014" H 6550 4800 50  0001 C CNN
-F 1 "+5V" H 6565 5123 50  0000 C CNN
-F 2 "" H 6550 4950 50  0001 C CNN
-F 3 "" H 6550 4950 50  0001 C CNN
-	1    6550 4950
-	1    0    0    -1
+F 0 "#PWR014" H 6550 4750 50  0001 C CNN
+F 1 "+5V" H 6565 5073 50  0000 C CNN
+F 2 "" H 6550 4900 50  0001 C CNN
+F 3 "" H 6550 4900 50  0001 C CNN
+	1    6550 4900
+	0    1    1    0
 $EndComp
 Wire Wire Line
@@
 A13
 Wire Wire Line
-	5750 8225 7500 8225
-Wire Wire Line
-	7500 8225 7500 6425
-Wire Wire Line
-	7500 6425 7600 6425
+	5750 8225 6300 8225
 Wire Wire Line
 	8000 6625 8000 6725
-$Comp
-L power:GND #PWR?
-U 1 1 5DEBFFC7
-P 7300 6725
-AR Path="/5DEBFFC7" Ref="#PWR?"  Part="1"
-AR Path="/5EB09E21/5DEBFFC7" Ref="#PWR016"  Part="1"
-F 0 "#PWR016" H 7300 6475 50  0001 C CNN
-F 1 "GND" H 7305 6552 50  0000 C CNN
-F 2 "" H 7300 6725 50  0001 C CNN
-F 3 "" H 7300 6725 50  0001 C CNN
-	1    7300 6725
-	1    0    0    -1
-$EndComp
-Wire Wire Line
-	7300 6325 7300 6725
-Wire Wire Line
-	7300 6325 7600 6325
 Wire Wire Line
 	4250 8325 5150 8325
@@
 Text Label 12350 2675 2    50   ~ 0
 ~CS_VIA_1
-Text HLabel 6200 4825 2    50   Input ~ 0
+Text HLabel 5800 4825 2    50   Input ~ 0
 ~NMI
 Wire Wire Line
@@
 NoConn ~ 5650 10425
 Wire Wire Line
-	5750 4825 6200 4825
+	5750 4825 5800 4825
 $Comp
 L Western_Design_Center:W65C22 IC10
@@
 Text HLabel 11950 4575 2    50   BiDi ~ 0
 D[0..7]
-Text HLabel 6200 5425 2    50   Output ~ 0
+Text HLabel 6025 5425 2    50   Output ~ 0
 R~W
 Wire Wire Line
-	5750 5425 6200 5425
+	5750 5425 6025 5425
 Wire Wire Line
 	5750 4325 6200 4325
@@
 	1    0    0    -1
 $EndComp
-NoConn ~ 5750 4725
 Wire Wire Line
 	5050 7575 5050 7675
@@
 NoConn ~ 10700 3375
 NoConn ~ 10700 3075
-Text HLabel 6200 5125 2    50   Output ~ 0
-~IRQ_Read
 $Comp
 L Device:R R?
 U 1 1 5EBEB08E
-P 6000 5025
+P 6350 4900
 AR Path="/5EBEB08E" Ref="R?"  Part="1"
 AR Path="/5EB09E21/5EBEB08E" Ref="R3"  Part="1"
-F 0 "R3" V 6000 4975 50  0000 L CNN
-F 1 "10k" V 5900 4950 50  0000 L CNN
-F 2 "Resistor_THT:R_Axial_DIN0207_L6.3mm_D2.5mm_P7.62mm_Horizontal" V 5930 5025 50  0001 C CNN
-F 3 "https://www.mouser.de/datasheet/2/447/Yageo%20LR_MFP_2013-594635.pdf" H 6000 5025 50  0001 C CNN
-F 4 "Yageo" H 6000 5025 50  0001 C CNN "Mfr."
-F 5 "MFP-25BRD52-10K" H 6000 5025 50  0001 C CNN "Mfr. No."
-F 6 "603-MFP-25BRD52-10K" H 6000 5025 50  0001 C CNN "Mouser"
-	1    6000 5025
+F 0 "R3" V 6350 4850 50  0000 L CNN
+F 1 "10k" V 6250 4825 50  0000 L CNN
+F 2 "Resistor_THT:R_Axial_DIN0207_L6.3mm_D2.5mm_P7.62mm_Horizontal" V 6280 4900 50  0001 C CNN
+F 3 "https://www.mouser.de/datasheet/2/447/Yageo%20LR_MFP_2013-594635.pdf" H 6350 4900 50  0001 C CNN
+F 4 "Yageo" H 6350 4900 50  0001 C CNN "Mfr."
+F 5 "MFP-25BRD52-10K" H 6350 4900 50  0001 C CNN "Mfr. No."
+F 6 "603-MFP-25BRD52-10K" H 6350 4900 50  0001 C CNN "Mouser"
+	1    6350 4900
 	0    1    1    0
 $EndComp
-Wire Wire Line
-	5750 5125 6200 5125
-Wire Wire Line
-	6550 5025 6550 4950
-Wire Wire Line
-	6150 5025 6550 5025
 NoConn ~ 5750 4425
 Text Notes 3875 1125 0    50   ~ 0
@@
 Wire Wire Line
 	5825 5275 5825 5325
+Wire Wire Line
+	6300 6425 6300 8225
+Wire Wire Line
+	6300 6425 7600 6425
+$Comp
+L power:GND #PWR?
+U 1 1 5DEBFFC7
+P 7300 6725
+AR Path="/5DEBFFC7" Ref="#PWR?"  Part="1"
+AR Path="/5EB09E21/5DEBFFC7" Ref="#PWR016"  Part="1"
+F 0 "#PWR016" H 7300 6475 50  0001 C CNN
+F 1 "GND" H 7305 6552 50  0000 C CNN
+F 2 "" H 7300 6725 50  0001 C CNN
+F 3 "" H 7300 6725 50  0001 C CNN
+	1    7300 6725
+	1    0    0    -1
+$EndComp
+Wire Wire Line
+	7300 6325 7300 6725
+Wire Wire Line
+	7300 6325 7600 6325
+Text HLabel 6350 5025 2    50   Input ~ 0
+RDY
+Wire Wire Line
+	6350 5025 6150 5025
+Wire Wire Line
+	6550 4900 6500 4900
+Connection ~ 6150 5025
+Wire Wire Line
+	6150 5025 5750 5025
+NoConn ~ 5750 5125
+Wire Wire Line
+	6200 4900 6150 4900
+Wire Wire Line
+	6150 4900 6150 5025
+Text HLabel 6350 4725 2    50   Output ~ 0
+Sync
+Wire Wire Line
+	5750 4725 6350 4725
 Wire Bus Line
 	11200 2675 11200 3525
