File: hardware/Mainboard/Mainboard.sch (KiCad schematic (older format))
At the start: 0 parts

Commit message: Misc: 	- Update README 	- Add 74HC138 datasheet 	- Update board image 	- Add layout for website tutorial
Changed lines of the file:
@@
 F6 "Clock" I R 9850 9200 50
 F7 "~Reset" O L 8250 8250 50
-F8 "CB[0..1]" O R 9850 8250 50
-F9 "A[0..15]" I R 9850 8900 50
-F10 "D[0..7]" B R 9850 9000 50
-F11 "RDY" O L 8250 8525 50
-F12 "Sync" I L 8250 8625 50
-F13 "~VP" I R 9850 8625 50
-F14 "~DCD" O R 9850 8800 50
+F8 "A[0..15]" I R 9850 8900 50
+F9 "D[0..7]" B R 9850 9000 50
+F10 "RDY" O L 8250 8525 50
+F11 "Sync" I L 8250 8625 50
+F12 "~VP" I R 9850 8625 50
+F13 "~DCD" O R 9850 8800 50
+F14 "CB[1..2]" O R 9850 8250 50
 $EndSheet
 Text Notes 900  1850 0    100  ~ 0
@@
 F13 "~IRQ_ACIA" O L 8250 7275 50
 F14 "~IRQ_CPU" I L 8250 7375 50
-F15 "CB[0..1]" I R 9850 7750 50
-F16 "A[0..15]" O R 9850 7050 50
-F17 "D[0..7]" B R 9850 7150 50
-F18 "RDY" I L 8250 7650 50
-F19 "Sync" O L 8250 7750 50
-F20 "~VP" O R 9850 7450 50
-F21 "~RTS" O R 9850 6550 50
-F22 "~CTS" I R 9850 6650 50
-F23 "~DSR" I R 9850 6850 50
-F24 "~DTR" O R 9850 6750 50
-F25 "~DCD" I R 9850 6950 50
-F26 "LCD[0..11]" B L 8250 6700 50
-F27 "Timer[0..1]" O L 8250 6900 50
+F15 "A[0..15]" O R 9850 7050 50
+F16 "D[0..7]" B R 9850 7150 50
+F17 "RDY" I L 8250 7650 50
+F18 "Sync" O L 8250 7750 50
+F19 "~VP" O R 9850 7450 50
+F20 "~RTS" O R 9850 6550 50
+F21 "~CTS" I R 9850 6650 50
+F22 "~DSR" I R 9850 6850 50
+F23 "~DTR" O R 9850 6750 50
+F24 "~DCD" I R 9850 6950 50
+F25 "LCD[0..11]" B L 8250 6700 50
+F26 "Timer[0..1]" O L 8250 6900 50
+F27 "CB[1..2]" I R 9850 7750 50
 $EndSheet
 Wire Bus Line
