File: hardware/Mainboard/Processor.sch (KiCad schematic (older format))
At the start: 22 parts, among them IC1 74HC00, IC10 W65C22, IC2 W65C02, IC3 74HC138, IC4 SYSTEM ROM, IC5 RAM, IC6 W65C22, IC7 W65C51, SW7 CLOCK INPUT, X6 EXT. CLOCK

Commit message: Misc: 	- Update README 	- Add 74HC138 datasheet 	- Update board image 	- Add layout for website tutorial
Parts:
- renumbered C2 to C1, C3 to C2, C18 to C3, C5 to C4, C1 to C5, C7 to C6, C6 to C7, IC3 to IC1, IC1 to IC3, IC10 to IC5, IC5 to IC6, IC6 to IC7, IC7 to IC8, R3 to R4, R4 to R5, SW7 to SW4, X6 to X4
Connections:
- net CB0 is gone; now on net CB1: IC7.18 (CB1)
- net CB1: no longer IC7.19 (CB2)
- new net CB2: IC7.19 (CB2)

Commit message: Hardware: 	- Add pull up resistor for PB
Documentation:
	- Add more datasheets
	- Update documentation

Misc:
	- Rename CHANGELOG
	- Remove old files

Signed-off-by: Daniel Kampert <DanielKampert@kampis-elektroecke.de>
Parts:
- C1: renamed from C2; Distributor (none) -> Mouser; Order Number (none) -> 810-FA18X8R1H104KRU6
- C2: renamed from C1; Distributor (none) -> Mouser; Order Number (none) -> 810-FA18X8R1H104KRU6
- C3, C4, C5, C6, C7: Distributor (none) -> Mouser; Order Number (none) -> 810-FA18X8R1H104KRU6
- C8: Distributor (none) -> Mouser; Order Number (none) -> 80-C315C300JCG5TA
- IC1: Distributor (none) -> Mouser; Order Number (none) -> 595-SN74HC138AN
- IC2: Distributor (none) -> Mouser; Order Number (none) -> 955-W65C02S6TPG-14
- IC3: Distributor (none) -> Mouser; Order Number (none) -> 595-SN74HC00AN
- IC4: Distributor (none) -> Mouser; Order Number (none) -> 556-AT28C25615PU
- IC5: Distributor (none) -> Mouser; Mfr. No. W65C22N6TPG-14 -> W65C22S6TPG-14; Mouser 955-W65C22N6TPG-14 -> 955-W65C22S6TPG-14; Order Number (none) -> 955-W65C22S6TPG-14
- IC6: Distributor (none) -> Mouser; Order Number (none) -> 913-AS6C62256-55PCN
- IC7: Distributor (none) -> Mouser; Mfr. No. W65C22N6TPG-14 -> W65C22S6TPG-14; Mouser 955-W65C22N6TPG-14 -> (none); Order Number (none) -> 955-W65C22S6TPG-14
- IC8: Distributor (none) -> Mouser; Order Number (none) -> 955-W65C51N6TPG-14
- R4: Distributor (none) -> Mouser; Order Number (none) -> 603-MFP-25BRD52-10K
- R5: Distributor (none) -> Mouser; Order Number (none) -> 603-MFR-25FRE52-1M
- SW4: Distributor (none) -> Mouser; Order Number (none) -> 612-EG1271
- X5: renamed from X4; Distributor (none) -> Mouser; Order Number (none) -> 538-73415-1475
- XTAL1: Distributor (none) -> Mouser; Order Number (none) -> 520-TCF100-X
- XTAL2: Distributor (none) -> Mouser; Order Number (none) -> 774-MP018B
Other:
- note added: "- WDC recommends to use an oscillator for system time base instead of PHI1O and \nPHI2O, because the clock delay of PHI1O and PHI2O to PHI2 is no longer tested."
- note added: "Info"
- note removed: "NOTE: WDC recommends to use an oscillator for system time base \ninstead of PHI1O and PHI2O, because the clock delay of PHI1O \nand PHI2O to PHI2 is no longer tested."
- moved on the sheet: C1, C2, C3, C4, C5, C6, C7, C8, IC1, IC2, IC3A, IC3B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
